File: nixx.brd (EAGLE design)
At the start: 20 x 50 mm, 2 parts

Commit message: working on it
Parts:
- added JP1, JP2: (no value), pinhead:1X07
- moved N1 0.51 mm to (10.2, 35.4)
- moved U$2 0.13 mm to (10.0, 11.7)
Changed lines of the file:
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@@
 </autorouter>
 <elements>
-<element name="N1" library="russian-nixies" package="IN-14" value="IN-14" x="9.652" y="35.433"/>
-<element name="U$2" library="Adafruit Feather M0 Adalogger" package="TQFP32-08" value="STM32F042K6" x="9.906" y="11.684"/>
+<element name="N1" library="russian-nixies" package="IN-14" value="IN-14" x="10.16" y="35.433"/>
+<element name="U$2" library="Adafruit Feather M0 Adalogger" package="TQFP32-08" value="STM32F042K6" x="10.033" y="11.684"/>
+<element name="JP1" library="pinhead" package="1X07" value="" x="9.779" y="47.752"/>
+<element name="JP2" library="pinhead" package="1X07" value="" x="10.287" y="2.032"/>
 </elements>
 <signals>
