File: nixx.sch (EAGLE design)
At the start: 2 parts

Commit message: working on it
Parts:
- added JP1, JP2: (no value), pinhead:PINHD-1X7
Changed lines of the file:
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@@
 <part name="N1" library="russian-nixies" deviceset="IN-14" device=""/>
 <part name="U$2" library="Adafruit Feather M0 Adalogger" deviceset="STM32F042K6" device=""/>
+<part name="JP1" library="pinhead" deviceset="PINHD-1X7" device=""/>
+<part name="JP2" library="pinhead" deviceset="PINHD-1X7" device=""/>
 </parts>
 <sheets>
@@
 <instance part="N1" gate="G$1" x="66.04" y="50.8"/>
 <instance part="U$2" gate="G$1" x="175.26" y="81.28"/>
+<instance part="JP1" gate="A" x="45.72" y="53.34"/>
+<instance part="JP2" gate="A" x="27.94" y="53.34"/>
 </instances>
 <busses>
