File: pcb/nixx.sch (EAGLE design)
At the start: 3 parts

Commit message: working on it
Parts:
- removed U$1: STM32F042K6-LQFP-32, Adafruit Feather M0 Adalogger:STM32F042K6-LQFP-32
- added JP1, JP2: (no value), pinhead:PINHD-1X7
- added Q1, Q10, Q2, Q3, Q4, Q5, Q6, Q7, Q8, Q9: (no value), nixx:BF820
Changed lines of the file:
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@@
 <part name="N1" library="russian-nixies" deviceset="IN-14" device=""/>
 <part name="U$2" library="Adafruit Feather M0 Adalogger" deviceset="STM32F042K6" device=""/>
-<part name="U$1" library="Adafruit Feather M0 Adalogger" deviceset="STM32F042K6" device="-LQFP-32"/>
+<part name="JP1" library="pinhead" deviceset="PINHD-1X7" device=""/>
+<part name="JP2" library="pinhead" deviceset="PINHD-1X7" device=""/>
+<part name="Q1" library="nixx" deviceset="BF820" device=""/>
+<part name="Q2" library="nixx" deviceset="BF820" device=""/>
+<part name="Q3" library="nixx" deviceset="BF820" device=""/>
+<part name="Q4" library="nixx" deviceset="BF820" device=""/>
+<part name="Q5" library="nixx" deviceset="BF820" device=""/>
+<part name="Q6" library="nixx" deviceset="BF820" device=""/>
+<part name="Q7" library="nixx" deviceset="BF820" device=""/>
+<part name="Q8" library="nixx" deviceset="BF820" device=""/>
+<part name="Q9" library="nixx" deviceset="BF820" device=""/>
+<part name="Q10" library="nixx" deviceset="BF820" device=""/>
 </parts>
 <sheets>
@@
 <instance part="N1" gate="G$1" x="66.04" y="50.8"/>
 <instance part="U$2" gate="G$1" x="175.26" y="81.28"/>
-<instance part="U$1" gate="G$1" x="114.3" y="81.28"/>
+<instance part="JP1" gate="A" x="45.72" y="53.34"/>
+<instance part="JP2" gate="A" x="27.94" y="53.34"/>
+<instance part="Q1" gate="A" x="111.76" y="60.96"/>
+<instance part="Q2" gate="A" x="111.76" y="45.72"/>
+<instance part="Q3" gate="A" x="111.76" y="30.48"/>
+<instance part="Q4" gate="A" x="111.76" y="15.24"/>
+<instance part="Q5" gate="A" x="111.76" y="0"/>
+<instance part="Q6" gate="A" x="152.4" y="60.96"/>
+<instance part="Q7" gate="A" x="152.4" y="45.72"/>
+<instance part="Q8" gate="A" x="152.4" y="30.48"/>
+<instance part="Q9" gate="A" x="152.4" y="15.24"/>
+<instance part="Q10" gate="A" x="152.4" y="-2.54"/>
 </instances>
 <busses>

Commit message: working on it
Parts:
- added C1, C2, C3: (no value), joyAnalog:CAP0805
- added D1: RGB_LED_CA-150141M173100-R&G&B, Wurth_Elektronik_Optoelectronics_rev15b:RGB_LED_CA-150141M173100-R&G&B
- added Q11, Q12: (no value), nixx:BF820
- added R1, R10, R11, R12, R13, R2, R3, R4, R5, R6, R7, R8, R9: (no value), joyAnalog:RESISTOR0805-RES
- JP1: device pinhead:PINHD-1X7 -> nixx:PINHD-1X7
Connections:
- new net +180V: N1.A, R13.1
- new net +3V3: C1.1, C2.1, C3.1, JP1.5, U$2.VDD, U$2.VDDA
- new net GND: C1.2, C2.2, C3.2, JP1.6, Q1.E, Q10.E, Q11.E, Q12.E, Q2.E, Q3.E, Q4.E, Q5.E, Q6.E, Q7.E, Q8.E, Q9.E, U$2.VSS
- new net N$1: Q1.B, R1.2
- new net N$10: Q8.B, R8.2
- new net N$11: Q9.B, R9.2
- new net N$12: Q10.B, R10.2
- new net N$13: Q11.B, R11.2
- new net N$14: Q12.B, R12.2
- new net N$2: JP1.1, R13.2
- new net N$4: Q2.B, R2.2
- new net N$5: Q3.B, R3.2
- new net N$6: Q4.B, R4.2
- new net N$7: Q5.B, R5.2
- new net N$8: Q6.B, R6.2
- new net N$9: Q7.B, R7.2
- new net NIXIE_1: N1.1, Q1.C
- new net NIXIE_10: N1.0, Q10.C
- new net NIXIE_2: N1.2, Q2.C
- new net NIXIE_3: N1.3, Q3.C
- new net NIXIE_4: N1.4, Q4.C
- new net NIXIE_5: N1.5, Q5.C
- new net NIXIE_6: N1.6, Q6.C
- new net NIXIE_7: N1.7, Q7.C
- new net NIXIE_8: N1.8, Q8.C
- new net NIXIE_9: N1.9, Q9.C
- new net NIXIE_DOT_LEFT: N1.LHDP, Q11.C
- new net NIXIE_DOT_RIGHT: N1.RHDP, Q12.C
- new net NRST: JP2.1, U$2.NRST
- new net SPI_CS: JP2.5, U$2.PA12
- new net SPI_MISO: JP2.3, U$2.PA6
- new net SPI_MOSI: JP2.4, U$2.PA7
- new net SPI_SCK: JP2.2, U$2.PA5
- new net SWD_CLK: JP2.7, U$2.PA14/SWCLK
- new net SWD_DIO: JP2.6, U$2.PA13/SWDIO
- new net UART_RX: JP1.3, U$2.PB7
- new net UART_TX: JP1.4, U$2.PB6
Other:
- moved on the sheet: JP2, N1, Q1, Q10, Q2, Q3, Q4, Q5, Q6, Q7, Q8, Q9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

Commit message: pcb routing done
Parts:
- added R14, R15, R16: (no value), joyAnalog:RESISTOR0805-RES
- added TP1, TP2, TP3: TEST-POINT3X4, joyAnalog:TEST-POINT3X4
- U$2: device Adafruit Feather M0 Adalogger:STM32F042K6 -> nixx:STM32F042K6
Connections:
- new net N$15: D1.RC, R14.1
- new net N$16: TP1.1, U$2.PF0/OSC_IN
- new net N$17: TP3.1, U$2.PB3
- new net N$18: TP2.1, U$2.PF1/OSC_OUT
- new net N$21: D1.BC, R16.1
- new net N$3: D1.GC, R15.1
- new net PWM_BLUE: R16.2, U$2.PB0
- new net PWM_GREEN: R15.2, U$2.PA4
- new net PWM_RED: R14.2, U$2.PB1
- new net STM_1: R1.1, U$2.PA1
- new net STM_10: R10.1, U$2.PA11
- new net STM_2: R2.1, U$2.PA2
- new net STM_3: R3.1, U$2.PA3
- new net STM_4: R4.1, U$2.PB5
- new net STM_5: R5.1, U$2.PA0
- new net STM_6: R6.1, U$2.PA10
- new net STM_7: R7.1, U$2.PB4
- new net STM_8: R8.1, U$2.PA8
- new net STM_9: R9.1, U$2.PA9
- new net STM_DOT_LEFT: R11.1, U$2.PA15
- new net STM_DOT_RIGHT: R12.1, U$2.PB8
- net +3V3: now also D1.A
Other:
- moved on the sheet: U$2

Commit message: silkscreen update
Parts:
- added C4: (no value), joyAnalog:CAP0805
- added R17, R18: (no value), joyAnalog:RESISTOR0805-RES
- D1: device Wurth_Elektronik_Optoelectronics_rev15b:RGB_LED_CA-150141M173100-R&G&B -> nixx:RGB_LED_CA-150141M173100-R&G&B
Connections:
- net +3V3: now also C4.1, R17.2, R18.2
- net GND: now also C4.2, JP1.7
- net NRST: now also R17.1
- net SPI_CS: now also R18.1
Changed lines of the file:
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@@
 <part name="GND15" library="joyAnalog" deviceset="GND" device=""/>
 <part name="+3V3" library="joyAnalog" deviceset="+3V3" device=""/>
-<part name="D1" library="Wurth_Elektronik_Optoelectronics_rev15b" deviceset="RGB_LED_CA" device="-150141M173100-R&amp;G&amp;B"/>
+<part name="D1" library="nixx" deviceset="RGB_LED_CA" device="-150141M173100-R&amp;G&amp;B"/>
 <part name="R13" library="joyAnalog" deviceset="RESISTOR" device="0805-RES"/>
 <part name="+3V4" library="joyAnalog" deviceset="+3V3" device=""/>
@@
 <part name="TP2" library="joyAnalog" deviceset="TEST-POINT" device="3X4" value="TEST-POINT3X4"/>
 <part name="TP3" library="joyAnalog" deviceset="TEST-POINT" device="3X4" value="TEST-POINT3X4"/>
+<part name="R17" library="joyAnalog" deviceset="RESISTOR" device="0805-RES"/>
+<part name="R18" library="joyAnalog" deviceset="RESISTOR" device="0805-RES"/>
+<part name="+3V5" library="joyAnalog" deviceset="+3V3" device=""/>
+<part name="+3V6" library="joyAnalog" deviceset="+3V3" device=""/>
+<part name="C4" library="joyAnalog" deviceset="CAP" device="0805"/>
 </parts>
 <sheets>
@@
 <instance part="TP2" gate="G$1" x="279.4" y="43.18" rot="R180"/>
 <instance part="TP3" gate="G$1" x="383.54" y="45.72"/>
+<instance part="R17" gate="G$1" x="401.32" y="17.78" rot="R90"/>
+<instance part="R18" gate="G$1" x="408.94" y="7.62" rot="R90"/>
+<instance part="+3V5" gate="G$1" x="401.32" y="25.4" rot="MR0"/>
+<instance part="+3V6" gate="G$1" x="408.94" y="15.24" rot="MR0"/>
+<instance part="C4" gate="G$1" x="109.22" y="81.28"/>
 </instances>
 <busses>
@@
 <junction x="83.82" y="78.74"/>
 <pinref part="GND14" gate="1" pin="GND"/>
+<pinref part="C4" gate="G$1" pin="2"/>
+<wire x1="99.06" y1="78.74" x2="109.22" y2="78.74" width="0.1524" layer="91"/>
+<junction x="99.06" y="78.74"/>
 </segment>
 <segment>
@@
 <pinref part="GND15" gate="1" pin="GND"/>
 <wire x1="391.16" y1="-43.18" x2="401.32" y2="-43.18" width="0.1524" layer="91"/>
+<pinref part="JP1" gate="A" pin="7"/>
+<wire x1="391.16" y1="-43.18" x2="391.16" y2="-45.72" width="0.1524" layer="91"/>
+<junction x="391.16" y="-43.18"/>
 </segment>
 </net>
@@
 <junction x="83.82" y="86.36"/>
 <pinref part="+3V2" gate="G$1" pin="+3V3"/>
+<pinref part="C4" gate="G$1" pin="1"/>
+<wire x1="99.06" y1="86.36" x2="109.22" y2="86.36" width="0.1524" layer="91"/>
+<junction x="99.06" y="86.36"/>
 </segment>
 <segment>
@@
 <wire x1="459.74" y1="0" x2="467.36" y2="0" width="0.1524" layer="91"/>
 </segment>
+<segment>
+<pinref part="R17" gate="G$1" pin="2"/>
+<pinref part="+3V5" gate="G$1" pin="+3V3"/>
+</segment>
+<segment>
+<pinref part="R18" gate="G$1" pin="2"/>
+<pinref part="+3V6" gate="G$1" pin="+3V3"/>
+</segment>
 </net>
 <net name="SPI_SCK" class="0">
@@
 <wire x1="368.3" y1="2.54" x2="391.16" y2="2.54" width="0.1524" layer="91"/>
 <label x="368.3" y="2.54" size="1.778" layer="95"/>
+<pinref part="R18" gate="G$1" pin="1"/>
+<wire x1="391.16" y1="2.54" x2="408.94" y2="2.54" width="0.1524" layer="91"/>
+<junction x="391.16" y="2.54"/>
 </segment>
 <segment>
@@
 <wire x1="368.3" y1="12.7" x2="391.16" y2="12.7" width="0.1524" layer="91"/>
 <label x="368.3" y="12.7" size="1.778" layer="95"/>
+<pinref part="R17" gate="G$1" pin="1"/>
+<wire x1="401.32" y1="12.7" x2="391.16" y2="12.7" width="0.1524" layer="91"/>
+<junction x="391.16" y="12.7"/>
 </segment>
 </net>
@@
 <pinref part="U$2" gate="G$1" pin="PB3"/>
 <wire x1="383.54" y1="45.72" x2="340.36" y2="45.72" width="0.1524" layer="91"/>
-<label x="342.9" y="45.72" size="1.778" layer="95"/>
 <pinref part="TP3" gate="G$1" pin="1"/>
 </segment>
