File: pcb/nixx.brd (EAGLE design)
At the start: 20 x 40 mm, 44 parts, among them IC1 24C64ST

Commit message: USBC, GPS etc
Parts:
- moved JP2 0.07 mm to (10.0, 2.25)
Routing:
- net SPI_SCK: track 6.85 -> 5.97 mm
Changed lines of the file:
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@@
 <grid distance="5" unitdist="mil" unit="mil" style="lines" multiple="1" display="no" altdistance="1" altunitdist="mil" altunit="mil"/>
 <layers>
-<layer number="1" name="Top" color="4" fill="1" visible="no" active="yes"/>
+<layer number="1" name="Top" color="4" fill="1" visible="yes" active="yes"/>
 <layer number="16" name="Bottom" color="1" fill="1" visible="yes" active="yes"/>
 <layer number="17" name="Pads" color="2" fill="1" visible="yes" active="yes"/>
@@
 <layer number="20" name="Dimension" color="15" fill="1" visible="yes" active="yes"/>
 <layer number="21" name="tPlace" color="7" fill="1" visible="no" active="yes"/>
-<layer number="22" name="bPlace" color="7" fill="1" visible="yes" active="yes"/>
-<layer number="23" name="tOrigins" color="15" fill="1" visible="no" active="yes"/>
-<layer number="24" name="bOrigins" color="15" fill="1" visible="yes" active="yes"/>
+<layer number="22" name="bPlace" color="7" fill="1" visible="no" active="yes"/>
+<layer number="23" name="tOrigins" color="15" fill="1" visible="yes" active="yes"/>
+<layer number="24" name="bOrigins" color="15" fill="1" visible="no" active="yes"/>
 <layer number="25" name="tNames" color="7" fill="1" visible="no" active="yes"/>
-<layer number="26" name="bNames" color="7" fill="1" visible="yes" active="yes"/>
+<layer number="26" name="bNames" color="7" fill="1" visible="no" active="yes"/>
 <layer number="27" name="tValues" color="7" fill="1" visible="no" active="yes"/>
 <layer number="28" name="bValues" color="7" fill="1" visible="no" active="yes"/>
@@
 <element name="N1" library="russian-nixies" package="IN-14" value="IN-14" x="10" y="25.381" smashed="yes"/>
 <element name="U$2" library="nixx" package="TQFP32-08" value="STM32F042K6" x="10" y="10.381" smashed="yes"/>
-<element name="JP2" library="pinhead" package="1X07" value="" x="10" y="2.181" smashed="yes">
-<attribute name="VALUE" x="1.11" y="-0.994" size="1.27" layer="27"/>
+<element name="JP2" library="pinhead" package="1X07" value="" x="10" y="2.25" smashed="yes">
+<attribute name="VALUE" x="1.11" y="-0.925" size="1.27" layer="27"/>
 </element>
 <element name="Q1" library="nixx" package="SOT323" value="" x="4.5" y="19.381" smashed="yes">
@@
 <attribute name="NAME" x="2.2987" y="33.02" size="0.8128" layer="25" font="vector" rot="R270"/>
 </element>
-<element name="JP1" library="nixx" package="1X07" value="" x="9.9746" y="37.7508" smashed="yes">
-<attribute name="VALUE" x="1.0846" y="34.5758" size="1.27" layer="27"/>
+<element name="JP1" library="nixx" package="1X07" value="" x="10" y="37.75" smashed="yes">
+<attribute name="VALUE" x="1.11" y="34.575" size="1.27" layer="27"/>
 </element>
 <element name="D1" library="nixx" package="3528-COMMON-ANODE" value="RGB_LED_CA-150141M173100-R&amp;G&amp;B" x="10" y="25.381" smashed="yes"/>
@@
 <wire x1="14.2926" y1="7.581" x2="13.374" y2="7.581" width="0.2032" layer="1"/>
 <wire x1="13.374" y1="7.581" x2="12.827" y2="8.128" width="0.2032" layer="1"/>
-<wire x1="7.4346" y1="37.7508" x2="7.4346" y2="39.624" width="0.254" layer="16"/>
-<wire x1="7.4346" y1="39.624" x2="18.2626" y2="39.624" width="0.254" layer="16"/>
 <wire x1="18.2626" y1="39.624" x2="19.177" y2="38.7096" width="0.254" layer="16"/>
 <wire x1="19.177" y1="38.7096" x2="19.177" y2="25.781" width="0.254" layer="16"/>
@@
 <wire x1="19.304" y1="1.27" x2="19.304" y2="5.3594" width="0.1778" layer="16"/>
 <wire x1="19.304" y1="5.3594" x2="17.2974" y2="7.366" width="0.1778" layer="16"/>
+<wire x1="7.46" y1="37.75" x2="7.46" y2="39.624" width="0.254" layer="16"/>
+<wire x1="7.46" y1="39.624" x2="18.2626" y2="39.624" width="0.254" layer="16"/>
 </signal>
 <signal name="SPI_SCK">
@@
 <wire x1="8.382" y1="4.191" x2="6.096" y2="4.191" width="0.254" layer="1"/>
 <wire x1="6.096" y1="4.191" x2="4.953" y2="3.048" width="0.254" layer="1"/>
-<wire x1="4.953" y1="3.048" x2="4.953" y2="2.214" width="0.254" layer="1"/>
-<wire x1="4.953" y1="2.214" x2="4.92" y2="2.181" width="0.254" layer="1"/>
+<wire x1="4.92" y1="2.25" x2="4.953" y2="3.048" width="0" layer="19" extent="1-1"/>
 </signal>
 <signal name="SPI_MISO">
 <contactref element="JP2" pad="3"/>
 <contactref element="U$2" pad="12"/>
-<wire x1="9.6" y1="6.0884" x2="9.6" y2="4.321" width="0.254" layer="1"/>
-<wire x1="9.6" y1="4.321" x2="7.46" y2="2.181" width="0.254" layer="1"/>
+<wire x1="9.6" y1="6.0884" x2="9.6" y2="4.39" width="0.254" layer="1"/>
+<wire x1="9.6" y1="4.39" x2="7.46" y2="2.25" width="0.254" layer="1"/>
 </signal>
 <signal name="SPI_MOSI">
 <contactref element="JP2" pad="4"/>
 <contactref element="U$2" pad="13"/>
-<wire x1="10.4" y1="6.0884" x2="10.4" y2="2.581" width="0.254" layer="1"/>
-<wire x1="10.4" y1="2.581" x2="10" y2="2.181" width="0.254" layer="1"/>
+<wire x1="10.4" y1="6.0884" x2="10.4" y2="2.65" width="0.254" layer="1"/>
+<wire x1="10.4" y1="2.65" x2="10" y2="2.25" width="0.254" layer="1"/>
 </signal>
 <signal name="SPI_CS">
@@
 <wire x1="11.684" y1="12.192" x2="11.684" y2="6.466" width="0.2032" layer="16"/>
 <wire x1="11.684" y1="6.466" x2="12.816" y2="5.334" width="0.2032" layer="16"/>
-<wire x1="12.54" y1="2.181" x2="12.54" y2="5.058" width="0.2032" layer="16"/>
+<wire x1="12.54" y1="2.25" x2="12.54" y2="5.058" width="0.2032" layer="16"/>
 <wire x1="12.54" y1="5.058" x2="12.816" y2="5.334" width="0.2032" layer="16"/>
 <contactref element="U$2" pad="25"/>
@@
 <via x="15.748" y="12.446" extent="1-16" drill="0.5"/>
 <wire x1="15.748" y1="12.446" x2="15.748" y2="2.849" width="0.2032" layer="16"/>
-<wire x1="15.748" y1="2.849" x2="15.08" y2="2.181" width="0.2032" layer="16"/>
+<wire x1="15.748" y1="2.849" x2="15.149" y2="2.25" width="0.2032" layer="16"/>
+<wire x1="15.149" y1="2.25" x2="15.08" y2="2.25" width="0.2032" layer="16"/>
 </signal>
 <signal name="SWD_CLK">
@@
 <wire x1="16.891" y1="12.7" x2="16.891" y2="3.302" width="0.2032" layer="16"/>
 <wire x1="16.891" y1="3.302" x2="17.62" y2="2.573" width="0.2032" layer="16"/>
-<wire x1="17.62" y1="2.573" x2="17.62" y2="2.181" width="0.2032" layer="16"/>
+<wire x1="17.62" y1="2.573" x2="17.62" y2="2.25" width="0.2032" layer="16"/>
 </signal>
 <signal name="NRST">
@@
 <wire x1="4.812" y1="10.781" x2="4.064" y2="10.033" width="0.2032" layer="1"/>
 <wire x1="4.688" y1="9.409" x2="4.064" y2="10.033" width="0.2032" layer="16"/>
-<wire x1="2.38" y1="2.181" x2="2.38" y2="3.142" width="0.2032" layer="16"/>
+<wire x1="2.38" y1="2.25" x2="2.38" y2="3.142" width="0.2032" layer="16"/>
 <wire x1="2.38" y1="3.142" x2="4.699" y2="5.461" width="0.2032" layer="16"/>
 <wire x1="4.699" y1="5.461" x2="4.699" y2="6.212" width="0.2032" layer="16"/>
@@
 <wire x1="4.445" y1="29.464" x2="4.445" y2="33.02" width="0.2032" layer="16"/>
 <wire x1="7.112" y1="35.687" x2="9.525" y2="35.687" width="0.2032" layer="16"/>
-<wire x1="9.525" y1="35.687" x2="9.906" y2="36.068" width="0.2032" layer="16"/>
-<wire x1="9.906" y1="36.068" x2="9.906" y2="37.6822" width="0.2032" layer="16"/>
-<wire x1="9.906" y1="37.6822" x2="9.9746" y2="37.7508" width="0.2032" layer="16"/>
 <wire x1="7.112" y1="35.687" x2="4.445" y2="33.02" width="0.2032" layer="16"/>
+<wire x1="9.525" y1="35.687" x2="10" y2="36.162" width="0.2032" layer="16"/>
+<wire x1="10" y1="36.162" x2="10" y2="37.75" width="0.2032" layer="16"/>
 </signal>
 <signal name="UART_TX">
@@
 <wire x1="6.985" y1="34.29" x2="7.874" y2="35.179" width="0.2032" layer="16"/>
 <wire x1="7.874" y1="35.179" x2="11.811" y2="35.179" width="0.2032" layer="16"/>
-<wire x1="11.811" y1="35.179" x2="12.5146" y2="35.8826" width="0.2032" layer="16"/>
-<wire x1="12.5146" y1="35.8826" x2="12.5146" y2="37.7508" width="0.2032" layer="16"/>
 <wire x1="9.6" y1="14.6736" x2="9.6" y2="16.943" width="0.2032" layer="1"/>
 <wire x1="9.6" y1="16.943" x2="8.89" y2="17.653" width="0.2032" layer="1"/>
 <wire x1="8.89" y1="17.653" x2="8.255" y2="18.288" width="0.2032" layer="16"/>
 <wire x1="8.255" y1="18.288" x2="8.255" y2="26.416" width="0.2032" layer="16"/>
+<wire x1="11.811" y1="35.179" x2="12.54" y2="35.908" width="0.2032" layer="16"/>
+<wire x1="12.54" y1="35.908" x2="12.54" y2="37.75" width="0.2032" layer="16"/>
 </signal>
 <signal name="N$2">
 <contactref element="JP1" pad="1"/>
 <contactref element="R13" pad="2"/>
-<wire x1="2.3546" y1="37.7508" x2="3.6038" y2="39" width="0.4064" layer="1"/>
-<wire x1="3.6038" y1="39" x2="4.953" y2="39" width="0.4064" layer="1"/>
+<wire x1="2.38" y1="37.75" x2="3.63" y2="39" width="0.4064" layer="1"/>
+<wire x1="3.63" y1="39" x2="4.953" y2="39" width="0.4064" layer="1"/>
 </signal>
 <signal name="STM_DOT_LEFT">

Commit message: added bake control
Parts:
- removed C4: 100nF, joyAnalog:0805
- removed IC1: 24C64ST, joyAnalog:TSSOP8
- removed R20: 4K7, joyAnalog:0805
- removed R21: 10K, joyAnalog:0805
- added Q13: (no value), nixx:SOT323
- added R22, R23: 10K, joyAnalog:0805
- added R24: 4K7, joyAnalog:0805
- added T1: (no value), zetex:SOT323
- added TP2, TP3, TP4: PTR1TP13R, testpad:TP13R
- R13: value 10K -> 68K
- R19: value 4K7 -> 10K
- moved R19 28.2 mm to (10.0, 36.7), flipped to the top, turned to 90 degrees
- moved C3 17.2 mm to (18.4, 33.1)
- moved TP1 5.78 mm to (7.37, 11.4)
- moved R4 5.10 mm to (1.69, 32.3), turned to 270 degrees
- moved R13 2.65 mm to (5.71, 35.6), turned to 180 degrees
Connections:
- removed net N$17: TP1.TP, U$2.22
- removed net N$18: IC1.6, R19.1, U$2.3
- new net BAKE: R24.2, U$2.22
- new net N$19: JP1.1, R13.2, R19.1, T1.3
- new net N$20: R22.1, T1.2
- new net N$22: Q13.3, R19.2, R22.2
- new net N$23: Q13.1, R24.1
- new net N$24: R23.2, T1.1
- net +180V: now also R23.1
- net +3V3: now also JP1.7; no longer C4.1, IC1.8, JP1.3, R19.2, R20.2
- net GND: now also Q13.2; no longer C4.2, IC1.1, IC1.2, IC1.3, IC1.4, IC1.7, JP1.7, R21.1
- net N$16: now also TP2.TP, U$2.3; no longer IC1.5, R20.1, U$2.2
- net N$2: now also TP1.TP, U$2.2; no longer JP1.1, R13.2
- net STM_DOT_RIGHT: no longer R21.2
- net UART_RX: now also TP4.TP; no longer JP1.4
- net UART_TX: now also TP3.TP; no longer JP1.5
Routing:
- net BAKE: track 0.00 -> 40.0 mm, vias 0 -> 2
- net UART_RX: track 34.2 -> 1.73 mm
- net +3V3: track 143.6 -> 114.1 mm, vias 5 -> 4
- net UART_TX: track 30.1 -> 2.89 mm
- net N$19: track 0.00 -> 10.6 mm
- net N$18: track 9.27 -> 0.00 mm, vias 1 -> 0
- net STM_4: track 25.4 -> 31.1 mm
- net N$16: track 5.99 -> 1.74 mm
- net N$22: track 0.00 -> 3.97 mm
- net N$20: track 0.00 -> 3.45 mm
- net +180V: track 23.1 -> 19.7 mm
- net N$17: track 3.21 -> 0.00 mm, vias 1 -> 0
- net STM_DOT_RIGHT: track 9.09 -> 6.95 mm, vias 1 -> 0
- net N$24: track 0.00 -> 1.85 mm
- net N$23: track 0.00 -> 1.69 mm
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Other:
- board text removed: "PA12"

Commit message: positioned boards
Parts:
- moved TP3 0.99 mm to (9.53, 11.4)
- moved JP1 0.45 mm to (10.0, 38.2)
- moved JP2 0.45 mm to (10.0, 1.80)
Routing:
- net +3V3: track 114.1 -> 72.8 mm
- net GND: track 60.9 -> 65.4 mm
- net SPI_CS: track 13.6 -> 14.5 mm

Commit message: fixed bake
Parts:
- R15: value 470 -> 1K
- R16: value 0 -> 470
- R19, R22: value 10K -> 100K
- R23: value 10K -> 75K
Changed lines of the file:
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@@
 <setting verticaltext="up"/>
 </settings>
-<grid distance="5" unitdist="mil" unit="mm" style="lines" multiple="1" display="no" altdistance="1" altunitdist="mil" altunit="mil"/>
+<grid distance="5" unitdist="mil" unit="mil" style="lines" multiple="1" display="no" altdistance="1" altunitdist="mil" altunit="mil"/>
 <layers>
 <layer number="1" name="Top" color="4" fill="1" visible="yes" active="yes"/>
@@
 <attribute name="NAME" x="16.3195" y="8.255" size="0.8128" layer="25" font="vector" rot="R90"/>
 </element>
-<element name="R15" library="joyAnalog" package="0805" value="470" x="3.048" y="4.953" smashed="yes">
+<element name="R15" library="joyAnalog" package="0805" value="1K" x="3.048" y="4.953" smashed="yes">
 <attribute name="NAME" x="3.7211" y="6.0198" size="0.8128" layer="25" font="vector" rot="R90"/>
 </element>
-<element name="R16" library="joyAnalog" package="0805" value="0" x="19.05" y="6.731" smashed="yes" rot="R270">
+<element name="R16" library="joyAnalog" package="0805" value="470" x="19.05" y="6.731" smashed="yes" rot="R270">
 <attribute name="NAME" x="17.3863" y="8.2804" size="0.8128" layer="25" font="vector" rot="R90"/>
 </element>
@@
 <attribute name="TP_SIGNAL_NAME" value="" x="7.366" y="8.89" size="1" layer="38" rot="MR0"/>
 </element>
-<element name="R22" library="joyAnalog" package="0805" value="10K" x="9.017" y="39.116" smashed="yes">
-<attribute name="NAME" x="7.747" y="39.8145" size="0.6096" layer="25" rot="R180"/>
-</element>
-<element name="R23" library="joyAnalog" package="0805" value="10K" x="8.255" y="36.703" smashed="yes" rot="R90">
+<element name="R22" library="joyAnalog" package="0805" value="100K" x="9.017" y="39.116" smashed="yes">
+<attribute name="NAME" x="7.62" y="39.6875" size="0.6096" layer="25" rot="R180"/>
+</element>
+<element name="R23" library="joyAnalog" package="0805" value="75K" x="8.255" y="36.703" smashed="yes" rot="R90">
 <attribute name="NAME" x="5.969" y="36.3855" size="0.6096" layer="25"/>
 </element>
@@
 <attribute name="NAME" x="10.9855" y="35.179" size="0.6096" layer="25" rot="R270"/>
 </element>
-<element name="R19" library="joyAnalog" package="0805" value="10K" x="10.033" y="36.703" smashed="yes" rot="R90">
+<element name="R19" library="joyAnalog" package="0805" value="100K" x="10.033" y="36.703" smashed="yes" rot="R90">
 <attribute name="NAME" x="8.509" y="34.6075" size="0.6096" layer="25"/>
 </element>
@@
 <contactref element="R13" pad="1"/>
 <via x="10.033" y="33.02" extent="1-16" drill="0.7"/>
-<wire x1="10.033" y1="33.02" x2="10.033" y2="19.2241" width="0.3048" layer="16"/>
+<wire x1="10.033" y1="33.02" x2="10.033" y2="19.2241" width="0.4064" layer="16"/>
 <wire x1="10.033" y1="19.2241" x2="10" y2="19.1911" width="0.3048" layer="16"/>
 <contactref element="R23" pad="1"/>
-<wire x1="6.615" y1="35.56" x2="6.858" y2="35.803" width="0.3048" layer="1"/>
-<wire x1="6.858" y1="35.803" x2="8.255" y2="35.803" width="0.3048" layer="1"/>
-<wire x1="8.255" y1="35.803" x2="8.255" y2="35.56" width="0.3048" layer="1"/>
-<wire x1="8.255" y1="35.56" x2="9.017" y2="34.798" width="0.3048" layer="1"/>
-<wire x1="9.017" y1="34.798" x2="10.033" y2="34.798" width="0.3048" layer="1"/>
-<wire x1="10.033" y1="34.798" x2="10.033" y2="33.02" width="0.3048" layer="1"/>
+<wire x1="10.033" y1="34.671" x2="10.033" y2="33.02" width="0.4064" layer="1"/>
+<wire x1="6.615" y1="35.56" x2="6.858" y2="35.803" width="0.4064" layer="1"/>
+<wire x1="6.858" y1="35.803" x2="8.255" y2="35.803" width="0.4064" layer="1"/>
+<wire x1="8.255" y1="35.803" x2="8.255" y2="34.671" width="0.4064" layer="1"/>
+<wire x1="8.255" y1="34.671" x2="10.033" y2="34.671" width="0.4064" layer="1"/>
 </signal>
 <signal name="GND">
@@
 <wire x1="10.4" y1="17.512" x2="10.541" y2="17.653" width="0.2032" layer="1"/>
 <wire x1="11.176" y1="18.288" x2="11.176" y2="29.21" width="0.2032" layer="16"/>
-<via x="7.62" y="33.274" extent="1-16" drill="0.5"/>
+<via x="7.493" y="33.274" extent="1-16" drill="0.5"/>
 <wire x1="12.827" y1="30.861" x2="12.827" y2="32.004" width="0.2032" layer="16"/>
 <wire x1="12.827" y1="32.004" x2="12.192" y2="32.639" width="0.2032" layer="16"/>
@@
 <wire x1="11.176" y1="33.02" x2="11.176" y2="33.655" width="0.2032" layer="16"/>
 <wire x1="11.176" y1="33.655" x2="10.795" y2="34.036" width="0.2032" layer="16"/>
-<wire x1="10.795" y1="34.036" x2="8.382" y2="34.036" width="0.2032" layer="16"/>
-<wire x1="8.382" y1="34.036" x2="7.62" y2="33.274" width="0.2032" layer="16"/>
-<wire x1="1.687" y1="33.157" x2="7.503" y2="33.157" width="0.2032" layer="1"/>
-<wire x1="7.503" y1="33.157" x2="7.62" y2="33.274" width="0.2032" layer="1"/>
+<wire x1="1.687" y1="33.157" x2="1.687" y2="33.274" width="0.2032" layer="1"/>
+<wire x1="1.687" y1="33.274" x2="7.493" y2="33.274" width="0.2032" layer="1"/>
+<wire x1="8.255" y1="34.036" x2="7.493" y2="33.274" width="0.2032" layer="16"/>
+<wire x1="10.795" y1="34.036" x2="8.255" y2="34.036" width="0.2032" layer="16"/>
 </signal>
 <signal name="STM_3">
@@
 <contactref element="R13" pad="2"/>
 <contactref element="R19" pad="1"/>
-<wire x1="2.68" y1="37.45" x2="4.815" y2="37.45" width="0.3048" layer="1"/>
-<wire x1="4.815" y1="37.45" x2="4.815" y2="36.703" width="0.3048" layer="1"/>
-<wire x1="4.815" y1="36.703" x2="4.815" y2="35.56" width="0.3048" layer="1"/>
-<wire x1="10.033" y1="35.803" x2="10.033" y2="36.703" width="0.3048" layer="1"/>
-<wire x1="10.033" y1="36.703" x2="4.815" y2="36.703" width="0.3048" layer="1"/>
-<wire x1="2.38" y1="38.2" x2="2.38" y2="37.75" width="0.3048" layer="1"/>
-<wire x1="2.38" y1="37.75" x2="2.68" y2="37.45" width="0.3048" layer="1"/>
+<wire x1="2.68" y1="37.45" x2="4.815" y2="37.45" width="0.4064" layer="1"/>
+<wire x1="4.815" y1="37.45" x2="4.815" y2="36.703" width="0.4064" layer="1"/>
+<wire x1="4.815" y1="36.703" x2="4.815" y2="35.56" width="0.4064" layer="1"/>
+<wire x1="10.033" y1="35.803" x2="10.033" y2="36.703" width="0.4064" layer="1"/>
+<wire x1="10.033" y1="36.703" x2="4.815" y2="36.703" width="0.4064" layer="1"/>
+<wire x1="2.38" y1="38.2" x2="2.38" y2="37.75" width="0.4064" layer="1"/>
+<wire x1="2.38" y1="37.75" x2="2.68" y2="37.45" width="0.4064" layer="1"/>
 </signal>
 <signal name="N$20">
 <contactref element="T1" pad="2"/>
 <contactref element="R22" pad="1"/>
-<wire x1="4.815" y1="38.75" x2="5.181" y2="39.116" width="0.3048" layer="1"/>
-<wire x1="5.181" y1="39.116" x2="8.117" y2="39.116" width="0.3048" layer="1"/>
+<wire x1="4.815" y1="38.75" x2="5.181" y2="39.116" width="0.4064" layer="1"/>
+<wire x1="5.181" y1="39.116" x2="8.117" y2="39.116" width="0.4064" layer="1"/>
 </signal>
 <signal name="N$22">
@@
 <contactref element="Q13" pad="3"/>
 <contactref element="R19" pad="2"/>
-<wire x1="9.917" y1="37.603" x2="9.917" y2="39.116" width="0.3048" layer="1"/>
-<wire x1="9.917" y1="37.603" x2="10.033" y2="37.603" width="0.3048" layer="1"/>
-<wire x1="9.917" y1="39.116" x2="9.917" y2="39.127" width="0.3048" layer="1"/>
-<wire x1="9.917" y1="39.116" x2="12.054" y2="39.116" width="0.3048" layer="1"/>
-<wire x1="12.054" y1="39.116" x2="12.192" y2="39.254" width="0.3048" layer="1"/>
+<wire x1="9.917" y1="39.127" x2="9.917" y2="39.116" width="0.3048" layer="1"/>
+<wire x1="9.917" y1="39.116" x2="10.033" y2="39" width="0.4064" layer="1"/>
+<wire x1="10.033" y1="39" x2="10.033" y2="37.603" width="0.4064" layer="1"/>
+<wire x1="9.917" y1="39.116" x2="10.055" y2="39.254" width="0.4064" layer="1"/>
+<wire x1="10.055" y1="39.254" x2="12.192" y2="39.254" width="0.4064" layer="1"/>
 </signal>
 <signal name="N$23">
 <contactref element="Q13" pad="1"/>
 <contactref element="R24" pad="1"/>
-<wire x1="11.542" y1="37.454" x2="11.542" y2="35.937" width="0.3048" layer="1"/>
-<wire x1="11.542" y1="35.937" x2="11.419" y2="35.814" width="0.3048" layer="1"/>
+<wire x1="11.542" y1="37.454" x2="11.542" y2="35.937" width="0.4064" layer="1"/>
+<wire x1="11.542" y1="35.937" x2="11.419" y2="35.814" width="0.4064" layer="1"/>
 </signal>
 <signal name="N$24">
 <contactref element="T1" pad="1"/>
 <contactref element="R23" pad="2"/>
-<wire x1="6.615" y1="38.1" x2="7.112" y2="37.603" width="0.3048" layer="1"/>
-<wire x1="7.112" y1="37.603" x2="8.255" y2="37.603" width="0.3048" layer="1"/>
+<wire x1="6.615" y1="38.1" x2="7.112" y2="37.603" width="0.4064" layer="1"/>
+<wire x1="7.112" y1="37.603" x2="8.255" y2="37.603" width="0.4064" layer="1"/>
 </signal>
 <signal name="N$2">
@@
 <wire x1="6.985" y1="34.544" x2="12.192" y2="34.544" width="0.2032" layer="16"/>
 <via x="12.192" y="34.544" extent="1-16" drill="0.5"/>
-<wire x1="12.192" y1="34.544" x2="13.219" y2="35.571" width="0.2032" layer="1"/>
-<wire x1="13.219" y1="35.571" x2="13.219" y2="35.814" width="0.2032" layer="1"/>
 <wire x1="7.493" y1="29.464" x2="7.493" y2="30.48" width="0.2032" layer="16"/>
 <wire x1="7.493" y1="30.48" x2="6.477" y2="31.496" width="0.2032" layer="16"/>
 <wire x1="6.477" y1="31.496" x2="6.477" y2="34.036" width="0.2032" layer="16"/>
+<wire x1="13.219" y1="35.814" x2="13.219" y2="35.571" width="0.4064" layer="1"/>
+<wire x1="13.219" y1="35.571" x2="12.192" y2="34.544" width="0.4064" layer="1"/>
 </signal>
 </signals>

Commit message: 6 tube time display
Parts:
- R19, R22: value 100K -> 1M
- R23: value 75K -> 100K
Changed lines of the file:
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@@
 <attribute name="TP_SIGNAL_NAME" value="" x="7.366" y="8.89" size="1" layer="38" rot="MR0"/>
 </element>
-<element name="R22" library="joyAnalog" package="0805" value="100K" x="9.017" y="39.116" smashed="yes">
+<element name="R22" library="joyAnalog" package="0805" value="1M" x="9.017" y="39.116" smashed="yes">
 <attribute name="NAME" x="7.62" y="39.6875" size="0.6096" layer="25" rot="R180"/>
 </element>
-<element name="R23" library="joyAnalog" package="0805" value="75K" x="8.255" y="36.703" smashed="yes" rot="R90">
+<element name="R23" library="joyAnalog" package="0805" value="100K" x="8.255" y="36.703" smashed="yes" rot="R90">
 <attribute name="NAME" x="5.969" y="36.3855" size="0.6096" layer="25"/>
 </element>
@@
 <attribute name="NAME" x="10.9855" y="35.179" size="0.6096" layer="25" rot="R270"/>
 </element>
-<element name="R19" library="joyAnalog" package="0805" value="100K" x="10.033" y="36.703" smashed="yes" rot="R90">
+<element name="R19" library="joyAnalog" package="0805" value="1M" x="10.033" y="36.703" smashed="yes" rot="R90">
 <attribute name="NAME" x="8.509" y="34.6075" size="0.6096" layer="25"/>
 </element>
