File: pcb/clock.brd (EAGLE design)
At the start: 145 x 50 mm, 69 parts, among them IC1 STM32F072C8T6, IC2 REG1117, IC3 24C64ST, X3 USB-MICROB

Commit message: added gps header
Parts:
- added JP4: (no value), pinhead:2X02
- added R17: (no value), clock:0805
- moved LED2 16.5 mm to (10.0, 4.83), turned to 0 degrees
- moved R7 9.40 mm to (138.8, 6.99)
- moved R9 9.00 mm to (13.0, 4.95), turned to 90 degrees
- moved PWR 6.51 mm to (137.0, 4.45)
- moved S4 3.00 mm to (113.0, 2.10)
- moved S5 3.00 mm to (128.0, 2.10)
Connections:
- net +5V: now also R17.2
- net GND: now also JP4.1
- net GPS_TP: now also JP4.3
- net N$21: now also R9.2; no longer R9.1
- net NIXIE_PWR_EN: now also R17.1
- net RX3: now also R9.1
- net TX3: no longer R9.2
- net USART1_RX: now also JP4.4
- net USART1_TX: now also JP4.2
Routing:
- net GPS_TP: track 65.6 -> 103.9 mm
- net USART1_RX: track 49.5 -> 82.0 mm
- net USART1_TX: track 50.9 -> 81.9 mm
- net +5V: track 60.7 -> 68.2 mm
- net RX3: track 47.9 -> 51.6 mm
- net NIXIE_PWR_EN: track 7.97 -> 10.6 mm
- net TX3: track 51.9 -> 49.6 mm
- net N$23: track 126.5 -> 124.5 mm
- net N$21: track 4.80 -> 2.93 mm
- net N$22: track 109.2 -> 108.4 mm
- net +3V3: track 80.5 -> 80.3 mm, vias 11 -> 12
