File: pcb/clock.brd (EAGLE design)
At the start: 145 x 50 mm, 69 parts, among them IC1 STM32F072C8T6, IC2 REG1117, IC3 24C64ST, X3 USB-MICROB

Commit message: new routing
Parts:
- removed U$9: DS18B20, DS18B20U:MSOP8
- added C1, C3: (no value), clock:0805
- added TP4: TEST-POINT3X5, SparkFun-Passives:PAD.03X.05
- added U1: DS18B20, SparkFun-Sensors:TO-92-AMMO
- TP2, TP3: value PTR1TP20R -> TEST-POINT3X5; device testpad:TP20R -> SparkFun-Passives:PAD.03X.05
- moved TP2 33.1 mm to (50.7, 25.5), flipped to the bottom
- moved TP3 30.8 mm to (49.9, 22.1)
- moved R16 3.56 mm to (140.3, 12.7), turned to 90 degrees
- moved R7 2.41 mm to (135.3, 6.22), turned to 0 degrees
- moved SD1 0.65 mm to (137.2, 25.4)
Connections:
- removed net N$22: IC1.31, S4.1
- removed net N$23: IC1.29, S5.1
- removed net N$24: IC1.30, R9.2
- removed net VDD: SD1.4
- removed net VSS: SD1.6
- new net A_BUTTON: IC1.5, S4.1
- new net B_BUTTON: IC1.6, S5.1
- new net GPS_FIX_LED: IC1.17, R9.2
- new net N$15: IC1.29, TP4.P$1
- new net N$6: IC1.31, TP2.P$1
- new net N$7: IC1.30, TP3.P$1
- new net SD_CS: IC1.10, SD1.2
- net +3V3: now also C1.1, C3.1, SD1.4, U1.3; no longer U$9.8
- net DS18B20_DATA: now also IC1.16, U1.2; no longer IC1.2, U$9.1
- net GND: now also C1.2, C3.2, SD1.6, U1.1; no longer U$9.4
- net GPS_RESET: now also IC1.2; no longer IC1.10
- net USART1_RX: no longer TP3.TP
- net USART1_TX: no longer TP2.TP
Routing:
- net N$23: track 128.1 -> 0.00 mm, vias 2 -> 0
- net DS18B20_DATA: track 0.00 -> 127.8 mm, vias 0 -> 2
- net GPS_FIX_LED: track 0.00 -> 110.1 mm, vias 0 -> 2
- net B_BUTTON: track 0.00 -> 107.9 mm, vias 0 -> 2
- net N$22: track 105.7 -> 0.00 mm, vias 2 -> 0
- net N$24: track 104.1 -> 0.00 mm, vias 2 -> 0
- net A_BUTTON: track 0.00 -> 94.5 mm, vias 0 -> 2
- net SD_CS: track 0.00 -> 91.1 mm, vias 0 -> 2
- net GND: track 137.6 -> 174.9 mm, vias 1 -> 2
- net GPS_RESET: track 71.8 -> 46.1 mm, vias 2 -> 0
- net SPI1_MOSI: track 197.8 -> 219.0 mm
- net SPI1_SCK: track 157.6 -> 174.3 mm
- net +3V3: track 76.0 -> 92.4 mm, vias 11 -> 12
- net SPI1_MISO: track 196.0 -> 210.1 mm
- net N$15: track 0.00 -> 5.59 mm, vias 0 -> 1
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Other:
- board text added: "+"
- board text added: "-"
- board text added: "A"
- board text added: "B"
- board text added: "PA10"
- board text added: "PA8"
- board text added: "PA9"
- board text removed: "DOWN"
- board text removed: "UP"

Commit message: main clock board adj
Parts:
- moved U$20 3.56 mm to (88.6, 32.0)
- moved LED2 1.40 mm to (140.1, 40.8)
- moved R9 1.40 mm to (140.1, 37.0)
Routing:
- net GPS_FIX_LED: track 110.1 -> 111.5 mm
- net +3V3: track 92.4 -> 93.8 mm
Changed lines of the file:
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@@
 <?xml version="1.0" encoding="utf-8"?>
 <!DOCTYPE eagle SYSTEM "eagle.dtd">
-<eagle version="8.2.0">
+<eagle version="8.2.2">
 <drawing>
 <settings>
-<setting alwaysvectorfont="no"/>
+<setting alwaysvectorfont="yes"/>
 <setting verticaltext="up"/>
 </settings>
@@
 <text x="114.427" y="7.874" size="2.54" layer="25" rot="R180">A</text>
 <text x="129.54" y="7.874" size="2.54" layer="25" rot="R180">B</text>
-<text x="139.954" y="42.672" size="1.27" layer="25" rot="R270">GPS
+<text x="141.224" y="42.799" size="1.27" layer="25" rot="R270">GPS
 FIX</text>
 <text x="46.355" y="21.59" size="1.016" layer="25">PA9</text>
@@
 <attribute name="OC_NEWARK" value="08R5418" x="61.341" y="33.401" size="1.778" layer="27" rot="R180" display="off"/>
 </element>
-<element name="LED2" library="backplane" package="CHIP-LED0805" value="" x="138.684" y="40.767" smashed="yes" rot="R180">
-<attribute name="VALUE" x="136.144" y="42.037" size="1.27" layer="27" rot="R270"/>
+<element name="LED2" library="backplane" package="CHIP-LED0805" value="" x="140.081" y="40.767" smashed="yes" rot="R180">
+<attribute name="VALUE" x="137.541" y="42.037" size="1.27" layer="27" rot="R270"/>
 </element>
 <element name="PWR" library="backplane" package="CHIP-LED0805" value="" x="136.779" y="2.921" smashed="yes">
@@
 </element>
 <element name="R7" library="clock" package="0805" value="" x="135.255" y="6.223" smashed="yes">
-<attribute name="NAME" x="133.477" y="4.5085" size="0.8128" layer="25"/>
+<attribute name="NAME" x="134.747" y="7.3025" size="0.8128" layer="25"/>
 </element>
 <element name="R8" library="clock" package="0805" value="" x="76.8604" y="3.937" smashed="yes" rot="R270">
@@
 <attribute name="NAME" x="81.7245" y="24.13" size="0.8128" layer="25" rot="R90"/>
 </element>
-<element name="R9" library="clock" package="0805" value="" x="138.684" y="36.957" rot="R270"/>
-<element name="U$20" library="a" package="M3_MOUNTING_HOLE_PACK" value="M3_MOUNTING_HOLE" x="85" y="32"/>
+<element name="R9" library="clock" package="0805" value="" x="140.081" y="36.957" rot="R270"/>
+<element name="U$20" library="a" package="M3_MOUNTING_HOLE_PACK" value="M3_MOUNTING_HOLE" x="88.556" y="32"/>
 <element name="SD1" library="basicBoard" package="TF-PULL" value="TF-HOLDER" x="137.16" y="25.4" smashed="yes" rot="R270"/>
-<element name="C1" library="clock" package="0805" value="" x="126.238" y="24.511" rot="R180"/>
-<element name="C3" library="clock" package="0805" value="" x="126.238" y="26.289" rot="R180"/>
+<element name="C1" library="clock" package="0805" value="" x="126.238" y="24.511" smashed="yes" rot="R180">
+<attribute name="NAME" x="127" y="23.5585" size="0.8128" layer="25" rot="R180"/>
+</element>
+<element name="C3" library="clock" package="0805" value="" x="126.238" y="26.289" smashed="yes" rot="R180">
+<attribute name="NAME" x="127" y="28.0035" size="0.8128" layer="25" rot="R180"/>
+</element>
 <element name="U1" library="SparkFun-Sensors" package="TO-92-AMMO" value="DS18B20" x="143.002" y="11.049" smashed="yes" rot="R90">
 <attribute name="NAME" x="141.097" y="14.224" size="0.4064" layer="25" ratio="10" rot="R90"/>
@@
 <wire x1="134.9502" y1="1.8796" x2="136.7704" y2="1.8796" width="0.2032" layer="1"/>
 <wire x1="136.7704" y1="1.8796" x2="136.779" y2="1.871" width="0.2032" layer="1"/>
-<wire x1="138.684" y1="41.817" x2="134.843" y2="41.817" width="0.2032" layer="1"/>
+<wire x1="140.081" y1="41.817" x2="134.843" y2="41.817" width="0.2032" layer="1"/>
 <wire x1="134.843" y1="41.817" x2="134.369" y2="42.291" width="0.2032" layer="1"/>
 <contactref element="SD1" pad="4"/>
@@
 <contactref element="LED2" pad="C"/>
 <contactref element="R9" pad="1"/>
-<wire x1="138.684" y1="37.857" x2="138.684" y2="39.717" width="0.2032" layer="1"/>
+<wire x1="140.081" y1="37.857" x2="140.081" y2="39.717" width="0.2032" layer="1"/>
 </signal>
 <signal name="N$25">
@@
 <via x="136.906" y="36.957" extent="1-16" drill="0.5"/>
 <wire x1="136.906" y1="36.957" x2="137.806" y2="36.057" width="0.2032" layer="1"/>
-<wire x1="137.806" y1="36.057" x2="138.684" y2="36.057" width="0.2032" layer="1"/>
+<wire x1="137.806" y1="36.057" x2="140.081" y2="36.057" width="0.2032" layer="1"/>
 <wire x1="50.546" y1="36.957" x2="136.906" y2="36.957" width="0.2032" layer="16"/>
 </signal>

Commit message: ready to fab
Parts:
- moved C4 7.01 mm to (39.4, 47.1), turned to 0 degrees
- moved C9 6.92 mm to (83.8, 47.1), turned to 0 degrees
- moved C5 6.82 mm to (63.6, 47.1), turned to 0 degrees
- moved C10 6.74 mm to (107.8, 47.0), turned to 0 degrees
- moved C13 6.74 mm to (128.1, 47.0), turned to 0 degrees
- moved C2 6.74 mm to (19.4, 47.1), turned to 0 degrees
Routing:
- net +3V3: track 93.8 -> 78.4 mm, vias 12 -> 18
Changed lines of the file:
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@@
 <layer number="49" name="Reference" color="7" fill="1" visible="no" active="yes"/>
 <layer number="50" name="dxf" color="7" fill="1" visible="no" active="no"/>
-<layer number="51" name="tDocu" color="7" fill="1" visible="yes" active="yes"/>
-<layer number="52" name="bDocu" color="7" fill="1" visible="yes" active="yes"/>
+<layer number="51" name="tDocu" color="7" fill="1" visible="no" active="yes"/>
+<layer number="52" name="bDocu" color="7" fill="1" visible="no" active="yes"/>
 <layer number="53" name="tGND_GNDA" color="7" fill="1" visible="no" active="no"/>
 <layer number="54" name="bGND_GNDA" color="7" fill="1" visible="no" active="no"/>
@@
 <rectangle x1="97.663" y1="45.212" x2="100.203" y2="49.276" layer="41"/>
 <rectangle x1="117.856" y1="45.085" x2="120.396" y2="49.149" layer="41"/>
-<rectangle x1="74.2188" y1="31.2928" x2="75.4888" y2="42.9768" layer="41"/>
 <rectangle x1="73.025" y1="44.704" x2="76.708" y2="50.038" layer="42"/>
 <text x="15.367" y="1.143" size="1.27" layer="25">TX</text>
@@
 <text x="48.895" y="21.59" size="1.016" layer="26" rot="MR0">PA8</text>
 <text x="55.118" y="25.019" size="1.016" layer="26" rot="MR0">PA10</text>
+<rectangle x1="74.041" y1="31.623" x2="75.692" y2="45.212" layer="41"/>
 </plain>
 <attributes>
@@
 <attribute name="NAME" x="49.2125" y="38.1" size="0.8128" layer="25" rot="R90"/>
 </element>
-<element name="C2" library="clock" package="C1210" value="" x="24.13" y="42.291" smashed="yes" rot="R180">
-<attribute name="NAME" x="24.765" y="40.386" size="0.8128" layer="25" rot="R180"/>
+<element name="C2" library="clock" package="C1210" value="" x="19.431" y="47.117" smashed="yes">
+<attribute name="NAME" x="18.796" y="49.022" size="0.8128" layer="25"/>
 </element>
 <element name="C6" library="clock" package="0805" value="" x="44.577" y="22.86" smashed="yes" rot="R225">
@@
 <element name="JP1" library="nixie_power" package="EBAY_PKG" value="" x="72.644" y="25.4" smashed="yes" rot="MR180"/>
 <element name="JP2" library="nixie_power" package="TAOBAO_PKG" value="" x="72.644" y="20.574" smashed="yes" rot="MR180"/>
-<element name="C4" library="clock" package="C1210" value="" x="44.45" y="42.291" smashed="yes" rot="R180">
-<attribute name="NAME" x="45.085" y="40.64" size="0.8128" layer="25" rot="R180"/>
-</element>
-<element name="C5" library="clock" package="C1210" value="" x="68.453" y="42.291" smashed="yes" rot="R180">
-<attribute name="NAME" x="69.215" y="40.386" size="0.8128" layer="25" rot="R180"/>
-</element>
-<element name="C9" library="clock" package="C1210" value="" x="88.773" y="42.291" smashed="yes" rot="R180">
-<attribute name="NAME" x="89.789" y="40.513" size="0.8128" layer="25" rot="R180"/>
-</element>
-<element name="C10" library="clock" package="C1210" value="" x="112.649" y="42.291" smashed="yes" rot="R180">
-<attribute name="NAME" x="113.919" y="40.386" size="0.8128" layer="25" rot="R180"/>
-</element>
-<element name="C13" library="clock" package="C1210" value="" x="132.969" y="42.291" smashed="yes" rot="R180">
-<attribute name="NAME" x="134.366" y="40.386" size="0.8128" layer="25" rot="R180"/>
+<element name="C4" library="clock" package="C1210" value="" x="39.37" y="47.117" smashed="yes">
+<attribute name="NAME" x="38.735" y="48.768" size="0.8128" layer="25"/>
+</element>
+<element name="C5" library="clock" package="C1210" value="" x="63.627" y="47.117" smashed="yes">
+<attribute name="NAME" x="62.865" y="49.022" size="0.8128" layer="25"/>
+</element>
+<element name="C9" library="clock" package="C1210" value="" x="83.82" y="47.117" smashed="yes">
+<attribute name="NAME" x="82.804" y="48.895" size="0.8128" layer="25"/>
+</element>
+<element name="C10" library="clock" package="C1210" value="" x="107.823" y="46.99" smashed="yes">
+<attribute name="NAME" x="106.553" y="48.895" size="0.8128" layer="25"/>
+</element>
+<element name="C13" library="clock" package="C1210" value="" x="128.143" y="46.99" smashed="yes">
+<attribute name="NAME" x="126.746" y="48.895" size="0.8128" layer="25"/>
 </element>
 <element name="S1" library="SparkFun-Retired" package="TACTILE-SWITCH-SMD" value="TAC_SWITCHSMD" x="69.596" y="5.08" smashed="yes">
@@
 <vertex x="145" y="50"/>
 </polygon>
-<wire x1="25.52" y1="47.2" x2="25.52" y2="42.301" width="0.4064" layer="1"/>
-<wire x1="25.52" y1="42.301" x2="25.53" y2="42.291" width="0.4064" layer="1"/>
-<wire x1="45.82" y1="42.321" x2="45.82" y2="47.2" width="0.4064" layer="1"/>
-<wire x1="45.82" y1="42.321" x2="45.85" y2="42.291" width="0.4064" layer="1"/>
-<wire x1="69.82" y1="42.324" x2="69.82" y2="47.2" width="0.4064" layer="1"/>
-<wire x1="69.82" y1="42.324" x2="69.853" y2="42.291" width="0.4064" layer="1"/>
-<wire x1="90.12" y1="47.2" x2="90.12" y2="42.344" width="0.4064" layer="1"/>
-<wire x1="90.12" y1="42.344" x2="90.173" y2="42.291" width="0.4064" layer="1"/>
-<wire x1="114.12" y1="47.2" x2="114.12" y2="42.362" width="0.4064" layer="1"/>
-<wire x1="114.12" y1="42.362" x2="114.049" y2="42.291" width="0.4064" layer="1"/>
-<wire x1="134.42" y1="47.2" x2="134.42" y2="42.342" width="0.4064" layer="1"/>
-<wire x1="134.369" y1="42.291" x2="134.42" y2="42.342" width="0.4064" layer="1"/>
 <contactref element="U$8" pad="COLLECTOR"/>
 <via x="27.94" y="4.572" extent="1-16" drill="0.6"/>
@@
 <wire x1="134.9502" y1="1.8796" x2="136.7704" y2="1.8796" width="0.2032" layer="1"/>
 <wire x1="136.7704" y1="1.8796" x2="136.779" y2="1.871" width="0.2032" layer="1"/>
-<wire x1="140.081" y1="41.817" x2="134.843" y2="41.817" width="0.2032" layer="1"/>
-<wire x1="134.843" y1="41.817" x2="134.369" y2="42.291" width="0.2032" layer="1"/>
 <contactref element="SD1" pad="4"/>
 <via x="131.3434" y="24.0792" extent="1-16" drill="0.5"/>
@@
 <wire x1="62.3062" y1="31.9278" x2="62.3062" y2="30.4858" width="0.2032" layer="1"/>
 <wire x1="62.3062" y1="30.4858" x2="62.316" y2="30.476" width="0.2032" layer="1"/>
+<via x="15.9512" y="47.0916" extent="1-16" drill="0.5"/>
+<via x="36.0172" y="47.0916" extent="1-16" drill="0.5"/>
+<via x="60.2742" y="47.0916" extent="1-16" drill="0.5"/>
+<via x="80.4672" y="47.0916" extent="1-16" drill="0.5"/>
+<via x="104.2162" y="46.9646" extent="1-16" drill="0.5"/>
+<via x="124.7902" y="46.9646" extent="1-16" drill="0.5"/>
+<wire x1="15.9512" y1="47.0916" x2="18.0056" y2="47.0916" width="0.4064" layer="1"/>
+<wire x1="18.0056" y1="47.0916" x2="18.031" y2="47.117" width="0.4064" layer="1"/>
+<wire x1="36.0172" y1="47.0916" x2="37.9446" y2="47.0916" width="0.4064" layer="1"/>
+<wire x1="37.9446" y1="47.0916" x2="37.97" y2="47.117" width="0.4064" layer="1"/>
+<wire x1="60.2742" y1="47.0916" x2="62.2016" y2="47.0916" width="0.4064" layer="1"/>
+<wire x1="62.2016" y1="47.0916" x2="62.227" y2="47.117" width="0.4064" layer="1"/>
+<wire x1="80.4672" y1="47.0916" x2="82.3946" y2="47.0916" width="0.4064" layer="1"/>
+<wire x1="82.3946" y1="47.0916" x2="82.42" y2="47.117" width="0.4064" layer="1"/>
+<wire x1="104.2162" y1="46.9646" x2="106.3976" y2="46.9646" width="0.4064" layer="1"/>
+<wire x1="106.3976" y1="46.9646" x2="106.423" y2="46.99" width="0.4064" layer="1"/>
+<wire x1="124.7902" y1="46.9646" x2="126.7176" y2="46.9646" width="0.4064" layer="1"/>
+<wire x1="126.7176" y1="46.9646" x2="126.743" y2="46.99" width="0.4064" layer="1"/>
+<wire x1="134.42" y1="47.2" x2="134.698" y2="47.2" width="0.2032" layer="1"/>
+<wire x1="134.698" y1="47.2" x2="140.081" y2="41.817" width="0.2032" layer="1"/>
 </signal>
 <signal name="N$27">
