File: pcb/clock.sch (EAGLE design)
At the start: 27 parts, among them IC1 STM32F10XCXT6, IC3 24C64ST

Commit message: rough layout
Parts:
- IC1: value STM32F10XCXT6 -> STM32F072C8T6; device stm32f072c8t6:STM32F10XCXT6 -> joyAnalog:STM32F072C8T6
Connections:
- new net N$1: C11.1, IC1PORTC.PC14, Y2.2
- new net N$2: C12.1, IC1PORTC.PC15, Y2.1
- new net N$3: IC1RESET.NRST, R8.1, S2.1, S2.2
- new net N$5: IC1RESET.BOOT0, R1.2
- new net N$6: C1.1, IC1PORTF/OSC.PF0/OSC<=, Y1.2
- new net N$7: C3.1, IC1PORTF/OSC.PF1/OSC=>, Y1.1
- net +3V3: now also U$1.VCC, U$2.VCC, U$3.VCC, U$4.VCC, U$5.VCC, U$6.VCC
- net GND: now also C11.2, C12.2, S2.3, S2.4, U$1.GND, U$2.GND, U$3.GND, U$4.GND, U$5.GND, U$6.GND
Other:
- moved on the sheet: S2
Changed lines of the file:
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@@
 <?xml version="1.0" encoding="utf-8"?>
 <!DOCTYPE eagle SYSTEM "eagle.dtd">
-<eagle version="7.7.0">
+<eagle version="8.1.1">
 <drawing>
 <settings>
@@
 <part name="+3V16" library="backplane" deviceset="+3V3" device=""/>
 <part name="R9" library="SparkFun-Passives" deviceset="RESISTOR" device="0805-RES"/>
-<part name="IC1" library="stm32f072c8t6" deviceset="STM32F10XCXT6" device=""/>
+<part name="IC1" library="joyAnalog" deviceset="STM32F072C8T6" device=""/>
 <part name="GND1" library="backplane" deviceset="GND" device=""/>
 <part name="R1" library="SparkFun-Passives" deviceset="RESISTOR" device="0805-RES"/>
@@
 <part name="U$5" library="exixe_module" deviceset="EXIXE" device=""/>
 <part name="U$6" library="exixe_module" deviceset="EXIXE" device=""/>
+<part name="GND4" library="backplane" deviceset="GND" device=""/>
+<part name="GND5" library="backplane" deviceset="GND" device=""/>
+<part name="GND6" library="backplane" deviceset="GND" device=""/>
+<part name="GND9" library="backplane" deviceset="GND" device=""/>
+<part name="GND15" library="backplane" deviceset="GND" device=""/>
+<part name="GND16" library="backplane" deviceset="GND" device=""/>
+<part name="+3V2" library="backplane" deviceset="+3V3" device=""/>
+<part name="+3V7" library="backplane" deviceset="+3V3" device=""/>
+<part name="+3V8" library="backplane" deviceset="+3V3" device=""/>
+<part name="+3V10" library="backplane" deviceset="+3V3" device=""/>
+<part name="+3V12" library="backplane" deviceset="+3V3" device=""/>
+<part name="+3V13" library="backplane" deviceset="+3V3" device=""/>
 </parts>
 <sheets>
@@
 <instance part="+3V6" gate="G$1" x="-58.42" y="7.62"/>
 <instance part="+3V9" gate="G$1" x="-45.72" y="-58.42" rot="MR0"/>
-<instance part="S2" gate="S" x="53.34" y="-76.2"/>
-<instance part="U$3" gate="G$1" x="30.48" y="-198.12"/>
-<instance part="U$1" gate="G$1" x="68.58" y="-198.12"/>
+<instance part="S2" gate="S" x="162.56" y="-104.14"/>
+<instance part="U$3" gate="G$1" x="12.7" y="-198.12"/>
+<instance part="U$1" gate="G$1" x="53.34" y="-198.12"/>
 <instance part="U$2" gate="G$1" x="104.14" y="-198.12"/>
-<instance part="U$4" gate="G$1" x="137.16" y="-198.12"/>
-<instance part="U$5" gate="G$1" x="175.26" y="-198.12"/>
-<instance part="U$6" gate="G$1" x="223.52" y="-198.12"/>
+<instance part="U$4" gate="G$1" x="142.24" y="-198.12"/>
+<instance part="U$5" gate="G$1" x="200.66" y="-198.12"/>
+<instance part="U$6" gate="G$1" x="238.76" y="-198.12"/>
+<instance part="GND4" gate="1" x="-2.54" y="-203.2"/>
+<instance part="GND5" gate="1" x="38.1" y="-203.2"/>
+<instance part="GND6" gate="1" x="88.9" y="-203.2"/>
+<instance part="GND9" gate="1" x="127" y="-203.2"/>
+<instance part="GND15" gate="1" x="185.42" y="-203.2"/>
+<instance part="GND16" gate="1" x="223.52" y="-203.2"/>
+<instance part="+3V2" gate="G$1" x="10.16" y="-175.26" rot="MR0"/>
+<instance part="+3V7" gate="G$1" x="50.8" y="-175.26" rot="MR0"/>
+<instance part="+3V8" gate="G$1" x="101.6" y="-175.26" rot="MR0"/>
+<instance part="+3V10" gate="G$1" x="139.7" y="-175.26" rot="MR0"/>
+<instance part="+3V12" gate="G$1" x="198.12" y="-175.26" rot="MR0"/>
+<instance part="+3V13" gate="G$1" x="236.22" y="-175.26" rot="MR0"/>
 </instances>
 <busses>
@@
 <pinref part="GND12" gate="1" pin="GND"/>
 </segment>
+<segment>
+<pinref part="U$3" gate="G$1" pin="GND"/>
+<pinref part="GND4" gate="1" pin="GND"/>
+</segment>
+<segment>
+<pinref part="U$1" gate="G$1" pin="GND"/>
+<pinref part="GND5" gate="1" pin="GND"/>
+</segment>
+<segment>
+<pinref part="U$2" gate="G$1" pin="GND"/>
+<pinref part="GND6" gate="1" pin="GND"/>
+</segment>
+<segment>
+<pinref part="U$4" gate="G$1" pin="GND"/>
+<pinref part="GND9" gate="1" pin="GND"/>
+</segment>
+<segment>
+<pinref part="U$5" gate="G$1" pin="GND"/>
+<pinref part="GND15" gate="1" pin="GND"/>
+</segment>
+<segment>
+<pinref part="U$6" gate="G$1" pin="GND"/>
+<pinref part="GND16" gate="1" pin="GND"/>
+</segment>
+<segment>
+<pinref part="C11" gate="G$1" pin="2"/>
+<pinref part="GND19" gate="1" pin="GND"/>
+<wire x1="-86.36" y1="-142.24" x2="-86.36" y2="-149.86" width="0.1524" layer="91"/>
+<pinref part="C12" gate="G$1" pin="2"/>
+<wire x1="-86.36" y1="-149.86" x2="-73.66" y2="-149.86" width="0.1524" layer="91"/>
+<wire x1="-73.66" y1="-149.86" x2="-73.66" y2="-147.32" width="0.1524" layer="91"/>
+<junction x="-86.36" y="-149.86"/>
+</segment>
+<segment>
+<pinref part="S2" gate="S" pin="3"/>
+<pinref part="S2" gate="S" pin="4"/>
+<wire x1="167.64" y1="-104.14" x2="167.64" y2="-106.68" width="0.1524" layer="91"/>
+<pinref part="GND2" gate="1" pin="GND"/>
+<wire x1="167.64" y1="-106.68" x2="172.72" y2="-106.68" width="0.1524" layer="91"/>
+<junction x="167.64" y="-106.68"/>
+</segment>
 </net>
 <net name="+3V3" class="0">
@@
 <pinref part="+3V6" gate="G$1" pin="+3V3"/>
 </segment>
+<segment>
+<pinref part="U$3" gate="G$1" pin="VCC"/>
+<pinref part="+3V2" gate="G$1" pin="+3V3"/>
+</segment>
+<segment>
+<pinref part="U$1" gate="G$1" pin="VCC"/>
+<pinref part="+3V7" gate="G$1" pin="+3V3"/>
+</segment>
+<segment>
+<pinref part="U$2" gate="G$1" pin="VCC"/>
+<pinref part="+3V8" gate="G$1" pin="+3V3"/>
+</segment>
+<segment>
+<pinref part="U$4" gate="G$1" pin="VCC"/>
+<pinref part="+3V10" gate="G$1" pin="+3V3"/>
+</segment>
+<segment>
+<pinref part="U$5" gate="G$1" pin="VCC"/>
+<pinref part="+3V12" gate="G$1" pin="+3V3"/>
+</segment>
+<segment>
+<pinref part="U$6" gate="G$1" pin="VCC"/>
+<pinref part="+3V13" gate="G$1" pin="+3V3"/>
+</segment>
 </net>
 <net name="N$27" class="0">
@@
 </segment>
 </net>
+<net name="N$1" class="0">
+<segment>
+<pinref part="Y2" gate="G$1" pin="2"/>
+<pinref part="IC1" gate="PORTC" pin="PC14"/>
+<wire x1="-63.5" y1="-134.62" x2="-53.34" y2="-134.62" width="0.1524" layer="91"/>
+<pinref part="C11" gate="G$1" pin="1"/>
+<wire x1="-86.36" y1="-134.62" x2="-63.5" y2="-134.62" width="0.1524" layer="91"/>
+<junction x="-63.5" y="-134.62"/>
+</segment>
+</net>
+<net name="N$2" class="0">
+<segment>
+<pinref part="IC1" gate="PORTC" pin="PC15"/>
+<wire x1="-53.34" y1="-137.16" x2="-53.34" y2="-139.7" width="0.1524" layer="91"/>
+<pinref part="Y2" gate="G$1" pin="1"/>
+<wire x1="-53.34" y1="-139.7" x2="-63.5" y2="-139.7" width="0.1524" layer="91"/>
+<pinref part="C12" gate="G$1" pin="1"/>
+<wire x1="-63.5" y1="-139.7" x2="-73.66" y2="-139.7" width="0.1524" layer="91"/>
+<junction x="-63.5" y="-139.7"/>
+</segment>
+</net>
+<net name="N$3" class="0">
+<segment>
+<pinref part="IC1" gate="RESET" pin="NRST"/>
+<pinref part="R8" gate="G$1" pin="1"/>
+<wire x1="147.32" y1="-106.68" x2="154.94" y2="-106.68" width="0.1524" layer="91"/>
+<pinref part="S2" gate="S" pin="2"/>
+<wire x1="154.94" y1="-106.68" x2="157.48" y2="-106.68" width="0.1524" layer="91"/>
+<junction x="154.94" y="-106.68"/>
+<pinref part="S2" gate="S" pin="1"/>
+<wire x1="157.48" y1="-106.68" x2="157.48" y2="-104.14" width="0.1524" layer="91"/>
+<junction x="157.48" y="-106.68"/>
+</segment>
+</net>
+<net name="N$5" class="0">
+<segment>
+<pinref part="IC1" gate="RESET" pin="BOOT0"/>
+<pinref part="R1" gate="G$1" pin="2"/>
+<wire x1="147.32" y1="-111.76" x2="152.4" y2="-111.76" width="0.1524" layer="91"/>
+<wire x1="152.4" y1="-111.76" x2="152.4" y2="-114.3" width="0.1524" layer="91"/>
+</segment>
+</net>
+<net name="N$6" class="0">
+<segment>
+<pinref part="IC1" gate="PORTF/OSC" pin="PF0/OSC&lt;="/>
+<pinref part="Y1" gate="G$1" pin="2"/>
+<wire x1="147.32" y1="-78.74" x2="165.1" y2="-78.74" width="0.1524" layer="91"/>
+<pinref part="C1" gate="G$1" pin="1"/>
+<wire x1="165.1" y1="-78.74" x2="190.5" y2="-78.74" width="0.1524" layer="91"/>
+<junction x="165.1" y="-78.74"/>
+</segment>
+</net>
+<net name="N$7" class="0">
+<segment>
+<pinref part="IC1" gate="PORTF/OSC" pin="PF1/OSC=&gt;"/>
+<wire x1="147.32" y1="-81.28" x2="157.48" y2="-81.28" width="0.1524" layer="91"/>
+<wire x1="157.48" y1="-81.28" x2="157.48" y2="-83.82" width="0.1524" layer="91"/>
+<pinref part="Y1" gate="G$1" pin="1"/>
+<wire x1="157.48" y1="-83.82" x2="165.1" y2="-83.82" width="0.1524" layer="91"/>
+<pinref part="C3" gate="G$1" pin="1"/>
+<wire x1="165.1" y1="-83.82" x2="172.72" y2="-83.82" width="0.1524" layer="91"/>
+<junction x="165.1" y="-83.82"/>
+</segment>
+</net>

Commit message: USBC, GPS etc
Parts:
- added CONN1: USB-C_WURTH_632723X00011USB-C, breakouts:USB-C_WURTH_632723X00011USB-C
- added SD1: TF-HOLDER, basicBoard:TF-HOLDER
- added U$7: MAX-M8, ubloxLib:MAX-M8
- added U$8: TEMT6000, ProtoSnap-v14a:TEMT6000
- added U$9: DS18B20, DS18B20U:DS18B20
- added X1: (no value), clock:SMACONNECTOR
Connections:
- new net N$4: U$7.11_RF_IN, X1.ANT
- net GND: now also CONN1.GND0, CONN1.GND1, CONN1.GND3, CONN1.GND4, CONN1.SHIELD1, CONN1.SHIELD2, CONN1.SHIELD3, CONN1.SHIELD4, CONN1.SHIELD5, CONN1.SHIELD6, U$7.10_GND, U$7.12_GND, X1.GND1, X1.GND2, X1.GND3, X1.GND4

Commit message: added bake control
Parts:
- removed Y1: (no value), backplane:CRYSTALHC49US
- removed Y2: (no value), backplane:CRYSTALTC26H_EZ
- added Q1: (no value), adafruit:XTAL-4-3225
- added X2: (no value), adafruit:XTAL-3.2X1.5
Connections:
- net GND: now also Q1.G1, Q1.G2
- net N$1: now also Q1.X1; no longer Y2.2
- net N$2: now also Q1.X2; no longer Y2.1
- net N$6: now also C3.1, IC1PORTF/OSC.PF1/OSC=>, X2.P$2; no longer C1.1, IC1PORTF/OSC.PF0/OSC<=, Y1.2
- net N$7: now also C1.1, IC1PORTF/OSC.PF0/OSC<=, X2.P$1; no longer C3.1, IC1PORTF/OSC.PF1/OSC=>, Y1.1
Other:
- moved on the sheet: C11, C12, IC1PORTC
Changed lines of the file:
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@@
 <part name="C1" library="backplane" deviceset="CAP" device="0805"/>
 <part name="C2" library="backplane" deviceset="C-US" device="C1210"/>
-<part name="Y1" library="backplane" deviceset="CRYSTAL" device="HC49US"/>
 <part name="GND2" library="backplane" deviceset="GND" device=""/>
 <part name="GND3" library="backplane" deviceset="GND" device=""/>
@@
 <part name="+3V14" library="backplane" deviceset="+3V3" device=""/>
 <part name="GND18" library="backplane" deviceset="GND" device=""/>
-<part name="Y2" library="backplane" deviceset="CRYSTAL" device="TC26H_EZ"/>
 <part name="C11" library="backplane" deviceset="CAP" device="0805"/>
 <part name="C12" library="backplane" deviceset="CAP" device="0805"/>
@@
 <part name="GND25" library="backplane" deviceset="GND" device=""/>
 <part name="SD1" library="basicBoard" deviceset="TF-HOLDER" device=""/>
+<part name="Q1" library="adafruit" deviceset="XTAL-4" device="-3225"/>
+<part name="X2" library="adafruit" deviceset="XTAL" device="-3.2X1.5"/>
+<part name="GND26" library="backplane" deviceset="GND" device=""/>
+<part name="GND27" library="backplane" deviceset="GND" device=""/>
+<part name="GND28" library="backplane" deviceset="GND" device=""/>
 </parts>
 <sheets>
@@
 <instance part="C1" gate="G$1" x="190.5" y="-83.82"/>
 <instance part="C2" gate="G$1" x="182.88" y="-43.18"/>
-<instance part="Y1" gate="G$1" x="165.1" y="-81.28" rot="R90"/>
 <instance part="GND2" gate="1" x="172.72" y="-109.22"/>
 <instance part="GND3" gate="1" x="-93.98" y="111.76"/>
@@
 <instance part="+3V14" gate="G$1" x="-223.52" y="58.42"/>
 <instance part="GND18" gate="1" x="-223.52" y="35.56"/>
-<instance part="Y2" gate="G$1" x="-63.5" y="-137.16" rot="R90"/>
-<instance part="C11" gate="G$1" x="-86.36" y="-139.7"/>
-<instance part="C12" gate="G$1" x="-73.66" y="-144.78"/>
-<instance part="GND19" gate="1" x="-86.36" y="-152.4"/>
+<instance part="C11" gate="G$1" x="-40.64" y="-149.86"/>
+<instance part="C12" gate="G$1" x="-45.72" y="-149.86" rot="MR0"/>
+<instance part="GND19" gate="1" x="-60.96" y="-147.32"/>
 <instance part="R8" gate="G$1" x="154.94" y="-101.6" rot="R90"/>
 <instance part="+3V15" gate="G$1" x="154.94" y="-93.98"/>
@@
 <instance part="IC1" gate="PORTB_H" x="-76.2" y="-43.18" rot="R270"/>
 <instance part="IC1" gate="POWER" x="-76.2" y="137.16"/>
-<instance part="IC1" gate="PORTC" x="-45.72" y="-134.62"/>
+<instance part="IC1" gate="PORTC" x="-30.48" y="-134.62"/>
 <instance part="IC1" gate="PORTF/OSC" x="139.7" y="-78.74"/>
 <instance part="IC1" gate="AN_POWER" x="-91.44" y="-106.68"/>
@@
 <instance part="GND25" gate="1" x="426.72" y="-170.18"/>
 <instance part="SD1" gate="G$1" x="391.16" y="-205.74"/>
+<instance part="Q1" gate="G$1" x="-53.34" y="-139.7" rot="R270"/>
+<instance part="X2" gate="G$1" x="162.56" y="-78.74" rot="R270"/>
+<instance part="GND26" gate="1" x="-45.72" y="-154.94"/>
+<instance part="GND27" gate="1" x="-40.64" y="-154.94"/>
+<instance part="GND28" gate="1" x="-60.96" y="-132.08" rot="R180"/>
 </instances>
 <busses>
@@
 <pinref part="U$6" gate="G$1" pin="GND"/>
 <pinref part="GND16" gate="1" pin="GND"/>
-</segment>
-<segment>
-<pinref part="C11" gate="G$1" pin="2"/>
-<pinref part="GND19" gate="1" pin="GND"/>
-<wire x1="-86.36" y1="-142.24" x2="-86.36" y2="-149.86" width="0.1524" layer="91"/>
-<pinref part="C12" gate="G$1" pin="2"/>
-<wire x1="-86.36" y1="-149.86" x2="-73.66" y2="-149.86" width="0.1524" layer="91"/>
-<wire x1="-73.66" y1="-149.86" x2="-73.66" y2="-147.32" width="0.1524" layer="91"/>
-<junction x="-86.36" y="-149.86"/>
 </segment>
 <segment>
@@
 <junction x="426.72" y="-167.64"/>
 </segment>
+<segment>
+<pinref part="C12" gate="G$1" pin="2"/>
+<pinref part="GND26" gate="1" pin="GND"/>
+</segment>
+<segment>
+<pinref part="C11" gate="G$1" pin="2"/>
+<pinref part="GND27" gate="1" pin="GND"/>
+</segment>
+<segment>
+<pinref part="Q1" gate="G$1" pin="G2"/>
+<pinref part="GND19" gate="1" pin="GND"/>
+</segment>
+<segment>
+<pinref part="Q1" gate="G$1" pin="G1"/>
+<pinref part="GND28" gate="1" pin="GND"/>
+</segment>
 </net>
 <net name="+3V3" class="0">
@@
 </segment>
 </net>
-<net name="N$1" class="0">
-<segment>
-<pinref part="Y2" gate="G$1" pin="2"/>
-<pinref part="IC1" gate="PORTC" pin="PC14"/>
-<wire x1="-63.5" y1="-134.62" x2="-53.34" y2="-134.62" width="0.1524" layer="91"/>
-<pinref part="C11" gate="G$1" pin="1"/>
-<wire x1="-86.36" y1="-134.62" x2="-63.5" y2="-134.62" width="0.1524" layer="91"/>
-<junction x="-63.5" y="-134.62"/>
-</segment>
-</net>
-<net name="N$2" class="0">
-<segment>
-<pinref part="IC1" gate="PORTC" pin="PC15"/>
-<wire x1="-53.34" y1="-137.16" x2="-53.34" y2="-139.7" width="0.1524" layer="91"/>
-<pinref part="Y2" gate="G$1" pin="1"/>
-<wire x1="-53.34" y1="-139.7" x2="-63.5" y2="-139.7" width="0.1524" layer="91"/>
-<pinref part="C12" gate="G$1" pin="1"/>
-<wire x1="-63.5" y1="-139.7" x2="-73.66" y2="-139.7" width="0.1524" layer="91"/>
-<junction x="-63.5" y="-139.7"/>
-</segment>
-</net>
 <net name="N$3" class="0">
 <segment>
@@
 </segment>
 </net>
-<net name="N$6" class="0">
-<segment>
-<pinref part="IC1" gate="PORTF/OSC" pin="PF0/OSC&lt;="/>
-<pinref part="Y1" gate="G$1" pin="2"/>
-<wire x1="147.32" y1="-78.74" x2="165.1" y2="-78.74" width="0.1524" layer="91"/>
-<pinref part="C1" gate="G$1" pin="1"/>
-<wire x1="165.1" y1="-78.74" x2="190.5" y2="-78.74" width="0.1524" layer="91"/>
-<junction x="165.1" y="-78.74"/>
-</segment>
-</net>
-<net name="N$7" class="0">
-<segment>
-<pinref part="IC1" gate="PORTF/OSC" pin="PF1/OSC=&gt;"/>
-<wire x1="147.32" y1="-81.28" x2="157.48" y2="-81.28" width="0.1524" layer="91"/>
-<wire x1="157.48" y1="-81.28" x2="157.48" y2="-83.82" width="0.1524" layer="91"/>
-<pinref part="Y1" gate="G$1" pin="1"/>
-<wire x1="157.48" y1="-83.82" x2="165.1" y2="-83.82" width="0.1524" layer="91"/>
-<pinref part="C3" gate="G$1" pin="1"/>
-<wire x1="165.1" y1="-83.82" x2="172.72" y2="-83.82" width="0.1524" layer="91"/>
-<junction x="165.1" y="-83.82"/>
-</segment>
-</net>
 <net name="N$4" class="0">
 <segment>
@@
 </segment>
 </net>
+<net name="N$6" class="0">
+<segment>
+<pinref part="IC1" gate="PORTF/OSC" pin="PF1/OSC=&gt;"/>
+<pinref part="X2" gate="G$1" pin="P$2"/>
+<wire x1="147.32" y1="-81.28" x2="147.32" y2="-83.82" width="0.1524" layer="91"/>
+<wire x1="147.32" y1="-83.82" x2="162.56" y2="-83.82" width="0.1524" layer="91"/>
+<pinref part="C3" gate="G$1" pin="1"/>
+<wire x1="162.56" y1="-83.82" x2="172.72" y2="-83.82" width="0.1524" layer="91"/>
+<junction x="162.56" y="-83.82"/>
+</segment>
+</net>
+<net name="N$7" class="0">
+<segment>
+<pinref part="IC1" gate="PORTF/OSC" pin="PF0/OSC&lt;="/>
+<pinref part="X2" gate="G$1" pin="P$1"/>
+<wire x1="147.32" y1="-78.74" x2="147.32" y2="-73.66" width="0.1524" layer="91"/>
+<wire x1="147.32" y1="-73.66" x2="162.56" y2="-73.66" width="0.1524" layer="91"/>
+<pinref part="C1" gate="G$1" pin="1"/>
+<wire x1="162.56" y1="-73.66" x2="190.5" y2="-73.66" width="0.1524" layer="91"/>
+<wire x1="190.5" y1="-73.66" x2="190.5" y2="-78.74" width="0.1524" layer="91"/>
+<junction x="162.56" y="-73.66"/>
+</segment>
+</net>
+<net name="N$1" class="0">
+<segment>
+<pinref part="IC1" gate="PORTC" pin="PC14"/>
+<pinref part="Q1" gate="G$1" pin="X1"/>
+<wire x1="-38.1" y1="-134.62" x2="-40.64" y2="-134.62" width="0.1524" layer="91"/>
+<pinref part="C11" gate="G$1" pin="1"/>
+<wire x1="-40.64" y1="-134.62" x2="-53.34" y2="-134.62" width="0.1524" layer="91"/>
+<wire x1="-40.64" y1="-144.78" x2="-40.64" y2="-134.62" width="0.1524" layer="91"/>
+<junction x="-40.64" y="-134.62"/>
+</segment>
+</net>
+<net name="N$2" class="0">
+<segment>
+<pinref part="IC1" gate="PORTC" pin="PC15"/>
+<wire x1="-38.1" y1="-137.16" x2="-45.72" y2="-137.16" width="0.1524" layer="91"/>
+<wire x1="-45.72" y1="-137.16" x2="-45.72" y2="-144.78" width="0.1524" layer="91"/>
+<pinref part="Q1" gate="G$1" pin="X2"/>
+<wire x1="-45.72" y1="-144.78" x2="-53.34" y2="-144.78" width="0.1524" layer="91"/>
+<pinref part="C12" gate="G$1" pin="1"/>
+<junction x="-45.72" y="-144.78"/>
+</segment>
+</net>

Commit message: positioned boards
Parts:
- removed SD1: TF-HOLDER, basicBoard:TF-HOLDER
- added U$10, U$11, U$12, U$13: M3_MOUNTING_HOLE, a:M3_MOUNTING_HOLE
Connections:
- net +3V3: now also U$1.3V, U$2.3V, U$3.3V, U$4.3V, U$5.3V, U$6.3V; no longer U$1.VCC, U$2.VCC, U$3.VCC, U$4.VCC, U$5.VCC, U$6.VCC

Commit message: added touch
Parts:
- added C10, C13, C14, C15, C16, C17, C4, C5, C9: (no value), clock:C-USC1210
- added C18, C19: (no value), clock:CAP0805
- added IC2: REG1117, clock:REG1117
- added JP1: (no value), nixie_power:EBAY_MODULEEBAY
- added JP2: (no value), nixie_power:EBAY_MODULETAOBAO
- added JP3: (no value), pinhead:PINHD-2X2
- added JP4: (no value), pinhead:PINHD-2X3
- added R10, R11, R12, R13, R4, R5, R6: (no value), clock:RESISTOR0805-RES
- added S1: TAC_SWITCHSMD, SparkFun-Retired:TAC_SWITCHSMD
- added U$14, U$15, U$16: TOUCHPAD, touch_pad:TOUCHPAD
- C1, C11, C12, C3, C6, C7, C8: device backplane:CAP0805 -> clock:CAP0805
- C2: device backplane:C-USC1210 -> clock:C-USC1210
- R1, R2, R3, R7, R8, R9: device SparkFun-Passives:RESISTOR0805-RES -> clock:RESISTOR0805-RES
Connections:
- new net +180V: JP1.HV, JP2.HV, U$1.HV, U$2.HV, U$3.HV, U$4.HV, U$5.HV, U$6.HV
- new net +5V: C14.1, CONN1.VBUS1, CONN1.VBUS2, CONN1.VBUS3, CONN1.VBUS4, IC2.VIN, JP1.5V, JP2.5V
- new net I2C_SCL: IC1PORTB_H.PB8, IC3.SCL, R2.1
- new net I2C_SDA: IC1PORTB_H.PB9, IC3.SDA, R3.1
- new net LIGHT_SENSOR_OUTPUT: R13.2, U$8.E1
- new net N$10: R6.2, U$16.PAD
- new net N$11: IC1PORTA_L.PA3, R12.1
- new net N$12: CONN1.CC2, R4.2
- new net N$13: CONN1.CC1, R5.2
- new net N$14: R11.2, U$14.PAD
- new net N$15: IC1PORTA_L.PA5, R10.1
- new net N$16: IC1PORTA_L.PA6, R6.1
- new net N$18: C19.1, IC1PORTA_L.PA2
- new net N$8: IC1PORTA_L.PA4, R11.1
- new net N$9: R10.2, U$15.PAD
- new net NIXIE_PWR_EN: JP1.EN, JP2.EN
- new net SPI1_MISO: IC1PORTB_L.PB4
- new net SPI1_MOSI: IC1PORTB_L.PB5, U$1.MOSI, U$2.MOSI, U$3.MOSI, U$4.MOSI, U$5.MOSI, U$6.MOSI
- new net SPI1_SCK: IC1PORTB_L.PB3, U$1.SCK, U$2.SCK, U$3.SCK, U$4.SCK, U$5.SCK, U$6.SCK
- new net SWCLK: IC1PORTA_H.PA14, JP3.4
- new net SWDIO: IC1PORTA_H.PA13, JP3.2
- new net TOUCH_SENSE: C18.2, IC1PORTA_L.PA7
- new net TOUCH_SHIELD: R12.2
- new net USART1_RX: IC1PORTB_L.PB7, U$7.2_TXD
- new net USART1_TX: IC1PORTB_L.PB6, U$7.3_RXD
- new net USB_DM: CONN1.DN1, CONN1.DN2, IC1PORTA_H.PA11
- new net USB_DP: CONN1.DP1, CONN1.DP2, IC1PORTA_H.PA12
- net +3V3: now also C10.1, C13.1, C15.1, C16.1, C2.1, C4.1, C5.1, C9.1, IC2.VOUT, JP3.3, S1.3, S1.4, U$8.C1
- net GND: now also C10.2, C13.2, C14.2, C15.2, C16.2, C18.1, C19.2, C2.2, C4.2, C5.2, C9.2, IC2.GND, IC3.A0, IC3.A1, IC3.A2, IC3.WP, JP1.GND, JP2.GND, JP3.1, R1.2, R13.1, R4.1, R5.1, U$7.1_GND; no longer R1.1
- net N$5: now also R1.1, S1.1, S1.2; no longer R1.2
Other:
- moved on the sheet: C2, IC1AN_POWER, IC1PORTA_L, IC1PORTB_H, IC1PORTB_L, R1

Commit message: routing
Parts:
- removed C15, C16: (no value), clock:C-USC1210
- removed CONN1: USB-C_WURTH_632723X00011USB-C, breakouts:USB-C_WURTH_632723X00011USB-C
- added L1: (no value), basicBoard:INDUCTOR0805
- added R14, R15: (no value), clock:RESISTOR0805-RES
- added X3: USB-MICROB, basicBoard:USB-MICROB
- C17: device clock:C-USC1210 -> clock:CAP0805
Connections:
- new net EXIXE_RESET: IC1PORTA_H.PA15, U$1.RST, U$2.RST, U$3.RST, U$4.RST, U$5.RST, U$6.RST
- new net N$17: IC1PORTB_L.PB3, R5.1
- new net N$19: IC1PORTB_L.PB5, R15.1
- new net N$20: IC1PORTB_L.PB4, R14.1
- net +3V3: no longer C15.1, C16.1
- net +5V: now also X3.VBUS; no longer CONN1.VBUS1, CONN1.VBUS2, CONN1.VBUS3, CONN1.VBUS4
- net GND: now also C17.2, X3.GND; no longer C15.2, C16.2, CONN1.GND0, CONN1.GND1, CONN1.GND3, CONN1.GND4, CONN1.SHIELD1, CONN1.SHIELD2, CONN1.SHIELD3, CONN1.SHIELD4, CONN1.SHIELD5, CONN1.SHIELD6, R4.1, R5.1
- net N$12: now also C17.1, L1.2; no longer CONN1.CC2
- net N$13: now also R4.1, U$7.14_VCC_RF; no longer CONN1.CC1, R5.2
- net N$4: now also L1.1
- net SPI1_MISO: now also R14.2, U$1.MISO, U$2.MISO, U$3.MISO, U$4.MISO, U$5.MISO, U$6.MISO; no longer IC1PORTB_L.PB4
- net SPI1_MOSI: now also R15.2; no longer IC1PORTB_L.PB5
- net SPI1_SCK: now also R5.2; no longer IC1PORTB_L.PB3
- net USART1_RX: now also U$7.3_RXD; no longer U$7.2_TXD
- net USART1_TX: now also U$7.2_TXD; no longer U$7.3_RXD
- net USB_DM: now also X3.D-; no longer CONN1.DN1, CONN1.DN2
- net USB_DP: now also X3.D+; no longer CONN1.DP1, CONN1.DP2
Other:
- moved on the sheet: IC1PORTB_L, R4, R5
