File: pcb/clock.sch (EAGLE design)
At the start: 64 parts, among them IC1 STM32F072C8T6, IC2 REG1117, IC3 24C64ST, X3 USB-MICROB

Commit message: routing done
Parts:
- removed JP4: (no value), pinhead:PINHD-2X3
- added G1: CH291-1220LF, basicBoard:CH291-1220LF
- added JP5: (no value), pinhead:PINHD-1X4
- added R16: (no value), clock:RESISTOR0805-RES
- added S4, S5: SWITCH-MOMENTARY-2SIDE_EZ, bus:SWITCH-MOMENTARY-2SIDE_EZ
- added TP1: PTR1TP20R, testpad:PTR1TP20R
Connections:
- new net DS18B20_DATA: IC1PORTC.PC13, R16.1, U$9.DATA
- new net EXIXE1_CS: IC1PORTB_L.PB0, U$1.CS
- new net EXIXE2_CS: IC1PORTB_L.PB1, U$2.CS
- new net EXIXE3_CS: IC1PORTB_L.PB2, U$3.CS
- new net EXIXE4_CS: IC1PORTB_H.PB12, U$4.CS
- new net EXIXE5_CS: IC1PORTB_H.PB13, U$5.CS
- new net EXIXE6_CS: IC1PORTB_H.PB14, U$6.CS
- new net GPS_RESET: IC1PORTA_L.PA0, U$7.9_V_RESET_N
- new net GPS_TP: IC1PORTB_H.PB15, U$7.4_TIMEPULSE
- new net N$21: LED2.C, R9.1
- new net N$22: IC1PORTA_H.PA10, S4.1
- new net N$23: IC1PORTA_H.PA8, S5.1
- new net RX3: IC1PORTB_H.PB10, JP5.1
- new net TX3: IC1PORTB_H.PB11, JP5.2, R9.2
- new net VBAT: G1.+, IC1AN_POWER.VBAT, U$7.6_V_BCKP
- net +3V3: now also IC1AN_POWER.VDDA, JP5.4, LED2.A, R16.2, U$7.7_VCC_IO, U$7.8_VCC, U$9.VCC
- net GND: now also G1.-, IC1AN_POWER.VSSA, JP5.3, S4.2, S4.ANCHOR, S5.2, S5.ANCHOR, U$9.GND
- net LIGHT_SENSOR_OUTPUT: now also IC1PORTA_L.PA1
Other:
- moved on the sheet: IC1AN_POWER, LED2, R9

Commit message: added gps header
Parts:
- added JP4: (no value), pinhead:PINHD-2X2
- added R17: (no value), clock:RESISTOR0805-RES
Connections:
- net +5V: now also R17.2
- net GND: now also JP4.1
- net GPS_TP: now also JP4.3
- net N$21: now also R9.2; no longer R9.1
- net NIXIE_PWR_EN: now also R17.1
- net RX3: now also R9.1
- net TX3: no longer R9.2
- net USART1_RX: now also JP4.4
- net USART1_TX: now also JP4.2
Other:
- moved on the sheet: LED2, R9
Changed lines of the file:
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@@
 <part name="LED2" library="backplane" deviceset="LED" device="CHIP-LED0805"/>
 <part name="+3V16" library="backplane" deviceset="+3V3" device=""/>
-<part name="R9" library="clock" deviceset="RESISTOR" device="0805-RES"/>
 <part name="IC1" library="joyAnalog" deviceset="STM32F072C8T6" device=""/>
 <part name="R1" library="clock" deviceset="RESISTOR" device="0805-RES"/>
@@
 <part name="GND48" library="backplane" deviceset="GND" device=""/>
 <part name="TP1" library="testpad" library_urn="urn:adsk.eagle:library:385" deviceset="PTR1" device="TP20R"/>
+<part name="R9" library="clock" deviceset="RESISTOR" device="0805-RES"/>
+<part name="JP4" library="pinhead" library_urn="urn:adsk.eagle:library:325" deviceset="PINHD-2X2" device=""/>
+<part name="GND41" library="backplane" deviceset="GND" device=""/>
+<part name="R17" library="clock" deviceset="RESISTOR" device="0805-RES"/>
 </parts>
 <sheets>
@@
 <instance part="R8" gate="G$1" x="154.94" y="-101.6" rot="R90"/>
 <instance part="+3V15" gate="G$1" x="154.94" y="-93.98"/>
-<instance part="LED2" gate="G$1" x="7.62" y="-53.34" rot="R180"/>
-<instance part="+3V16" gate="G$1" x="7.62" y="-60.96" rot="R180"/>
-<instance part="R9" gate="G$1" x="7.62" y="-40.64" rot="R90"/>
+<instance part="LED2" gate="G$1" x="22.86" y="-15.24"/>
+<instance part="+3V16" gate="G$1" x="22.86" y="-7.62"/>
 <instance part="IC1" gate="PORTA_L" x="55.88" y="-7.62" rot="R180"/>
 <instance part="IC1" gate="PORTA_H" x="55.88" y="-33.02" rot="R180"/>
@@
 <instance part="GND48" gate="1" x="101.6" y="-68.58"/>
 <instance part="TP1" gate="G$1" x="66.04" y="-78.74"/>
+<instance part="R9" gate="G$1" x="22.86" y="-27.94" rot="R90"/>
+<instance part="JP4" gate="A" x="520.7" y="-215.9"/>
+<instance part="GND41" gate="1" x="497.84" y="-215.9"/>
+<instance part="R17" gate="G$1" x="88.9" y="-256.54" rot="R270"/>
 </instances>
 <busses>
@@
 <junction x="93.98" y="-66.04"/>
 </segment>
+<segment>
+<pinref part="GND41" gate="1" pin="GND"/>
+<pinref part="JP4" gate="A" pin="1"/>
+<wire x1="497.84" y1="-213.36" x2="515.62" y2="-213.36" width="0.1524" layer="91"/>
+</segment>
 </net>
 <net name="+3V3" class="0">
@@
 <pinref part="+3V16" gate="G$1" pin="+3V3"/>
 <pinref part="LED2" gate="G$1" pin="A"/>
-<wire x1="7.62" y1="-58.42" x2="7.62" y2="-55.88" width="0.1524" layer="91"/>
+<wire x1="22.86" y1="-10.16" x2="22.86" y2="-12.7" width="0.1524" layer="91"/>
 </segment>
 <segment>
@@
 <wire x1="58.42" y1="-261.62" x2="27.94" y2="-261.62" width="0.1524" layer="91"/>
 <junction x="27.94" y="-261.62"/>
+<pinref part="R17" gate="G$1" pin="2"/>
+<wire x1="58.42" y1="-261.62" x2="88.9" y2="-261.62" width="0.1524" layer="91"/>
+<junction x="58.42" y="-261.62"/>
 </segment>
 <segment>
@@
 <junction x="27.94" y="-259.08"/>
 <label x="-12.7" y="-259.08" size="1.778" layer="95"/>
+<wire x1="58.42" y1="-259.08" x2="83.82" y2="-259.08" width="0.1524" layer="91"/>
+<wire x1="83.82" y1="-259.08" x2="83.82" y2="-251.46" width="0.1524" layer="91"/>
+<junction x="58.42" y="-259.08"/>
+<pinref part="R17" gate="G$1" pin="1"/>
+<wire x1="83.82" y1="-251.46" x2="88.9" y2="-251.46" width="0.1524" layer="91"/>
 </segment>
 </net>
@@
 <segment>
 <pinref part="U$7" gate="G$1" pin="2_TXD"/>
-<wire x1="508" y1="-193.04" x2="482.6" y2="-193.04" width="0.1524" layer="91"/>
+<wire x1="535.94" y1="-193.04" x2="525.78" y2="-193.04" width="0.1524" layer="91"/>
 <label x="492.76" y="-193.04" size="1.778" layer="95"/>
+<pinref part="JP4" gate="A" pin="2"/>
+<wire x1="525.78" y1="-193.04" x2="482.6" y2="-193.04" width="0.1524" layer="91"/>
+<wire x1="523.24" y1="-213.36" x2="525.78" y2="-213.36" width="0.1524" layer="91"/>
+<wire x1="525.78" y1="-213.36" x2="525.78" y2="-193.04" width="0.1524" layer="91"/>
+<junction x="525.78" y="-193.04"/>
 </segment>
 </net>
@@
 <segment>
 <pinref part="U$7" gate="G$1" pin="3_RXD"/>
-<wire x1="508" y1="-187.96" x2="482.6" y2="-187.96" width="0.1524" layer="91"/>
+<wire x1="535.94" y1="-187.96" x2="528.32" y2="-187.96" width="0.1524" layer="91"/>
 <label x="492.76" y="-187.96" size="1.778" layer="95"/>
+<pinref part="JP4" gate="A" pin="4"/>
+<wire x1="528.32" y1="-187.96" x2="482.6" y2="-187.96" width="0.1524" layer="91"/>
+<wire x1="523.24" y1="-215.9" x2="528.32" y2="-215.9" width="0.1524" layer="91"/>
+<wire x1="528.32" y1="-215.9" x2="528.32" y2="-187.96" width="0.1524" layer="91"/>
+<junction x="528.32" y="-187.96"/>
 </segment>
 </net>
@@
 <segment>
 <pinref part="U$7" gate="G$1" pin="4_TIMEPULSE"/>
-<wire x1="508" y1="-182.88" x2="482.6" y2="-182.88" width="0.1524" layer="91"/>
+<wire x1="535.94" y1="-182.88" x2="510.54" y2="-182.88" width="0.1524" layer="91"/>
 <label x="492.76" y="-182.88" size="1.778" layer="95"/>
+<pinref part="JP4" gate="A" pin="3"/>
+<wire x1="510.54" y1="-182.88" x2="482.6" y2="-182.88" width="0.1524" layer="91"/>
+<wire x1="515.62" y1="-215.9" x2="510.54" y2="-215.9" width="0.1524" layer="91"/>
+<wire x1="510.54" y1="-215.9" x2="510.54" y2="-182.88" width="0.1524" layer="91"/>
+<junction x="510.54" y="-182.88"/>
 </segment>
 </net>
@@
 <pinref part="JP5" gate="A" pin="1"/>
 <label x="7.62" y="-33.02" size="1.778" layer="95"/>
-<wire x1="17.78" y1="-33.02" x2="30.48" y2="-33.02" width="0.1524" layer="91"/>
+<wire x1="17.78" y1="-33.02" x2="22.86" y2="-33.02" width="0.1524" layer="91"/>
 <pinref part="IC1" gate="PORTB_H" pin="PB10"/>
+<wire x1="22.86" y1="-33.02" x2="30.48" y2="-33.02" width="0.1524" layer="91"/>
 <wire x1="-10.16" y1="-35.56" x2="17.78" y2="-33.02" width="0.1524" layer="91"/>
+<pinref part="R9" gate="G$1" pin="1"/>
+<junction x="22.86" y="-33.02"/>
 </segment>
 </net>
@@
 <pinref part="JP5" gate="A" pin="2"/>
 <label x="7.62" y="-35.56" size="1.778" layer="95"/>
-<pinref part="R9" gate="G$1" pin="2"/>
 <wire x1="7.62" y1="-35.56" x2="30.48" y2="-35.56" width="0.1524" layer="91"/>
 <pinref part="IC1" gate="PORTB_H" pin="PB11"/>
 <wire x1="-10.16" y1="-33.02" x2="7.62" y2="-35.56" width="0.1524" layer="91"/>
-<junction x="7.62" y="-35.56"/>
-</segment>
-</net>
-<net name="N$21" class="0">
-<segment>
-<pinref part="LED2" gate="G$1" pin="C"/>
-<pinref part="R9" gate="G$1" pin="1"/>
-<wire x1="7.62" y1="-48.26" x2="7.62" y2="-45.72" width="0.1524" layer="91"/>
 </segment>
 </net>
@@
 </segment>
 </net>
+<net name="N$21" class="0">
+<segment>
+<pinref part="R9" gate="G$1" pin="2"/>
+<pinref part="LED2" gate="G$1" pin="C"/>
+<wire x1="22.86" y1="-20.32" x2="22.86" y2="-22.86" width="0.1524" layer="91"/>
+</segment>
+</net>
