File: pcb/clock.sch (EAGLE design)
At the start: 69 parts, among them IC1 STM32F072C8T6, IC2 REG1117, IC3 24C64ST, X3 USB-MICROB

Commit message: new routing
Parts:
- removed U$9: DS18B20, DS18B20U:DS18B20
- added C1, C3: (no value), clock:CAP0805
- added TP4: TEST-POINT3X5, SparkFun-Passives:TEST-POINT3X5
- added U1: DS18B20, SparkFun-Sensors:DS18B20
- TP2, TP3: value PTR1TP20R -> TEST-POINT3X5; device testpad:PTR1TP20R -> SparkFun-Passives:TEST-POINT3X5
Connections:
- removed net N$22: IC1PORTA_H.PA10, S4.1
- removed net N$23: IC1PORTA_H.PA8, S5.1
- removed net N$24: IC1PORTA_H.PA9, R9.2
- new net A_BUTTON: IC1PORTF/OSC.PF0/OSC<=, S4.1
- new net B_BUTTON: IC1PORTF/OSC.PF1/OSC=>, S5.1
- new net GPS_FIX_LED: IC1PORTA_L.PA7, R9.2
- new net N$15: IC1PORTA_H.PA8, TP4.1
- new net N$6: IC1PORTA_H.PA10, TP2.1
- new net N$7: IC1PORTA_H.PA9, TP3.1
- new net SD_CS: IC1PORTA_L.PA0, SD1.CD/DAT3(!CS!)
- net +3V3: now also C1.1, C3.1, SD1.VDD, U1.VDD; no longer U$9.VCC
- net DS18B20_DATA: now also IC1PORTA_L.PA6, U1.DQ; no longer IC1PORTC.PC13, U$9.DATA
- net GND: now also C1.2, C3.2, SD1.VSS, U1.GND; no longer U$9.GND
- net GPS_RESET: now also IC1PORTC.PC13; no longer IC1PORTA_L.PA0
- net USART1_RX: no longer TP3.TP
- net USART1_TX: no longer TP2.TP
Other:
- moved on the sheet: IC1PORTF/OSC, LED2, R9, S4, S5
