File: pcb/clock_rev0.brd (EAGLE design)
At the start: 145 x 50 mm, 69 parts, among them IC1 STM32F072C8T6, IC2 REG1117, IC3 24C64ST, X3 USB-MICROB

Commit message: all 6
Parts:
- removed SD1: TF-HOLDER, basicBoard:TF-PULL
- added C1, C3, R10, R6: (no value), clock:0805
- added Q1: (no value), adafruit:NX3225
- added U$16: TOUCHPAD, touch_pad:TOUCHPAD_PAK
- moved U$9 90.5 mm to (61.1, 47.8), turned to 270 degrees
- moved R16 89.7 mm to (58.2, 43.1), turned to 0 degrees
- moved U$15 8.00 mm to (4.00, 28.0)
- moved U$14 4.00 mm to (4.00, 39.0)
- moved R12 3.68 mm to (44.8, 33.0)
- moved C18 3.56 mm to (41.1, 26.3)
- moved C11 3.18 mm to (55.6, 37.2)
- moved C12 3.01 mm to (53.2, 40.1), turned to 0 degrees
- moved C19 2.26 mm to (44.9, 35.4), turned to 180 degrees
- moved X2 2.24 mm to (49.6, 36.7), turned to 90 degrees
- moved R11 0.36 mm to (41.1, 32.0)
Connections:
- removed net VDD: SD1.4
- removed net VSS: SD1.6
- new net N$15: IC1.15, R10.1
- new net N$16: IC1.16, R6.1
- new net N$6: C3.1, IC1.6, X2.P$2
- new net N$7: C1.1, IC1.5, X2.P$1
- new net TOUCH_SENSE: C18.2, IC1.17
- new net TOUCH_SHIELD: R12.2
- net GND: now also C1.2, C3.2, Q1.2, Q1.4; no longer SD1.S1, SD1.S2, SD1.S3, SD1.S4
- net N$1: now also Q1.1; no longer X2.P$2
- net N$10: now also R6.2, U$16.P$1; no longer R12.2, U$14.P$1
- net N$14: now also R11.2, U$14.P$1; no longer C18.2, IC1.15
- net N$2: now also Q1.3; no longer X2.P$1
- net N$9: now also R10.2; no longer R11.2
- net SPI1_MISO: no longer SD1.7
- net SPI1_MOSI: no longer SD1.3
- net SPI1_SCK: no longer SD1.5
Routing:
- net N$14: track 3.68 -> 40.3 mm
- net GND: track 137.6 -> 167.9 mm
- net DS18B20_DATA: track 0.00 -> 21.6 mm
- net TOUCH_SHIELD: track 0.00 -> 18.1 mm
- net +3V3: track 76.0 -> 85.9 mm, vias 11 -> 12
- net N$10: track 36.9 -> 44.6 mm
- net N$7: track 0.00 -> 7.48 mm
- net N$23: track 128.1 -> 121.7 mm
- net N$6: track 0.00 -> 5.40 mm
- net TOUCH_SENSE: track 0.00 -> 4.74 mm
- net N$16: track 0.00 -> 4.08 mm
- net N$9: track 41.1 -> 37.1 mm
- net N$15: track 0.00 -> 3.73 mm
- net N$11: track 4.65 -> 2.08 mm
- net N$2: track 5.55 -> 7.94 mm
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- added copper zone on layer 1, net TOUCH_SHIELD
Other:
- board text added: "*"
- board text added: "+"
- board text added: "-"
- board text added: "exixe clock dekuNukem 2017"
