File: pcb/clock_rev0.sch (EAGLE design)
At the start: 69 parts, among them IC1 STM32F072C8T6, IC2 REG1117, IC3 24C64ST, X3 USB-MICROB

Commit message: all 6
Parts:
- removed SD1: TF-HOLDER, basicBoard:TF-HOLDER
- added C1, C3: (no value), clock:CAP0805
- added Q1: (no value), adafruit:XTAL-4-3225
- added R10, R6: (no value), clock:RESISTOR0805-RES
- added U$16: TOUCHPAD, touch_pad:TOUCHPAD
Connections:
- new net N$15: IC1PORTA_L.PA5, R10.1
- new net N$16: IC1PORTA_L.PA6, R6.1
- new net N$6: C3.1, IC1PORTF/OSC.PF1/OSC=>, X2.P$2
- new net N$7: C1.1, IC1PORTF/OSC.PF0/OSC<=, X2.P$1
- new net TOUCH_SENSE: C18.2, IC1PORTA_L.PA7
- new net TOUCH_SHIELD: R12.2
- net GND: now also C1.2, C3.2, Q1.G1, Q1.G2; no longer SD1.S1, SD1.S2, SD1.S3, SD1.S4
- net N$1: now also Q1.X1; no longer X2.P$2
- net N$10: now also R6.2, U$16.PAD; no longer R12.2, U$14.PAD
- net N$14: now also R11.2, U$14.PAD; no longer C18.2, IC1PORTA_L.PA5
- net N$2: now also Q1.X2; no longer X2.P$1
- net N$9: now also R10.2; no longer R11.2
- net SPI1_MISO: no longer SD1.DAT0(DO)
- net SPI1_MOSI: no longer SD1.CMD(DI)
- net SPI1_SCK: no longer SD1.CLK(SCLK)
Other:
- moved on the sheet: C18, X2
