File: pcb/exixe12.brd (EAGLE design)
At the start: 20 x 40 mm, 42 parts

Commit message: sending out
Parts:
- added R12: (no value), SparkFun-Resistors:0603-RES
- moved Q6 32.9 mm to (2.41, 33.7), turned to 0 degrees
- moved Q5 31.0 mm to (1.52, 30.4)
- moved R5 28.1 mm to (1.43, 26.6)
- moved R6 27.7 mm to (10.0, 31.8), turned to 180 degrees
- moved R3 25.5 mm to (1.43, 20.0), turned to 270 degrees
- moved Q3 25.2 mm to (2.25, 22.9)
- moved Q1 25.2 mm to (3.10, 17.5)
- moved Q11 24.8 mm to (10.4, 19.3)
- moved R1 24.6 mm to (3.10, 15.0), turned to 180 degrees
- moved R11 24.5 mm to (12.6, 20.6)
- moved R15 24.2 mm to (2.54, 9.53)
- moved R8 23.9 mm to (18.0, 27.7), turned to 0 degrees
- moved R9 23.1 mm to (18.5, 22.6), turned to 180 degrees
- moved Q8 22.8 mm to (18.3, 30.1)
- moved Q4 22.7 mm to (6.43, 27.7), turned to 0 degrees
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
Commit message: new routing
Parts:
- moved R16 25.4 mm to (17.1, 9.14)
- moved R14 22.2 mm to (18.7, 8.89)
- moved C1 2.33 mm to (40.6, 8.89)
- moved R6 0.46 mm to (10.4, 31.5)
- moved D1 0.36 mm to (10.4, 29.2)
Changed lines of the file:
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@@
 <attribute name="NAME" x="4.7645" y="15.549" size="0.8128" layer="25" font="vector" rot="R270"/>
 </element>
-<element name="C1" library="joyAnalog" package="0805" value="1uF" x="38.481" y="8.001" smashed="yes">
-<attribute name="NAME" x="38.6334" y="8.8011" size="0.8128" layer="25" font="vector"/>
+<element name="C1" library="joyAnalog" package="0805" value="1uF" x="40.64" y="8.89" smashed="yes">
+<attribute name="NAME" x="40.7924" y="9.6901" size="0.8128" layer="25" font="vector"/>
 </element>
 <element name="Q2" library="nixx" package="SOT323" value="" x="7.218" y="21.685" smashed="yes" rot="R90">
@@
 <attribute name="VALUE" x="3.638" y="32.325" size="1.016" layer="27"/>
 </element>
-<element name="R6" library="joyAnalog" package="0805" value="4K7" x="10.011" y="31.78" smashed="yes" rot="R180">
-<attribute name="NAME" x="7.9976" y="32.5455" size="0.8128" layer="25" font="vector"/>
+<element name="R6" library="joyAnalog" package="0805" value="4K7" x="10.392" y="31.526" smashed="yes" rot="R180">
+<attribute name="NAME" x="8.3786" y="32.2915" size="0.8128" layer="25" font="vector"/>
 </element>
 <element name="Q7" library="nixx" package="SOT323" value="" x="17.004" y="33.274" smashed="yes">
@@
 <attribute name="VALUE" x="1.11" y="35.025" size="1.27" layer="27"/>
 </element>
-<element name="D1" library="nixx" package="3528-COMMON-ANODE" value="RGB_LED_CA-150141M173100-R&amp;G&amp;B" x="10.181" y="29.445" smashed="yes"/>
+<element name="D1" library="nixx" package="3528-COMMON-ANODE" value="RGB_LED_CA-150141M173100-R&amp;G&amp;B" x="10.435" y="29.191" smashed="yes"/>
 <element name="R13" library="joyAnalog" package="0805" value="68K" x="5.715" y="36.449" smashed="yes" rot="R180">
 <attribute name="NAME" x="6.7818" y="35.6997" size="0.7112" layer="25" font="vector" rot="R180"/>
 </element>
-<element name="R14" library="joyAnalog" package="0805" value="470" x="40.894" y="8.636" smashed="yes" rot="R270">
-<attribute name="NAME" x="39.8145" y="10.16" size="0.8128" layer="25" font="vector" rot="R90"/>
+<element name="R14" library="joyAnalog" package="0805" value="470" x="18.669" y="8.89" smashed="yes" rot="R270">
+<attribute name="NAME" x="17.5895" y="10.414" size="0.8128" layer="25" font="vector" rot="R90"/>
 </element>
 <element name="R15" library="joyAnalog" package="0805" value="470" x="2.54" y="9.525" smashed="yes">
 <attribute name="NAME" x="3.2131" y="10.5918" size="0.8128" layer="25" font="vector" rot="R90"/>
 </element>
-<element name="R16" library="joyAnalog" package="0805" value="0" x="42.545" y="8.636" smashed="yes" rot="R270">
-<attribute name="NAME" x="40.8813" y="10.1854" size="0.8128" layer="25" font="vector" rot="R90"/>
+<element name="R16" library="joyAnalog" package="0805" value="0" x="17.145" y="9.144" smashed="yes" rot="R270">
+<attribute name="NAME" x="15.4813" y="10.6934" size="0.8128" layer="25" font="vector" rot="R90"/>
 </element>
 <element name="R17" library="joyAnalog" package="0805" value="4K7" x="29.083" y="8.128" smashed="yes" rot="MR180">
@@
 <wire x1="7.08" y1="26.786" x2="8.118" y2="22.335" width="0" layer="19" extent="1-1"/>
 <wire x1="19.158" y1="24.013" x2="18.944" y2="18.735" width="0" layer="19" extent="1-1"/>
-<wire x1="39.381" y1="8.001" x2="28.967" y2="16.637" width="0" layer="19" extent="1-1"/>
+<wire x1="41.54" y1="8.89" x2="28.967" y2="16.637" width="0" layer="19" extent="1-1"/>
 </signal>
 <signal name="N$1">
@@
 <contactref element="Q6" pad="1"/>
 <contactref element="R6" pad="2"/>
-<wire x1="1.763" y1="32.755" x2="9.111" y2="31.78" width="0" layer="19" extent="1-1"/>
+<wire x1="1.763" y1="32.755" x2="9.492" y2="31.526" width="0" layer="19" extent="1-1"/>
 </signal>
 <signal name="N$9">
@@
 <wire x1="19.177" y1="36.643" x2="17.62" y2="38.2" width="0.2032" layer="16"/>
 <wire x1="19.177" y1="36.643" x2="41.91" y2="35.952" width="0" layer="19" extent="1-16"/>
-<wire x1="11.731" y1="30.295" x2="18.415" y2="37.405" width="0" layer="19" extent="1-1"/>
-<wire x1="5.8344" y1="12.038" x2="11.731" y2="30.295" width="0" layer="19" extent="1-1"/>
+<wire x1="11.985" y1="30.041" x2="18.415" y2="37.405" width="0" layer="19" extent="1-1"/>
+<wire x1="5.8344" y1="12.038" x2="11.985" y2="30.041" width="0" layer="19" extent="1-1"/>
 <wire x1="5.8344" y1="8.838" x2="5.8344" y2="12.038" width="0" layer="19" extent="1-1"/>
 <wire x1="14.4196" y1="6.438" x2="5.8344" y2="8.838" width="0" layer="19" extent="1-1"/>
 <wire x1="29.983" y1="8.128" x2="14.4196" y2="6.438" width="0" layer="19" extent="1-16"/>
-<wire x1="37.581" y1="8.001" x2="29.983" y2="8.128" width="0" layer="19" extent="1-16"/>
-<wire x1="38.111" y1="7.239" x2="37.581" y2="8.001" width="0" layer="19" extent="1-16"/>
+<wire x1="39.74" y1="8.89" x2="29.983" y2="8.128" width="0" layer="19" extent="1-16"/>
+<wire x1="38.111" y1="7.239" x2="39.74" y2="8.89" width="0" layer="19" extent="1-16"/>
 <wire x1="27.167" y1="16.637" x2="29.983" y2="8.128" width="0" layer="19" extent="1-16"/>
 </signal>
@@
 <contactref element="D1" pad="2"/>
 <contactref element="R16" pad="1"/>
-<wire x1="11.731" y1="28.595" x2="42.545" y2="9.536" width="0" layer="19" extent="1-1"/>
+<wire x1="11.985" y1="28.341" x2="17.145" y2="10.044" width="0" layer="19" extent="1-1"/>
 </signal>
 <signal name="PWM_BLUE">
@@
 <contactref element="D1" pad="4"/>
 <contactref element="R15" pad="1"/>
-<wire x1="1.64" y1="9.525" x2="8.631" y2="28.595" width="0" layer="19" extent="1-1"/>
+<wire x1="1.64" y1="9.525" x2="8.885" y2="28.341" width="0" layer="19" extent="1-1"/>
 </signal>
 <signal name="N$15">
 <contactref element="D1" pad="3"/>
 <contactref element="R14" pad="1"/>
-<wire x1="8.631" y1="30.295" x2="40.894" y2="9.536" width="0" layer="19" extent="1-1"/>
+<wire x1="8.885" y1="30.041" x2="18.669" y2="9.79" width="0" layer="19" extent="1-1"/>
 </signal>
 <signal name="N$19">

Commit message: removed bake
Parts:
- removed Q13: (no value), nixx:SOT323
- removed R12: (no value), SparkFun-Resistors:0603-RES
- removed R22, R23: 10K, joyAnalog:0805
- removed R24: 4K7, joyAnalog:0805
- removed T1: (no value), zetex:SOT323
- added JP3: JUMPER-SMT_2_NO_NO-SILK, SparkFun-Jumpers:SMT-JUMPER_2_NO_NO-SILK
- R19: value 10K -> 68K
- moved R5 16.0 mm to (2.52, 10.6), turned to 180 degrees
- moved R8 13.4 mm to (17.4, 14.4)
- moved R3 13.3 mm to (2.45, 6.70), turned to 180 degrees
- moved R2 12.0 mm to (2.46, 8.73)
- moved R4 10.7 mm to (2.54, 14.7), turned to 180 degrees
- moved R9 10.2 mm to (17.3, 12.5), turned to 0 degrees
- moved Q6 9.00 mm to (10.2, 38.2), turned to 180 degrees
- moved R6 7.00 mm to (12.3, 38.2), turned to 90 degrees
- moved R10 5.97 mm to (17.3, 10.5), turned to 0 degrees
- moved Q1 5.69 mm to (7.57, 21.0), turned to 180 degrees
- moved Q2 5.26 mm to (2.89, 18.7), turned to 0 degrees
- moved R15 4.57 mm to (2.41, 4.95)
- moved Q5 3.92 mm to (3.17, 33.9)
- moved R19 3.84 mm to (6.86, 39.0), turned to 180 degrees
- moved R14 2.92 mm to (17.0, 6.48), turned to 180 degrees
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Connections:
- removed net BAKE: R24.2
- removed net N$20: R22.1, T1.2
- removed net N$22: Q13.3, R19.2, R22.2
- removed net N$23: Q13.1, R24.1
- removed net N$24: R23.2, T1.1
- new net N$2: JP3.1, R19.2
- net +180V: now also R19.1; no longer R23.1
- net GND: no longer Q13.2
- net N$19: now also JP3.2; no longer R19.1, T1.3
Routing:
- net N$19: track 0.87 -> 0.00 mm

Commit message: working on exixe 12
Parts:
- moved C1 24.0 mm to (16.9, 5.21), turned to 180 degrees
- moved R5 20.2 mm to (2.06, 30.8), turned to 90 degrees
- moved R8 13.1 mm to (18.4, 27.4), turned to 180 degrees
- moved R4 12.0 mm to (6.70, 25.9), turned to 90 degrees
- moved R1 10.6 mm to (9.07, 21.1), turned to 90 degrees
- moved R9 9.77 mm to (18.5, 22.2), turned to 180 degrees
- moved R2 7.64 mm to (2.97, 16.4)
- moved R3 7.13 mm to (2.96, 13.8)
- moved R10 5.58 mm to (17.1, 16.1), turned to 90 degrees
- moved R15 1.53 mm to (2.54, 6.48)
- moved Q1 0.90 mm to (6.93, 21.6)
- moved Q10 0.90 mm to (17.0, 19.3)
- moved Q4 0.76 mm to (6.68, 29.2)
- moved Q11 0.76 mm to (11.0, 20.4)
- moved Q2 0.52 mm to (3.02, 19.2)
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Routing:
- net +180V: track 0.00 -> 23.9 mm, vias 0 -> 1
- net SPI_SCK: track 0.00 -> 7.15 mm
- net SPI_MISO: track 0.00 -> 4.79 mm
- net N$19: track 0.00 -> 4.15 mm
- net SPI_MOSI: track 0.00 -> 4.07 mm
- net NIXIE_5: track 0.00 -> 3.19 mm
- net NIXIE_1: track 0.00 -> 2.61 mm
- net NIXIE_4: track 0.00 -> 2.57 mm
- net NIXIE_3: track 0.00 -> 2.54 mm
- net NIXIE_DOT_LEFT: track 0.00 -> 2.46 mm
- net NIXIE_10: track 0.00 -> 2.30 mm
- net NIXIE_2: track 0.00 -> 2.28 mm
- net N$4: track 0.00 -> 2.07 mm
- net N$13: track 0.00 -> 1.80 mm
- net N$6: track 0.00 -> 1.77 mm
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Other:
- board text removed: "+"
- board text removed: "2017"
- board text removed: "PF0"
- board text removed: "PF1"
- board text removed: "RX"
- board text removed: "TX"
- board text removed: "dekuNukem"
- board text removed: "eixie"

Commit message: exixe12 draft finishewd
Parts:
- removed C3: 100nF, joyAnalog:0805
- removed R17: 4K7, joyAnalog:0805
- added TP1, TP2, TP3, TP4, TP5, TP6: PTR1TP13R, nixx:TP13R
- moved R18 24.8 mm to (14.1, 16.3), flipped to the top, turned to 0 degrees
- moved C2 22.6 mm to (5.51, 14.8), turned to 90 degrees
- moved R14 14.2 mm to (2.84, 6.88), turned to 0 degrees
- moved R16 5.63 mm to (18.0, 13.9), turned to 270 degrees
- moved R9 3.54 mm to (15.4, 24.0), turned to 0 degrees
- moved R8 3.18 mm to (15.5, 28.5), turned to 0 degrees
- moved R15 2.31 mm to (4.47, 5.21)
- moved R11 2.12 mm to (11.5, 22.9), turned to 0 degrees
- moved C1 1.77 mm to (15.2, 5.77), turned to 0 degrees
- moved Q7 1.26 mm to (17.0, 35.2), turned to 90 degrees
- moved R7 1.12 mm to (17.8, 33.0), turned to 0 degrees
- moved R3 0.97 mm to (2.03, 13.6), turned to 90 degrees
- moved R10 0.86 mm to (16.4, 15.7)
- moved R1 0.57 mm to (8.82, 21.6)
- moved R5 0.51 mm to (1.55, 30.8)
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Connections:
- new net N$14: TP6.TP, U$2.10
- new net N$16: TP2.TP, U$2.20
- new net N$17: TP3.TP, U$2.14
- new net N$18: TP4.TP, U$2.15
- new net N$20: TP5.TP, U$2.26
- new net TX: TP1.TP, U$2.19
- net +3V3: no longer C3.1, R17.2
- net GND: no longer C3.2
- net NRST: no longer R17.1
- net PWM_BLUE: now also U$2.21
- net PWM_GREEN: now also U$2.9
- net PWM_RED: now also U$2.8
- net STM_1: now also U$2.31
- net STM_10: now also U$2.22
- net STM_2: now also U$2.3
- net STM_3: now also U$2.6
- net STM_4: now also U$2.2
- net STM_5: now also U$2.7
- net STM_6: now also U$2.18
- net STM_7: now also U$2.29
- net STM_8: now also U$2.28
- net STM_9: now also U$2.27
- net STM_DOT_LEFT: now also U$2.30
Routing:
- net STM_6: track 0.00 -> 37.6 mm, vias 0 -> 2
- net GND: track 0.00 -> 33.5 mm
- net N$3: track 0.00 -> 31.6 mm, vias 0 -> 2
- net N$15: track 0.00 -> 30.4 mm, vias 0 -> 2
- net STM_5: track 0.00 -> 25.2 mm
- net STM_7: track 0.00 -> 23.4 mm
- net N$21: track 0.00 -> 20.3 mm, vias 0 -> 2
- net STM_4: track 0.00 -> 18.1 mm
- net SPI_CS: track 0.00 -> 17.1 mm, vias 0 -> 1
- net STM_8: track 0.00 -> 16.2 mm
- net SWD_CLK: track 0.00 -> 14.3 mm, vias 0 -> 1
- net SWD_DIO: track 0.00 -> 11.7 mm, vias 0 -> 1
- net STM_9: track 0.00 -> 11.1 mm
- net NRST: track 0.00 -> 10.8 mm, vias 0 -> 1
- net STM_DOT_LEFT: track 0.00 -> 10.1 mm
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Other:
- board text added: "+"
- board text added: "MI"
- board text added: "MO"
- board text removed: "MISO"
- board text removed: "MOSI"

Commit message: added restrict
Routing:
- net GND: track 33.5 -> 40.3 mm
Changed lines of the file:
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@@
 <layer number="39" name="tKeepout" color="4" fill="11" visible="no" active="yes"/>
 <layer number="40" name="bKeepout" color="1" fill="11" visible="no" active="yes"/>
-<layer number="41" name="tRestrict" color="4" fill="10" visible="yes" active="yes"/>
-<layer number="42" name="bRestrict" color="1" fill="10" visible="yes" active="yes"/>
+<layer number="41" name="tRestrict" color="4" fill="10" visible="no" active="yes"/>
+<layer number="42" name="bRestrict" color="1" fill="10" visible="no" active="yes"/>
 <layer number="43" name="vRestrict" color="2" fill="10" visible="no" active="yes"/>
 <layer number="44" name="Drills" color="7" fill="1" visible="no" active="yes"/>
@@
 <text x="15.4178" y="35.3314" size="1.143" layer="26" font="vector" rot="MR0">G</text>
 <text x="11.6078" y="32.639" size="1.143" layer="25" font="vector">+</text>
+<polygon width="0.1524" layer="41">
+<vertex x="3.5052" y="39.878"/>
+<vertex x="7.9756" y="39.878"/>
+<vertex x="8.2804" y="39.5732"/>
+<vertex x="8.2804" y="36.2712"/>
+<vertex x="7.9248" y="35.9156"/>
+<vertex x="7.4676" y="35.9156"/>
+<vertex x="7.0104" y="36.3728"/>
+<vertex x="1.778" y="36.3728"/>
+<vertex x="0.6604" y="37.4904"/>
+<vertex x="0.6604" y="39.0144"/>
+<vertex x="1.524" y="39.878"/>
+<vertex x="3.556" y="39.878"/>
+</polygon>
+<polygon width="0.254" layer="42">
+<vertex x="7.366" y="36.0172"/>
+<vertex x="8.5344" y="32.5628"/>
+<vertex x="8.7884" y="29.21"/>
+<vertex x="7.1628" y="27.4828"/>
+<vertex x="7.1628" y="24.892"/>
+<vertex x="12.6492" y="19.2024"/>
+<vertex x="12.7508" y="17.4244"/>
+<vertex x="13.462" y="17.018"/>
+<vertex x="14.5288" y="16.8656"/>
+<vertex x="15.3416" y="17.4244"/>
+<vertex x="15.6464" y="18.542"/>
+<vertex x="15.2908" y="19.5072"/>
+<vertex x="14.5796" y="20.0152"/>
+<vertex x="13.4112" y="19.812"/>
+<vertex x="9.144" y="24.2316"/>
+<vertex x="9.652" y="29.0576"/>
+<vertex x="9.6012" y="33.02"/>
+<vertex x="8.1788" y="36.6268"/>
+<vertex x="7.2644" y="36.3728"/>
+<vertex x="7.366" y="36.068"/>
+</polygon>
 </plain>
 <attributes>
@@
 <wire x1="4.9276" y1="28.702" x2="5.4356" y2="29.21" width="0.254" layer="1"/>
 <wire x1="5.4356" y1="29.21" x2="6.604" y2="29.21" width="0.254" layer="1"/>
-<wire x1="10.399" y1="21.2708" x2="9.8044" y2="21.8654" width="0.254" layer="1"/>
-<wire x1="9.8044" y1="21.8654" x2="9.8044" y2="23.114" width="0.254" layer="1"/>
-<wire x1="9.8044" y1="23.114" x2="9.4996" y2="23.4188" width="0.1524" layer="1"/>
-<wire x1="9.4996" y1="23.4188" x2="8.7376" y2="23.4188" width="0.1524" layer="1"/>
-<wire x1="8.7376" y1="23.4188" x2="7.7216" y2="24.4348" width="0.1524" layer="1"/>
+<wire x1="10.399" y1="21.2708" x2="9.8044" y2="21.8654" width="0.2032" layer="1"/>
+<wire x1="9.8044" y1="21.8654" x2="9.8044" y2="23.114" width="0.2032" layer="1"/>
+<wire x1="9.8044" y1="23.114" x2="9.4996" y2="23.4188" width="0.2032" layer="1"/>
+<wire x1="9.4996" y1="23.4188" x2="8.7376" y2="23.4188" width="0.2032" layer="1"/>
+<wire x1="8.7376" y1="23.4188" x2="7.7216" y2="24.4348" width="0.2032" layer="1"/>
 <wire x1="7.7216" y1="24.4348" x2="7.7216" y2="27.432" width="0.2032" layer="1"/>
 <wire x1="7.7216" y1="27.432" x2="7.334" y2="27.8196" width="0.2032" layer="1"/>
 <wire x1="7.334" y1="27.8196" x2="7.334" y2="28.31" width="0.1524" layer="1"/>
-<wire x1="3.825" y1="33.009" x2="2.6675625" y2="31.8515625" width="0.1524" layer="1"/>
-<wire x1="2.6675625" y1="31.8515625" x2="2.6675625" y2="28.702" width="0.1524" layer="1"/>
+<wire x1="3.825" y1="33.009" x2="2.6675625" y2="31.8515625" width="0.2032" layer="1"/>
+<wire x1="2.6675625" y1="31.8515625" x2="2.6675625" y2="28.702" width="0.2032" layer="1"/>
+<wire x1="15.08" y1="38.2" x2="9.256" y2="38.2" width="0.254" layer="1"/>
+<wire x1="9.256" y1="38.2" x2="9.256" y2="39.127" width="0.254" layer="1"/>
 </signal>
 <signal name="N$1">
