File: pcb/exixe12.brd (EAGLE design)
At the start: 20 x 40 mm, 42 parts

Commit message: increased board isolation
Parts:
- R12, R17: value 68K -> 10K
- moved TP1 3.89 mm to (12.4, 9.91), flipped to the bottom
- renumbered U$2 to IC1
Routing:
- net GND: track 59.2 -> 79.5 mm
- net +3V3: track 11.9 -> 28.3 mm
- net TX: track 2.11 -> 2.30 mm, vias 0 -> 1

Commit message: changed testpoints to unpopulated resistors
Parts:
- removed TP1, TP2, TP3, TP5: PTR1TP13R, nixx:TP13R
- added R20, R21, R22, R23, R24: 10K, joyAnalog:0805
Connections:
- new net N$20: IC1.7, R20.2
- net +3V3: now also R20.1, R21.1, R22.1, R23.2, R24.2
- net N$14: now also R22.2; no longer TP2.TP
- net N$16: now also R23.1; no longer TP3.TP
- net N$17: now also R24.1; no longer TP5.TP
- net STM_5: no longer IC1.7
- net TX: now also R21.2; no longer TP1.TP
Routing:
- net STM_5: track 29.3 -> 33.6 mm
- net GND: track 79.5 -> 76.5 mm, vias 3 -> 1
- net N$20: track 0.00 -> 2.25 mm, vias 0 -> 1
- net N$16: track 2.08 -> 2.62 mm
Other:
- board text removed: "PB6"
- board text removed: "PF0"
- board text removed: "PF1"
- board text removed: "TX"

Commit message: adjusted more values
Parts:
- C1: value 1uF -> 100nF
Changed lines of the file:
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@@
 <attribute name="NAME" x="9.5862" y="19.977284375" size="0.8128" layer="25" font="vector" rot="R180"/>
 </element>
-<element name="C1" library="joyAnalog" package="0805" value="1uF" x="15.2146" y="5.7658" smashed="yes">
+<element name="C1" library="joyAnalog" package="0805" value="100nF" x="15.2146" y="5.7658" smashed="yes">
 <attribute name="NAME" x="15.5448" y="6.8707" size="0.8128" layer="25" font="vector"/>
 </element>
