File: pcb/exixe18.sch (EAGLE design)
At the start: 50 parts

Commit message: added pulldown on boot0
Parts:
- added R25: 68K, joyAnalog:RESISTOR0805-RES
Connections:
- net GND: now also R25.1
- net STM_DOT_RIGHT: now also R25.2
Changed lines of the file:
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@@
 <part name="R20" library="joyAnalog" deviceset="RESISTOR" device="0805-RES" value="4K7"/>
 <part name="R21" library="joyAnalog" deviceset="RESISTOR" device="0805-RES" value="4K7"/>
+<part name="R25" library="joyAnalog" deviceset="RESISTOR" device="0805-RES" value="68K"/>
+<part name="GND16" library="joyAnalog" deviceset="GND" device=""/>
 </parts>
 <sheets>
@@
 <instance part="R20" gate="G$1" x="238.76" y="53.34"/>
 <instance part="R21" gate="G$1" x="238.76" y="27.94"/>
+<instance part="R25" gate="G$1" x="429.26" y="33.02" rot="R90"/>
+<instance part="GND16" gate="1" x="429.26" y="25.4"/>
 </instances>
 <busses>
@@
 <wire x1="431.8" y1="-43.18" x2="441.96" y2="-43.18" width="0.1524" layer="91"/>
 </segment>
+<segment>
+<pinref part="R25" gate="G$1" pin="1"/>
+<pinref part="GND16" gate="1" pin="GND"/>
+</segment>
 </net>
 <net name="N$1" class="0">
@@
 <pinref part="U$2" gate="G$1" pin="PB8"/>
 <label x="426.72" y="38.1" size="1.778" layer="95"/>
-<wire x1="439.42" y1="38.1" x2="424.18" y2="38.1" width="0.1524" layer="91"/>
-</segment>
-</net>
+<wire x1="439.42" y1="38.1" x2="429.26" y2="38.1" width="0.1524" layer="91"/>
+<pinref part="R25" gate="G$1" pin="2"/>
+<wire x1="429.26" y1="38.1" x2="424.18" y2="38.1" width="0.1524" layer="91"/>
+<junction x="429.26" y="38.1"/>
+</segment>
+</net>
