File: pcb/exixe12.sch (EAGLE design)
At the start: 42 parts

Commit message: sending out
Parts:
- added R12: (no value), SparkFun-Resistors:RESISTOR0603
Changed lines of the file:
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@@
 <part name="R19" library="joyAnalog" deviceset="RESISTOR" device="0805-RES" value="10K"/>
 <part name="N1" library="0-nixies-russian" deviceset="IN-12B" device=""/>
+<part name="R12" library="SparkFun-Resistors" deviceset="RESISTOR" device="0603"/>
 </parts>
 <sheets>
@@
 <instance part="R19" gate="G$1" x="378.46" y="-58.42" rot="R270"/>
 <instance part="N1" gate="G$1" x="226.06" y="-33.02"/>
+<instance part="R12" gate="G$1" x="93.98" y="40.64"/>
 </instances>
 <busses>

Commit message: removed bake
Parts:
- removed Q13: (no value), nixx:BF820
- removed R12: (no value), SparkFun-Resistors:RESISTOR0603
- removed R22, R23: 10K, joyAnalog:RESISTOR0805-RES
- removed R24: 4K7, joyAnalog:RESISTOR0805-RES
- removed T1: (no value), zetex:PNPSOT323
- added JP3: JUMPER-SMT_2_NO_NO-SILK, SparkFun-Jumpers:JUMPER-SMT_2_NO_NO-SILK
- R19: value 10K -> 68K
Connections:
- removed net BAKE: R24.2
- removed net N$20: R22.1, T1.B
- removed net N$22: Q13.C, R19.2, R22.2
- removed net N$23: Q13.B, R24.1
- removed net N$24: R23.2, T1.C
- new net N$2: JP3.1, R19.2
- net +180V: now also R19.1; no longer R23.1
- net GND: no longer Q13.E
- net N$19: now also JP3.2; no longer R19.1, T1.E
Other:
- moved on the sheet: R13, R19
Changed lines of the file:
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@@
 <?xml version="1.0" encoding="utf-8"?>
 <!DOCTYPE eagle SYSTEM "eagle.dtd">
-<eagle version="8.2.0">
+<eagle version="8.2.2">
 <drawing>
 <settings>
@@
 <part name="+3V5" library="joyAnalog" deviceset="+3V3" device=""/>
 <part name="+3V6" library="joyAnalog" deviceset="+3V3" device=""/>
-<part name="R22" library="joyAnalog" deviceset="RESISTOR" device="0805-RES" value="10K"/>
-<part name="R23" library="joyAnalog" deviceset="RESISTOR" device="0805-RES" value="10K"/>
-<part name="T1" library="zetex" deviceset="PNPSOT323" device=""/>
-<part name="Q13" library="nixx" deviceset="BF820" device=""/>
-<part name="R24" library="joyAnalog" deviceset="RESISTOR" device="0805-RES" value="4K7"/>
-<part name="GND18" library="joyAnalog" deviceset="GND" device=""/>
-<part name="R19" library="joyAnalog" deviceset="RESISTOR" device="0805-RES" value="10K"/>
 <part name="N1" library="0-nixies-russian" deviceset="IN-12B" device=""/>
-<part name="R12" library="SparkFun-Resistors" deviceset="RESISTOR" device="0603"/>
+<part name="R19" library="joyAnalog" deviceset="RESISTOR" device="0805-RES" value="68K"/>
+<part name="JP3" library="SparkFun-Jumpers" deviceset="JUMPER-SMT_2_NO" device="_NO-SILK"/>
 </parts>
 <sheets>
@@
 <instance part="Q1" gate="A" x="101.6" y="48.26"/>
 <instance part="P+2" gate="1" x="236.22" y="-27.94" rot="MR0"/>
-<instance part="P+1" gate="1" x="363.22" y="-27.94"/>
+<instance part="P+1" gate="1" x="381" y="-27.94"/>
 <instance part="R1" gate="G$1" x="93.98" y="48.26"/>
 <instance part="C1" gate="G$1" x="68.58" y="81.28"/>
@@
 <instance part="+3V3" gate="G$1" x="424.18" y="-43.18"/>
 <instance part="D1" gate="G$1" x="477.52" y="0"/>
-<instance part="R13" gate="G$1" x="386.08" y="-30.48"/>
+<instance part="R13" gate="G$1" x="401.32" y="-30.48"/>
 <instance part="+3V4" gate="G$1" x="459.74" y="2.54"/>
 <instance part="R14" gate="G$1" x="495.3" y="0"/>
@@
 <instance part="+3V5" gate="G$1" x="340.36" y="-20.32" rot="MR0"/>
 <instance part="+3V6" gate="G$1" x="347.98" y="-30.48" rot="MR0"/>
-<instance part="R22" gate="G$1" x="391.16" y="-63.5" rot="R180"/>
-<instance part="R23" gate="G$1" x="406.4" y="-73.66" rot="R90"/>
-<instance part="T1" gate="A" x="403.86" y="-63.5"/>
-<instance part="Q13" gate="A" x="375.92" y="-68.58"/>
-<instance part="R24" gate="G$1" x="368.3" y="-68.58" rot="R180"/>
-<instance part="GND18" gate="1" x="378.46" y="-76.2"/>
-<instance part="R19" gate="G$1" x="378.46" y="-58.42" rot="R270"/>
 <instance part="N1" gate="G$1" x="226.06" y="-33.02"/>
-<instance part="R12" gate="G$1" x="93.98" y="40.64"/>
+<instance part="R19" gate="G$1" x="401.32" y="-38.1"/>
+<instance part="JP3" gate="G$1" x="414.02" y="-38.1"/>
 </instances>
 <busses>
@@
 <pinref part="R13" gate="G$1" pin="1"/>
 <pinref part="P+1" gate="1" pin="+180V"/>
-<wire x1="363.22" y1="-30.48" x2="373.38" y2="-30.48" width="0.1524" layer="91"/>
-<pinref part="R23" gate="G$1" pin="1"/>
-<wire x1="373.38" y1="-30.48" x2="381" y2="-30.48" width="0.1524" layer="91"/>
-<wire x1="406.4" y1="-78.74" x2="406.4" y2="-86.36" width="0.1524" layer="91"/>
-<wire x1="406.4" y1="-86.36" x2="340.36" y2="-86.36" width="0.1524" layer="91"/>
-<wire x1="340.36" y1="-86.36" x2="340.36" y2="-45.72" width="0.1524" layer="91"/>
-<wire x1="340.36" y1="-45.72" x2="373.38" y2="-45.72" width="0.1524" layer="91"/>
-<wire x1="373.38" y1="-45.72" x2="373.38" y2="-30.48" width="0.1524" layer="91"/>
-<junction x="373.38" y="-30.48"/>
+<wire x1="381" y1="-30.48" x2="391.16" y2="-30.48" width="0.1524" layer="91"/>
+<pinref part="R19" gate="G$1" pin="1"/>
+<wire x1="391.16" y1="-30.48" x2="396.24" y2="-30.48" width="0.1524" layer="91"/>
+<wire x1="396.24" y1="-38.1" x2="391.16" y2="-38.1" width="0.1524" layer="91"/>
+<wire x1="391.16" y1="-38.1" x2="391.16" y2="-30.48" width="0.1524" layer="91"/>
+<junction x="391.16" y="-30.48"/>
 </segment>
 </net>
@@
 </segment>
 <segment>
-<pinref part="Q13" gate="A" pin="E"/>
-<pinref part="GND18" gate="1" pin="GND"/>
-</segment>
-<segment>
 <pinref part="JP1" gate="A" pin="6"/>
 <pinref part="GND15" gate="1" pin="GND"/>
@@
 <net name="N$19" class="0">
 <segment>
-<pinref part="T1" gate="A" pin="E"/>
-<wire x1="406.4" y1="-30.48" x2="406.4" y2="-53.34" width="0.1524" layer="91"/>
 <pinref part="JP1" gate="A" pin="1"/>
 <pinref part="R13" gate="G$1" pin="2"/>
-<wire x1="406.4" y1="-53.34" x2="406.4" y2="-58.42" width="0.1524" layer="91"/>
-<wire x1="431.8" y1="-30.48" x2="406.4" y2="-30.48" width="0.1524" layer="91"/>
-<wire x1="406.4" y1="-30.48" x2="391.16" y2="-30.48" width="0.1524" layer="91"/>
-<junction x="406.4" y="-30.48"/>
-<pinref part="R19" gate="G$1" pin="1"/>
-<wire x1="378.46" y1="-53.34" x2="406.4" y2="-53.34" width="0.1524" layer="91"/>
-<junction x="406.4" y="-53.34"/>
-</segment>
-</net>
-<net name="N$20" class="0">
-<segment>
-<pinref part="T1" gate="A" pin="B"/>
-<pinref part="R22" gate="G$1" pin="1"/>
-<wire x1="396.24" y1="-63.5" x2="401.32" y2="-63.5" width="0.1524" layer="91"/>
-</segment>
-</net>
-<net name="N$22" class="0">
-<segment>
-<pinref part="R22" gate="G$1" pin="2"/>
-<pinref part="Q13" gate="A" pin="C"/>
-<wire x1="378.46" y1="-63.5" x2="386.08" y2="-63.5" width="0.1524" layer="91"/>
+<wire x1="431.8" y1="-30.48" x2="419.1" y2="-30.48" width="0.1524" layer="91"/>
+<pinref part="JP3" gate="G$1" pin="2"/>
+<wire x1="419.1" y1="-30.48" x2="406.4" y2="-30.48" width="0.1524" layer="91"/>
+<wire x1="419.1" y1="-38.1" x2="419.1" y2="-30.48" width="0.1524" layer="91"/>
+<junction x="419.1" y="-30.48"/>
+</segment>
+</net>
+<net name="N$2" class="0">
+<segment>
 <pinref part="R19" gate="G$1" pin="2"/>
-<junction x="378.46" y="-63.5"/>
-</segment>
-</net>
-<net name="N$23" class="0">
-<segment>
-<pinref part="Q13" gate="A" pin="B"/>
-<pinref part="R24" gate="G$1" pin="1"/>
-</segment>
-</net>
-<net name="N$24" class="0">
-<segment>
-<pinref part="T1" gate="A" pin="C"/>
-<pinref part="R23" gate="G$1" pin="2"/>
-</segment>
-</net>
-<net name="BAKE" class="0">
-<segment>
-<pinref part="R24" gate="G$1" pin="2"/>
-<wire x1="345.44" y1="-68.58" x2="363.22" y2="-68.58" width="0.1524" layer="91"/>
-<label x="347.98" y="-68.58" size="1.778" layer="95"/>
-</segment>
-</net>
+<pinref part="JP3" gate="G$1" pin="1"/>
+<wire x1="406.4" y1="-38.1" x2="408.94" y2="-38.1" width="0.1524" layer="91"/>
+</segment>
+</net>

Commit message: exixe12 draft finishewd
Parts:
- removed C3: 100nF, joyAnalog:CAP0805
- removed R17: 4K7, joyAnalog:RESISTOR0805-RES
- added TP1, TP2, TP3, TP4, TP5, TP6: PTR1TP13R, nixx:PTR1TP13R
Connections:
- new net N$14: TP6.TP, U$2.PA4
- new net N$16: TP2.TP, U$2.PA10
- new net N$17: TP3.TP, U$2.PB0
- new net N$18: TP4.TP, U$2.PB1
- new net N$20: TP5.TP, U$2.PB3
- new net TX: TP1.TP, U$2.PA9
- net +3V3: no longer C3.1, R17.2
- net GND: no longer C3.2
- net NRST: no longer R17.1
- net PWM_BLUE: now also U$2.PA11
- net PWM_GREEN: now also U$2.PA3
- net PWM_RED: now also U$2.PA2
- net STM_1: now also U$2.PB8
- net STM_10: now also U$2.PA12
- net STM_2: now also U$2.PF1/OSC_OUT
- net STM_3: now also U$2.PA0
- net STM_4: now also U$2.PF0/OSC_IN
- net STM_5: now also U$2.PA1
- net STM_6: now also U$2.PA8
- net STM_7: now also U$2.PB6
- net STM_8: now also U$2.PB5
- net STM_9: now also U$2.PB4
- net STM_DOT_LEFT: now also U$2.PB7
Changed lines of the file:
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@@
 <part name="+3V1" library="joyAnalog" deviceset="+3V3" device=""/>
 <part name="C2" library="joyAnalog" deviceset="CAP" device="0805" value="100nF"/>
-<part name="C3" library="joyAnalog" deviceset="CAP" device="0805" value="100nF"/>
 <part name="GND14" library="joyAnalog" deviceset="GND" device=""/>
 <part name="+3V2" library="joyAnalog" deviceset="+3V3" device=""/>
@@
 <part name="R15" library="joyAnalog" deviceset="RESISTOR" device="0805-RES" value="470"/>
 <part name="R16" library="joyAnalog" deviceset="RESISTOR" device="0805-RES" value="0"/>
-<part name="R17" library="joyAnalog" deviceset="RESISTOR" device="0805-RES" value="4K7"/>
 <part name="R18" library="joyAnalog" deviceset="RESISTOR" device="0805-RES" value="4K7"/>
-<part name="+3V5" library="joyAnalog" deviceset="+3V3" device=""/>
 <part name="+3V6" library="joyAnalog" deviceset="+3V3" device=""/>
 <part name="N1" library="0-nixies-russian" deviceset="IN-12B" device=""/>
 <part name="R19" library="joyAnalog" deviceset="RESISTOR" device="0805-RES" value="68K"/>
 <part name="JP3" library="SparkFun-Jumpers" deviceset="JUMPER-SMT_2_NO" device="_NO-SILK"/>
+<part name="TP1" library="nixx" deviceset="PTR1" device="TP13R"/>
+<part name="TP2" library="nixx" deviceset="PTR1" device="TP13R"/>
+<part name="TP3" library="nixx" deviceset="PTR1" device="TP13R"/>
+<part name="TP4" library="nixx" deviceset="PTR1" device="TP13R"/>
+<part name="TP5" library="nixx" deviceset="PTR1" device="TP13R"/>
+<part name="TP6" library="nixx" deviceset="PTR1" device="TP13R"/>
 </parts>
 <sheets>
@@
 <instance part="+3V1" gate="G$1" x="375.92" y="104.14"/>
 <instance part="C2" gate="G$1" x="83.82" y="81.28"/>
-<instance part="C3" gate="G$1" x="99.06" y="81.28"/>
 <instance part="GND14" gate="1" x="83.82" y="76.2"/>
 <instance part="+3V2" gate="G$1" x="83.82" y="88.9"/>
@@
 <instance part="R15" gate="G$1" x="495.3" y="7.62"/>
 <instance part="R16" gate="G$1" x="495.3" y="-7.62"/>
-<instance part="R17" gate="G$1" x="340.36" y="-27.94" rot="R90"/>
 <instance part="R18" gate="G$1" x="347.98" y="-38.1" rot="R90"/>
-<instance part="+3V5" gate="G$1" x="340.36" y="-20.32" rot="MR0"/>
 <instance part="+3V6" gate="G$1" x="347.98" y="-30.48" rot="MR0"/>
 <instance part="N1" gate="G$1" x="226.06" y="-33.02"/>
 <instance part="R19" gate="G$1" x="401.32" y="-38.1"/>
 <instance part="JP3" gate="G$1" x="414.02" y="-38.1"/>
+<instance part="TP1" gate="G$1" x="459.74" y="76.2" rot="R90"/>
+<instance part="TP2" gate="G$1" x="447.04" y="73.66" rot="R90"/>
+<instance part="TP3" gate="G$1" x="436.88" y="55.88" rot="R90"/>
+<instance part="TP4" gate="G$1" x="449.58" y="53.34" rot="R90"/>
+<instance part="TP5" gate="G$1" x="462.28" y="50.8" rot="R90"/>
+<instance part="TP6" gate="G$1" x="449.58" y="91.44" rot="R90"/>
 </instances>
 <busses>
@@
 </segment>
 <segment>
-<pinref part="C3" gate="G$1" pin="2"/>
 <pinref part="C2" gate="G$1" pin="2"/>
-<wire x1="83.82" y1="78.74" x2="99.06" y2="78.74" width="0.1524" layer="91"/>
 <junction x="83.82" y="78.74"/>
 <pinref part="GND14" gate="1" pin="GND"/>
@@
 </segment>
 <segment>
-<pinref part="R17" gate="G$1" pin="2"/>
-<pinref part="+3V5" gate="G$1" pin="+3V3"/>
-</segment>
-<segment>
 <pinref part="R18" gate="G$1" pin="2"/>
 <pinref part="+3V6" gate="G$1" pin="+3V3"/>
 </segment>
 <segment>
-<pinref part="C3" gate="G$1" pin="1"/>
 <pinref part="C2" gate="G$1" pin="1"/>
-<wire x1="99.06" y1="86.36" x2="83.82" y2="86.36" width="0.1524" layer="91"/>
 <pinref part="C1" gate="G$1" pin="1"/>
 <wire x1="83.82" y1="86.36" x2="68.58" y2="86.36" width="0.1524" layer="91"/>
@@
 <wire x1="307.34" y1="-33.02" x2="330.2" y2="-33.02" width="0.1524" layer="91"/>
 <label x="307.34" y="-33.02" size="1.778" layer="95"/>
-<pinref part="R17" gate="G$1" pin="1"/>
-<wire x1="340.36" y1="-33.02" x2="330.2" y2="-33.02" width="0.1524" layer="91"/>
-<junction x="330.2" y="-33.02"/>
 </segment>
 </net>
@@
 <label x="193.04" y="48.26" size="1.778" layer="95"/>
 </segment>
+<segment>
+<pinref part="U$2" gate="G$1" pin="PB7"/>
+<wire x1="444.5" y1="40.64" x2="424.18" y2="40.64" width="0.1524" layer="91"/>
+<label x="429.26" y="40.64" size="1.778" layer="95"/>
+</segment>
 </net>
 <net name="STM_6" class="0">
@@
 <label x="144.78" y="48.26" size="1.778" layer="95"/>
 </segment>
+<segment>
+<label x="426.72" y="78.74" size="1.778" layer="95"/>
+<pinref part="U$2" gate="G$1" pin="PA8"/>
+<wire x1="439.42" y1="78.74" x2="424.18" y2="78.74" width="0.1524" layer="91"/>
+</segment>
 </net>
 <net name="STM_7" class="0">
@@
 <label x="144.78" y="22.86" size="1.778" layer="95"/>
 </segment>
+<segment>
+<pinref part="U$2" gate="G$1" pin="PB6"/>
+<wire x1="444.5" y1="43.18" x2="424.18" y2="43.18" width="0.1524" layer="91"/>
+<label x="429.26" y="43.18" size="1.778" layer="95"/>
+</segment>
 </net>
 <net name="STM_8" class="0">
@@
 <label x="144.78" y="-2.54" size="1.778" layer="95"/>
 </segment>
+<segment>
+<pinref part="U$2" gate="G$1" pin="PB5"/>
+<wire x1="444.5" y1="45.72" x2="424.18" y2="45.72" width="0.1524" layer="91"/>
+<label x="429.26" y="45.72" size="1.778" layer="95"/>
+</segment>
 </net>
 <net name="STM_9" class="0">
@@
 <label x="144.78" y="-27.94" size="1.778" layer="95"/>
 </segment>
+<segment>
+<pinref part="U$2" gate="G$1" pin="PB4"/>
+<wire x1="444.5" y1="48.26" x2="424.18" y2="48.26" width="0.1524" layer="91"/>
+<label x="429.26" y="48.26" size="1.778" layer="95"/>
+</segment>
 </net>
 <net name="STM_10" class="0">
@@
 <label x="144.78" y="-55.88" size="1.778" layer="95"/>
 </segment>
+<segment>
+<pinref part="U$2" gate="G$1" pin="PA12"/>
+<wire x1="439.42" y1="68.58" x2="424.18" y2="68.58" width="0.1524" layer="91"/>
+<label x="426.72" y="68.58" size="1.778" layer="95"/>
+</segment>
 </net>
 <net name="STM_5" class="0">
@@
 <label x="78.74" y="-55.88" size="1.778" layer="95"/>
 </segment>
+<segment>
+<pinref part="U$2" gate="G$1" pin="PA1"/>
+<wire x1="439.42" y1="99.06" x2="424.18" y2="99.06" width="0.1524" layer="91"/>
+<label x="426.72" y="99.06" size="1.778" layer="95"/>
+</segment>
 </net>
 <net name="STM_4" class="0">
@@
 <label x="78.74" y="-27.94" size="1.778" layer="95"/>
 </segment>
+<segment>
+<pinref part="U$2" gate="G$1" pin="PF0/OSC_IN"/>
+<wire x1="368.3" y1="55.88" x2="383.54" y2="55.88" width="0.1524" layer="91"/>
+<label x="370.84" y="55.88" size="1.778" layer="95"/>
+</segment>
 </net>
 <net name="STM_3" class="0">
@@
 <label x="78.74" y="-2.54" size="1.778" layer="95"/>
 </segment>
+<segment>
+<pinref part="U$2" gate="G$1" pin="PA0"/>
+<wire x1="439.42" y1="101.6" x2="424.18" y2="101.6" width="0.1524" layer="91"/>
+<label x="426.72" y="101.6" size="1.778" layer="95"/>
+</segment>
 </net>
 <net name="STM_2" class="0">
@@
 <label x="78.74" y="22.86" size="1.778" layer="95"/>
 </segment>
+<segment>
+<pinref part="U$2" gate="G$1" pin="PF1/OSC_OUT"/>
+<wire x1="368.3" y1="53.34" x2="383.54" y2="53.34" width="0.1524" layer="91"/>
+<label x="370.84" y="53.34" size="1.778" layer="95"/>
+</segment>
 </net>
 <net name="STM_1" class="0">
@@
 <label x="78.74" y="48.26" size="1.778" layer="95"/>
 </segment>
+<segment>
+<pinref part="U$2" gate="G$1" pin="PB8"/>
+<wire x1="444.5" y1="38.1" x2="424.18" y2="38.1" width="0.1524" layer="91"/>
+<label x="429.26" y="38.1" size="1.778" layer="95"/>
+</segment>
 </net>
 <net name="N$21" class="0">
@@
 <label x="502.92" y="-7.62" size="1.778" layer="95"/>
 </segment>
+<segment>
+<pinref part="U$2" gate="G$1" pin="PA11"/>
+<wire x1="439.42" y1="71.12" x2="424.18" y2="71.12" width="0.1524" layer="91"/>
+<label x="426.72" y="71.12" size="1.778" layer="95"/>
+</segment>
 </net>
 <net name="PWM_GREEN" class="0">
@@
 <label x="502.92" y="7.62" size="1.778" layer="95"/>
 </segment>
+<segment>
+<pinref part="U$2" gate="G$1" pin="PA3"/>
+<wire x1="439.42" y1="93.98" x2="424.18" y2="93.98" width="0.1524" layer="91"/>
+<label x="426.72" y="93.98" size="1.778" layer="95"/>
+</segment>
 </net>
 <net name="PWM_RED" class="0">
@@
 <wire x1="515.62" y1="0" x2="500.38" y2="0" width="0.1524" layer="91"/>
 <label x="502.92" y="0" size="1.778" layer="95"/>
+</segment>
+<segment>
+<pinref part="U$2" gate="G$1" pin="PA2"/>
+<wire x1="439.42" y1="96.52" x2="424.18" y2="96.52" width="0.1524" layer="91"/>
+<label x="426.72" y="96.52" size="1.778" layer="95"/>
 </segment>
 </net>
@@
 </segment>
 </net>
+<net name="TX" class="0">
+<segment>
+<pinref part="U$2" gate="G$1" pin="PA9"/>
+<pinref part="TP1" gate="G$1" pin="TP"/>
+<wire x1="457.2" y1="76.2" x2="424.18" y2="76.2" width="0.1524" layer="91"/>
+<label x="447.04" y="76.2" size="1.778" layer="95"/>
+</segment>
+</net>
+<net name="N$16" class="0">
+<segment>
+<pinref part="U$2" gate="G$1" pin="PA10"/>
+<pinref part="TP2" gate="G$1" pin="TP"/>
+<wire x1="444.5" y1="73.66" x2="424.18" y2="73.66" width="0.1524" layer="91"/>
+</segment>
+</net>
+<net name="N$14" class="0">
+<segment>
+<pinref part="U$2" gate="G$1" pin="PA4"/>
+<pinref part="TP6" gate="G$1" pin="TP"/>
+<wire x1="424.18" y1="91.44" x2="447.04" y2="91.44" width="0.1524" layer="91"/>
+</segment>
+</net>
+<net name="N$17" class="0">
+<segment>
+<pinref part="U$2" gate="G$1" pin="PB0"/>
+<pinref part="TP3" gate="G$1" pin="TP"/>
+<wire x1="424.18" y1="55.88" x2="434.34" y2="55.88" width="0.1524" layer="91"/>
+</segment>
+</net>
+<net name="N$18" class="0">
+<segment>
+<pinref part="U$2" gate="G$1" pin="PB1"/>
+<pinref part="TP4" gate="G$1" pin="TP"/>
+<wire x1="424.18" y1="53.34" x2="447.04" y2="53.34" width="0.1524" layer="91"/>
+</segment>
+</net>
+<net name="N$20" class="0">
+<segment>
+<pinref part="U$2" gate="G$1" pin="PB3"/>
+<pinref part="TP5" gate="G$1" pin="TP"/>
+<wire x1="424.18" y1="50.8" x2="459.74" y2="50.8" width="0.1524" layer="91"/>
+</segment>
+</net>

Commit message: clened up added credit
Parts:
- N1: device 0-nixies-russian:IN-12B -> exixe12:IN-12B
Changed lines of the file:
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@@
 <part name="R18" library="joyAnalog" deviceset="RESISTOR" device="0805-RES" value="4K7"/>
 <part name="+3V6" library="joyAnalog" deviceset="+3V3" device=""/>
-<part name="N1" library="0-nixies-russian" deviceset="IN-12B" device=""/>
+<part name="N1" library="exixe12" deviceset="IN-12B" device=""/>
 <part name="R19" library="joyAnalog" deviceset="RESISTOR" device="0805-RES" value="68K"/>
 <part name="JP3" library="SparkFun-Jumpers" deviceset="JUMPER-SMT_2_NO" device="_NO-SILK"/>
