File: pcb/exixe12.sch (EAGLE design)
At the start: 42 parts

Commit message: adjust passive values and added bom
Parts:
- R12: value 510K -> 68K
- R17: value 47K -> 68K
Changed lines of the file:
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@@
 <part name="JP3" library="SparkFun-Jumpers" deviceset="JUMPER-SMT_2_NO" device="_NO-SILK"/>
 <part name="TP1" library="nixx" deviceset="PTR1" device="TP13R"/>
-<part name="R12" library="joyAnalog" deviceset="RESISTOR" device="0805-RES" value="510K"/>
-<part name="R17" library="joyAnalog" deviceset="RESISTOR" device="0805-RES" value="47K"/>
+<part name="R12" library="joyAnalog" deviceset="RESISTOR" device="0805-RES" value="68K"/>
+<part name="R17" library="joyAnalog" deviceset="RESISTOR" device="0805-RES" value="68K"/>
 <part name="GND12" library="joyAnalog" deviceset="GND" device=""/>
 <part name="TP2" library="nixx" deviceset="PTR1" device="TP13R"/>

Commit message: increased board isolation
Parts:
- R12, R17: value 68K -> 10K
- renumbered U$2 to IC1
Changed lines of the file:
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@@
 </classes>
 <parts>
-<part name="U$2" library="nixx" deviceset="STM32F042K6" device=""/>
+<part name="IC1" library="nixx" deviceset="STM32F042K6" device=""/>
 <part name="JP2" library="pinhead" deviceset="PINHD-1X7" device=""/>
 <part name="Q1" library="nixx" deviceset="BF820" device=""/>
@@
 <part name="JP3" library="SparkFun-Jumpers" deviceset="JUMPER-SMT_2_NO" device="_NO-SILK"/>
 <part name="TP1" library="nixx" deviceset="PTR1" device="TP13R"/>
-<part name="R12" library="joyAnalog" deviceset="RESISTOR" device="0805-RES" value="68K"/>
-<part name="R17" library="joyAnalog" deviceset="RESISTOR" device="0805-RES" value="68K"/>
+<part name="R12" library="joyAnalog" deviceset="RESISTOR" device="0805-RES" value="10K"/>
+<part name="R17" library="joyAnalog" deviceset="RESISTOR" device="0805-RES" value="10K"/>
 <part name="GND12" library="joyAnalog" deviceset="GND" device=""/>
 <part name="TP2" library="nixx" deviceset="PTR1" device="TP13R"/>
@@
 </plain>
 <instances>
-<instance part="U$2" gate="G$1" x="386.08" y="104.14"/>
+<instance part="IC1" gate="G$1" x="386.08" y="104.14"/>
 <instance part="JP2" gate="A" x="332.74" y="-40.64"/>
 <instance part="Q1" gate="A" x="101.6" y="48.26"/>
@@
 <segment>
 <pinref part="GND13" gate="1" pin="GND"/>
-<pinref part="U$2" gate="G$1" pin="VSS"/>
+<pinref part="IC1" gate="G$1" pin="VSS"/>
 <wire x1="375.92" y1="38.1" x2="383.54" y2="38.1" width="0.1524" layer="91"/>
 </segment>
@@
 <segment>
 <pinref part="+3V1" gate="G$1" pin="+3V3"/>
-<pinref part="U$2" gate="G$1" pin="VDD"/>
+<pinref part="IC1" gate="G$1" pin="VDD"/>
 <wire x1="375.92" y1="101.6" x2="383.54" y2="101.6" width="0.1524" layer="91"/>
-<pinref part="U$2" gate="G$1" pin="VDDA"/>
+<pinref part="IC1" gate="G$1" pin="VDDA"/>
 <wire x1="383.54" y1="99.06" x2="375.92" y2="99.06" width="0.1524" layer="91"/>
 <wire x1="375.92" y1="99.06" x2="375.92" y2="101.6" width="0.1524" layer="91"/>
@@
 </segment>
 <segment>
-<pinref part="U$2" gate="G$1" pin="PA5"/>
+<pinref part="IC1" gate="G$1" pin="PA5"/>
 <wire x1="439.42" y1="88.9" x2="424.18" y2="88.9" width="0.1524" layer="91"/>
 <label x="426.72" y="88.9" size="1.778" layer="95"/>
@@
 </segment>
 <segment>
-<pinref part="U$2" gate="G$1" pin="PA6"/>
+<pinref part="IC1" gate="G$1" pin="PA6"/>
 <wire x1="439.42" y1="86.36" x2="424.18" y2="86.36" width="0.1524" layer="91"/>
 <label x="426.72" y="86.36" size="1.778" layer="95"/>
@@
 </segment>
 <segment>
-<pinref part="U$2" gate="G$1" pin="PA7"/>
+<pinref part="IC1" gate="G$1" pin="PA7"/>
 <wire x1="439.42" y1="83.82" x2="424.18" y2="83.82" width="0.1524" layer="91"/>
 <label x="426.72" y="83.82" size="1.778" layer="95"/>
@@
 <segment>
 <label x="426.72" y="60.96" size="1.778" layer="95"/>
-<pinref part="U$2" gate="G$1" pin="PA15"/>
+<pinref part="IC1" gate="G$1" pin="PA15"/>
 <wire x1="439.42" y1="60.96" x2="424.18" y2="60.96" width="0.1524" layer="91"/>
 </segment>
@@
 </segment>
 <segment>
-<pinref part="U$2" gate="G$1" pin="PA13/SWDIO"/>
+<pinref part="IC1" gate="G$1" pin="PA13/SWDIO"/>
 <wire x1="439.42" y1="66.04" x2="424.18" y2="66.04" width="0.1524" layer="91"/>
 <label x="426.72" y="66.04" size="1.778" layer="95"/>
@@
 </segment>
 <segment>
-<pinref part="U$2" gate="G$1" pin="PA14/SWCLK"/>
+<pinref part="IC1" gate="G$1" pin="PA14/SWCLK"/>
 <wire x1="439.42" y1="63.5" x2="424.18" y2="63.5" width="0.1524" layer="91"/>
 <label x="426.72" y="63.5" size="1.778" layer="95"/>
@@
 <net name="NRST" class="0">
 <segment>
-<pinref part="U$2" gate="G$1" pin="NRST"/>
+<pinref part="IC1" gate="G$1" pin="NRST"/>
 <wire x1="370.84" y1="78.74" x2="383.54" y2="78.74" width="0.1524" layer="91"/>
 <label x="370.84" y="78.74" size="1.778" layer="95"/>
@@
 </segment>
 <segment>
-<pinref part="U$2" gate="G$1" pin="PB7"/>
+<pinref part="IC1" gate="G$1" pin="PB7"/>
 <wire x1="444.5" y1="40.64" x2="424.18" y2="40.64" width="0.1524" layer="91"/>
 <label x="429.26" y="40.64" size="1.778" layer="95"/>
@@
 <segment>
 <label x="426.72" y="78.74" size="1.778" layer="95"/>
-<pinref part="U$2" gate="G$1" pin="PA8"/>
+<pinref part="IC1" gate="G$1" pin="PA8"/>
 <wire x1="439.42" y1="78.74" x2="424.18" y2="78.74" width="0.1524" layer="91"/>
 </segment>
@@
 <segment>
 <label x="429.26" y="45.72" size="1.778" layer="95"/>
-<pinref part="U$2" gate="G$1" pin="PB5"/>
+<pinref part="IC1" gate="G$1" pin="PB5"/>
 <wire x1="444.5" y1="45.72" x2="424.18" y2="45.72" width="0.1524" layer="91"/>
 </segment>
@@
 <segment>
 <label x="429.26" y="48.26" size="1.778" layer="95"/>
-<pinref part="U$2" gate="G$1" pin="PB4"/>
+<pinref part="IC1" gate="G$1" pin="PB4"/>
 <wire x1="444.5" y1="48.26" x2="424.18" y2="48.26" width="0.1524" layer="91"/>
 </segment>
@@
 <segment>
 <label x="429.26" y="50.8" size="1.778" layer="95"/>
-<pinref part="U$2" gate="G$1" pin="PB3"/>
+<pinref part="IC1" gate="G$1" pin="PB3"/>
 <wire x1="444.5" y1="50.8" x2="424.18" y2="50.8" width="0.1524" layer="91"/>
 </segment>
@@
 <segment>
 <label x="426.72" y="71.12" size="1.778" layer="95"/>
-<pinref part="U$2" gate="G$1" pin="PA11"/>
+<pinref part="IC1" gate="G$1" pin="PA11"/>
 <wire x1="439.42" y1="71.12" x2="424.18" y2="71.12" width="0.1524" layer="91"/>
 </segment>
@@
 </segment>
 <segment>
-<pinref part="U$2" gate="G$1" pin="PA1"/>
+<pinref part="IC1" gate="G$1" pin="PA1"/>
 <wire x1="452.12" y1="99.06" x2="424.18" y2="99.06" width="0.1524" layer="91"/>
 <label x="426.72" y="99.06" size="1.778" layer="95"/>
-<pinref part="U$2" gate="G$1" pin="PA4"/>
+<pinref part="IC1" gate="G$1" pin="PA4"/>
 <wire x1="452.12" y1="99.06" x2="452.12" y2="91.44" width="0.1524" layer="91"/>
 <wire x1="452.12" y1="91.44" x2="424.18" y2="91.44" width="0.1524" layer="91"/>
@@
 <segment>
 <label x="429.26" y="53.34" size="1.778" layer="95"/>
-<pinref part="U$2" gate="G$1" pin="PB1"/>
+<pinref part="IC1" gate="G$1" pin="PB1"/>
 <wire x1="444.5" y1="53.34" x2="424.18" y2="53.34" width="0.1524" layer="91"/>
 </segment>
@@
 </segment>
 <segment>
-<pinref part="U$2" gate="G$1" pin="PA0"/>
+<pinref part="IC1" gate="G$1" pin="PA0"/>
 <wire x1="439.42" y1="101.6" x2="424.18" y2="101.6" width="0.1524" layer="91"/>
 <label x="426.72" y="101.6" size="1.778" layer="95"/>
@@
 <segment>
 <label x="429.26" y="55.88" size="1.778" layer="95"/>
-<pinref part="U$2" gate="G$1" pin="PB0"/>
+<pinref part="IC1" gate="G$1" pin="PB0"/>
 <wire x1="444.5" y1="55.88" x2="424.18" y2="55.88" width="0.1524" layer="91"/>
 </segment>
@@
 </segment>
 <segment>
-<pinref part="U$2" gate="G$1" pin="PB8"/>
+<pinref part="IC1" gate="G$1" pin="PB8"/>
 <wire x1="444.5" y1="38.1" x2="439.42" y2="38.1" width="0.1524" layer="91"/>
 <label x="429.26" y="38.1" size="1.778" layer="95"/>
@@
 <segment>
 <label x="426.72" y="73.66" size="1.778" layer="95"/>
-<pinref part="U$2" gate="G$1" pin="PA10"/>
+<pinref part="IC1" gate="G$1" pin="PA10"/>
 <wire x1="439.42" y1="73.66" x2="424.18" y2="73.66" width="0.1524" layer="91"/>
 </segment>
@@
 </segment>
 <segment>
-<pinref part="U$2" gate="G$1" pin="PA3"/>
+<pinref part="IC1" gate="G$1" pin="PA3"/>
 <wire x1="439.42" y1="93.98" x2="424.18" y2="93.98" width="0.1524" layer="91"/>
 <label x="426.72" y="93.98" size="1.778" layer="95"/>
@@
 </segment>
 <segment>
-<pinref part="U$2" gate="G$1" pin="PA2"/>
+<pinref part="IC1" gate="G$1" pin="PA2"/>
 <wire x1="439.42" y1="96.52" x2="424.18" y2="96.52" width="0.1524" layer="91"/>
 <label x="426.72" y="96.52" size="1.778" layer="95"/>
@@
 <net name="TX" class="0">
 <segment>
-<pinref part="U$2" gate="G$1" pin="PA9"/>
+<pinref part="IC1" gate="G$1" pin="PA9"/>
 <pinref part="TP1" gate="G$1" pin="TP"/>
 <wire x1="457.2" y1="76.2" x2="424.18" y2="76.2" width="0.1524" layer="91"/>
@@
 <net name="N$14" class="0">
 <segment>
-<pinref part="U$2" gate="G$1" pin="PB6"/>
+<pinref part="IC1" gate="G$1" pin="PB6"/>
 <wire x1="424.18" y1="43.18" x2="449.58" y2="43.18" width="0.1524" layer="91"/>
 <pinref part="TP2" gate="G$1" pin="TP"/>
@@
 <net name="N$16" class="0">
 <segment>
-<pinref part="U$2" gate="G$1" pin="PF0/OSC_IN"/>
+<pinref part="IC1" gate="G$1" pin="PF0/OSC_IN"/>
 <wire x1="370.84" y1="55.88" x2="383.54" y2="55.88" width="0.1524" layer="91"/>
 <pinref part="TP3" gate="G$1" pin="TP"/>
@@
 <segment>
 <pinref part="TP5" gate="G$1" pin="TP"/>
-<pinref part="U$2" gate="G$1" pin="PF1/OSC_OUT"/>
+<pinref part="IC1" gate="G$1" pin="PF1/OSC_OUT"/>
 <wire x1="370.84" y1="53.34" x2="383.54" y2="53.34" width="0.1524" layer="91"/>
 </segment>

Commit message: changed testpoints to unpopulated resistors
Parts:
- removed TP1, TP2, TP3, TP5: PTR1TP13R, nixx:PTR1TP13R
- added R20, R21, R22, R23, R24: 10K, joyAnalog:RESISTOR0805-RES
Connections:
- new net N$20: IC1.PA1, R20.2
- net +3V3: now also R20.1, R21.1, R22.1, R23.2, R24.2
- net N$14: now also R22.2; no longer TP2.TP
- net N$16: now also R23.1; no longer TP3.TP
- net N$17: now also R24.1; no longer TP5.TP
- net STM_5: no longer IC1.PA1
- net TX: now also R21.2; no longer TP1.TP
Changed lines of the file:
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@@
 <part name="R19" library="joyAnalog" deviceset="RESISTOR" device="0805-RES" value="68K"/>
 <part name="JP3" library="SparkFun-Jumpers" deviceset="JUMPER-SMT_2_NO" device="_NO-SILK"/>
-<part name="TP1" library="nixx" deviceset="PTR1" device="TP13R"/>
 <part name="R12" library="joyAnalog" deviceset="RESISTOR" device="0805-RES" value="10K"/>
 <part name="R17" library="joyAnalog" deviceset="RESISTOR" device="0805-RES" value="10K"/>
 <part name="GND12" library="joyAnalog" deviceset="GND" device=""/>
-<part name="TP2" library="nixx" deviceset="PTR1" device="TP13R"/>
-<part name="TP3" library="nixx" deviceset="PTR1" device="TP13R"/>
-<part name="TP5" library="nixx" deviceset="PTR1" device="TP13R"/>
+<part name="R20" library="joyAnalog" deviceset="RESISTOR" device="0805-RES" value="10K"/>
+<part name="+3V5" library="joyAnalog" deviceset="+3V3" device=""/>
+<part name="R21" library="joyAnalog" deviceset="RESISTOR" device="0805-RES" value="10K"/>
+<part name="+3V7" library="joyAnalog" deviceset="+3V3" device=""/>
+<part name="R22" library="joyAnalog" deviceset="RESISTOR" device="0805-RES" value="10K"/>
+<part name="+3V8" library="joyAnalog" deviceset="+3V3" device=""/>
+<part name="R23" library="joyAnalog" deviceset="RESISTOR" device="0805-RES" value="10K"/>
+<part name="R24" library="joyAnalog" deviceset="RESISTOR" device="0805-RES" value="10K"/>
+<part name="+3V9" library="joyAnalog" deviceset="+3V3" device=""/>
+<part name="+3V10" library="joyAnalog" deviceset="+3V3" device=""/>
 </parts>
 <sheets>
@@
 <instance part="R19" gate="G$1" x="401.32" y="-38.1"/>
 <instance part="JP3" gate="G$1" x="414.02" y="-38.1"/>
-<instance part="TP1" gate="G$1" x="459.74" y="76.2" rot="R90"/>
 <instance part="R12" gate="G$1" x="238.76" y="53.34"/>
 <instance part="R17" gate="G$1" x="439.42" y="33.02" rot="R90"/>
 <instance part="GND12" gate="1" x="439.42" y="25.4"/>
-<instance part="TP2" gate="G$1" x="452.12" y="43.18" rot="R90"/>
-<instance part="TP3" gate="G$1" x="368.3" y="55.88" rot="R270"/>
-<instance part="TP5" gate="G$1" x="368.3" y="53.34" rot="R270"/>
+<instance part="R20" gate="G$1" x="452.12" y="99.06" rot="R180"/>
+<instance part="+3V5" gate="G$1" x="462.28" y="101.6"/>
+<instance part="R21" gate="G$1" x="462.28" y="76.2" rot="R180"/>
+<instance part="+3V7" gate="G$1" x="472.44" y="78.74"/>
+<instance part="R22" gate="G$1" x="454.66" y="43.18" rot="R180"/>
+<instance part="+3V8" gate="G$1" x="467.36" y="45.72"/>
+<instance part="R23" gate="G$1" x="365.76" y="55.88" rot="R180"/>
+<instance part="R24" gate="G$1" x="365.76" y="53.34" rot="R180"/>
+<instance part="+3V9" gate="G$1" x="358.14" y="58.42"/>
+<instance part="+3V10" gate="G$1" x="350.52" y="55.88"/>
 </instances>
 <busses>
@@
 <wire x1="424.18" y1="-45.72" x2="431.8" y2="-45.72" width="0.1524" layer="91"/>
 </segment>
+<segment>
+<pinref part="R20" gate="G$1" pin="1"/>
+<pinref part="+3V5" gate="G$1" pin="+3V3"/>
+<wire x1="457.2" y1="99.06" x2="462.28" y2="99.06" width="0.1524" layer="91"/>
+</segment>
+<segment>
+<pinref part="+3V9" gate="G$1" pin="+3V3"/>
+<pinref part="R23" gate="G$1" pin="2"/>
+<wire x1="358.14" y1="55.88" x2="360.68" y2="55.88" width="0.1524" layer="91"/>
+</segment>
+<segment>
+<pinref part="+3V10" gate="G$1" pin="+3V3"/>
+<pinref part="R24" gate="G$1" pin="2"/>
+<wire x1="350.52" y1="53.34" x2="360.68" y2="53.34" width="0.1524" layer="91"/>
+</segment>
+<segment>
+<pinref part="R22" gate="G$1" pin="1"/>
+<pinref part="+3V8" gate="G$1" pin="+3V3"/>
+<wire x1="459.74" y1="43.18" x2="467.36" y2="43.18" width="0.1524" layer="91"/>
+</segment>
+<segment>
+<pinref part="R21" gate="G$1" pin="1"/>
+<pinref part="+3V7" gate="G$1" pin="+3V3"/>
+<wire x1="467.36" y1="76.2" x2="472.44" y2="76.2" width="0.1524" layer="91"/>
+</segment>
 </net>
 <net name="SPI_SCK" class="0">
@@
 </segment>
 <segment>
-<pinref part="IC1" gate="G$1" pin="PA1"/>
-<wire x1="452.12" y1="99.06" x2="424.18" y2="99.06" width="0.1524" layer="91"/>
-<label x="426.72" y="99.06" size="1.778" layer="95"/>
 <pinref part="IC1" gate="G$1" pin="PA4"/>
-<wire x1="452.12" y1="99.06" x2="452.12" y2="91.44" width="0.1524" layer="91"/>
-<wire x1="452.12" y1="91.44" x2="424.18" y2="91.44" width="0.1524" layer="91"/>
+<wire x1="439.42" y1="91.44" x2="424.18" y2="91.44" width="0.1524" layer="91"/>
+<label x="426.72" y="91.44" size="1.778" layer="95"/>
 </segment>
 </net>
@@
 <segment>
 <pinref part="IC1" gate="G$1" pin="PA9"/>
-<pinref part="TP1" gate="G$1" pin="TP"/>
 <wire x1="457.2" y1="76.2" x2="424.18" y2="76.2" width="0.1524" layer="91"/>
 <label x="447.04" y="76.2" size="1.778" layer="95"/>
+<pinref part="R21" gate="G$1" pin="2"/>
 </segment>
 </net>
@@
 <pinref part="IC1" gate="G$1" pin="PB6"/>
 <wire x1="424.18" y1="43.18" x2="449.58" y2="43.18" width="0.1524" layer="91"/>
-<pinref part="TP2" gate="G$1" pin="TP"/>
+<pinref part="R22" gate="G$1" pin="2"/>
 </segment>
 </net>
@@
 <pinref part="IC1" gate="G$1" pin="PF0/OSC_IN"/>
 <wire x1="370.84" y1="55.88" x2="383.54" y2="55.88" width="0.1524" layer="91"/>
-<pinref part="TP3" gate="G$1" pin="TP"/>
+<pinref part="R23" gate="G$1" pin="1"/>
 </segment>
 </net>
 <net name="N$17" class="0">
 <segment>
-<pinref part="TP5" gate="G$1" pin="TP"/>
 <pinref part="IC1" gate="G$1" pin="PF1/OSC_OUT"/>
 <wire x1="370.84" y1="53.34" x2="383.54" y2="53.34" width="0.1524" layer="91"/>
-</segment>
-</net>
+<pinref part="R24" gate="G$1" pin="1"/>
+</segment>
+</net>
+<net name="N$20" class="0">
+<segment>
+<pinref part="IC1" gate="G$1" pin="PA1"/>
+<wire x1="424.18" y1="99.06" x2="447.04" y2="99.06" width="0.1524" layer="91"/>
+<pinref part="R20" gate="G$1" pin="2"/>
+</segment>
+</net>

Commit message: adjusted more values
Parts:
- C1: value 1uF -> 100nF
Changed lines of the file:
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@@
 <part name="P+1" library="nixx" deviceset="+180V" device=""/>
 <part name="R1" library="joyAnalog" deviceset="RESISTOR" device="0805-RES" value="10K"/>
-<part name="C1" library="joyAnalog" deviceset="CAP" device="0805" value="1uF"/>
+<part name="C1" library="joyAnalog" deviceset="CAP" device="0805" value="100nF"/>
 <part name="GND1" library="joyAnalog" deviceset="GND" device=""/>
 <part name="Q2" library="nixx" deviceset="BF820" device=""/>
