File: pcb/exixe14.brd (EAGLE design)
At the start: 20 x 40 mm, 51 parts

Commit message: adjusted values
Parts:
- R14, R16: value 470 -> 330
- R15: value 1K -> 680
- R23: value 100K -> 68K
Changed lines of the file:
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@@
 <attribute name="NAME" x="6.731" y="34.7599" size="0.7112" layer="25" font="vector" rot="R180"/>
 </element>
-<element name="R14" library="joyAnalog" package="0805" value="470" x="17.399" y="6.731" smashed="yes" rot="R270">
+<element name="R14" library="joyAnalog" package="0805" value="330" x="17.399" y="6.731" smashed="yes" rot="R270">
 <attribute name="NAME" x="16.3195" y="8.255" size="0.8128" layer="25" font="vector" rot="R90"/>
 </element>
-<element name="R15" library="joyAnalog" package="0805" value="1K" x="3.048" y="4.953" smashed="yes">
+<element name="R15" library="joyAnalog" package="0805" value="680" x="3.048" y="4.953" smashed="yes">
 <attribute name="NAME" x="2.9718" y="5.8293" size="0.8128" layer="25" font="vector"/>
 </element>
-<element name="R16" library="joyAnalog" package="0805" value="470" x="19.05" y="6.731" smashed="yes" rot="R270">
+<element name="R16" library="joyAnalog" package="0805" value="330" x="19.05" y="6.731" smashed="yes" rot="R270">
 <attribute name="NAME" x="17.3863" y="8.2804" size="0.8128" layer="25" font="vector" rot="R90"/>
 </element>
@@
 <attribute name="NAME" x="7.62" y="39.6875" size="0.6096" layer="25" rot="R180"/>
 </element>
-<element name="R23" library="joyAnalog" package="0805" value="100K" x="8.255" y="36.703" smashed="yes" rot="R90">
+<element name="R23" library="joyAnalog" package="0805" value="68K" x="8.255" y="36.703" smashed="yes" rot="R90">
 <attribute name="NAME" x="8.9662" y="35.2425" size="0.6096" layer="25" rot="R180"/>
 </element>

Commit message: adjust passive values and added bom
Parts:
- R20, R21: value 510K -> 68K
- R6: value 4K7 -> 10K
Changed lines of the file:
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@@
 <?xml version="1.0" encoding="utf-8"?>
 <!DOCTYPE eagle SYSTEM "eagle.dtd">
-<eagle version="8.2.2">
+<eagle version="8.3.2">
 <drawing>
 <settings>
 <setting alwaysvectorfont="yes"/>
+<setting keepoldvectorfont="yes"/>
 <setting verticaltext="up"/>
 </settings>
@@
 <attribute name="VALUE" x="13.014" y="29.927" size="1.016" layer="27" rot="R90"/>
 </element>
-<element name="R6" library="joyAnalog" package="0805" value="4K7" x="14.127" y="27.708" smashed="yes" rot="R90">
+<element name="R6" library="joyAnalog" package="0805" value="10K" x="14.127" y="27.708" smashed="yes" rot="R90">
 <attribute name="NAME" x="14.8925" y="29.7214" size="0.8128" layer="25" font="vector" rot="R270"/>
 </element>
@@
 <attribute name="VALUE" x="9.144" y="12.192" size="0.0254" layer="28" rot="MR0"/>
 </element>
-<element name="R20" library="joyAnalog" package="0805" value="510K" x="13.97" y="18.288" smashed="yes" rot="MR180">
+<element name="R20" library="joyAnalog" package="0805" value="68K" x="13.97" y="18.288" smashed="yes" rot="MR180">
 <attribute name="NAME" x="15.494" y="18.6309" size="0.8128" layer="26" rot="MR180"/>
 </element>
-<element name="R21" library="joyAnalog" package="0805" value="510K" x="6.223" y="18.034" smashed="yes" rot="MR180">
+<element name="R21" library="joyAnalog" package="0805" value="68K" x="6.223" y="18.034" smashed="yes" rot="MR180">
 <attribute name="NAME" x="5.461" y="17.2085" size="0.8128" layer="26" rot="MR180"/>
 </element>
