File: pcb/exixe14.sch (EAGLE design)
At the start: 50 parts, among them IC1 STM32F042K6

Commit message: adjusted values
Parts:
- C1: value 1uF -> 100nF
Changed lines of the file:
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@@
 <part name="P+1" library="nixx" deviceset="+180V" device=""/>
 <part name="R1" library="joyAnalog" deviceset="RESISTOR" device="0805-RES" value="10K"/>
-<part name="C1" library="joyAnalog" deviceset="CAP" device="0805" value="1uF"/>
+<part name="C1" library="joyAnalog" deviceset="CAP" device="0805" value="100nF"/>
 <part name="GND1" library="joyAnalog" deviceset="GND" device=""/>
 <part name="Q2" library="nixx" deviceset="BF820" device=""/>
