File: pogo_rig/pcb/exixe_pogo.sch (EAGLE design)
At the start: 14 parts, among them X1 USB-MICROB

Commit message: working on pogo rig
Parts:
- added C1, C2: (no value), clock:CAP0805
- added C3, C4: (no value), clock:C-USC1210
- added IC1: REG1117, clock:REG1117
- added IC2: STM32F030F4, stm32f030f4:STM32F030F4
- added JP3, JP4: (no value), clock:PINHD-1X4/90
- added LED1, LED2: (no value), clock:LEDCHIP-LED0805
- added R1: (no value), clock:RESISTOR0805-RES
- added S1, S2: TAC_SWITCHSMD, clock:TAC_SWITCHSMD
- added U$11, U$12, U$13, U$14: M3_MOUNTING_HOLE, clock:M3_MOUNTING_HOLE
Connections:
- new net +3V3: C1.1, C2.1, C3.1, IC1.VOUT, IC2.VDD, IC2.VDDA, JP3.2, JP4.2, LED1.A, U$1.3V, U$2.3V
- new net +5V: C4.1, IC1.VIN, X1.VBUS
- new net CS: IC2.PA4, U$1.CS, U$2.CS
- new net EXIXE_RST: U$1.RST, U$2.RST
- new net GND: C1.2, C2.2, C3.2, C4.2, IC1.GND, IC2.BOOT0, IC2.VSS, JP3.1, JP4.1, R1.2, U$1.GND, U$2.GND, X1.GND
- new net MISO: IC2.PA6, U$1.MISO, U$2.MISO
- new net MOSI: IC2.PA7, U$1.MOSI, U$2.MOSI
- new net N$1: N1.1, U$1.DIGIT1, U$2.DIGIT1
- new net N$10: N1.9, U$1.DIGIT9, U$2.DIGIT9
- new net N$11: N1.0, U$1.DIGIT0, U$2.DIGIT0
- new net N$12: N1.RHDP, U$2.DOT_RIGHT
- new net N$13: N1.LHDP, U$1.DOT_LEFT, U$2.DOT_LEFT
- new net N$14: N1.A, U$1.ANODE, U$2.ANODE
- new net N$15: LED1.C, R1.1
- new net N$2: IC2.NRST, S1.3
- new net N$3: N1.2, U$1.DIGIT2, U$2.DIGIT2
- new net N$4: N1.3, U$1.DIGIT3, U$2.DIGIT3
- new net N$5: N1.4, U$1.DIGIT4, U$2.DIGIT4
- new net N$6: N1.5, U$1.DIGIT5, U$2.DIGIT5
- new net N$7: N1.6, U$1.DIGIT6, U$2.DIGIT6
- new net N$8: N1.7, U$1.DIGIT7, U$2.DIGIT7
- new net N$9: N1.8, U$1.DIGIT8, U$2.DIGIT8
- new net RX: IC2.PA3
- new net SCK: IC2.PA5, U$1.SCK, U$2.SCK
- new net SWCLK: IC2.PA14
- new net SWDIO: IC2.PA13
- new net TX: IC2.PA2
Other:
- note added: "HV enable siignal HV indicator LED HV pullup resistor"
- moved on the sheet: N1

Commit message: working on pogo board
Parts:
- added R2, R3: (no value), clock:RESISTOR0805-RES
- added U$15, U$16, U$17, U$18: M3_MOUNTING_HOLE, clock:M3_MOUNTING_HOLE
Connections:
- new net +180V: JP1.HV, JP2.HV, U$1.HV, U$2.HV
- new net EXIXE_SWCLK: JP3.3, U$1.CLK, U$2.CLK
- new net EXIXE_SWDIO: JP3.4, U$1.DIO, U$2.DIO
- new net HV_EN: IC2.PA10, JP1.EN, JP2.EN, R3.1
- new net N$16: IC2.PA0, LED1.A
- new net N$18: LED2.C, R2.1
- new net N$19: IC2.PA9, LED2.A
- new net USER_BUTTON: IC2.PB1, S2.1
- net +3V3: no longer JP4.2, LED1.A
- net +5V: now also JP1.5V, JP2.5V, R3.2
- net EXIXE_RST: now also IC2.PA1
- net GND: now also JP1.GND, JP2.GND, R2.2, S1.1, S1.2, S2.3; no longer JP4.1
- net RX: now also JP4.2
- net SWCLK: now also JP4.3
- net SWDIO: now also JP4.4
- net TX: now also JP4.1
Other:
- moved on the sheet: JP1, JP2, JP4, LED1, LED2, N1, R1, S2

Commit message: pogo rig mostly finished
Parts:
- added JP5: (no value), pinhead:PINHD-1X2
- added JP6, JP7: (no value), pinhead:PINHD-1X6
- added LED3: (no value), clock:LEDCHIP-LED0805
- added R4, R5: (no value), clock:RESISTOR0805-RES
- added TP1, TP10, TP11, TP2, TP3, TP4, TP5, TP6, TP7, TP8, TP9: TEST-POINT3X5, clock:TEST-POINT3X5
- JP3, JP4: device clock:PINHD-1X4/90 -> pinhead:PINHD-1X4
Connections:
- new net N$17: JP5.1, R4.1
- new net N$20: IC2.PF0/OSC_IN, TP1.1
- new net N$21: IC2.PF1/OSC_OUT, TP2.1
- new net N$22: TP4.1, U$1.PF1
- new net N$23: TP5.1, U$1.PB6
- new net N$24: TP6.1, U$1.PA9
- new net N$25: TP7.1, U$1.PA1
- new net N$26: TP8.1, U$2.PF0
- new net N$27: TP9.1, U$2.PF1
- new net N$28: TP10.1, U$2.PB3
- new net N$29: TP11.1, U$2.TX
- new net N$30: TP3.1, U$1.PF0
- new net N$31: LED3.C, R5.1
- net +180V: now also R4.2
- net +3V3: now also JP6.1, JP7.1, LED3.A
- net GND: now also JP5.2, JP6.6, JP7.6, R5.2
