File: pogo_rig/pcb/exixe_pogo.sch (EAGLE design)
At the start: 44 parts, among them IC1 REG1117, IC2 STM32F030F4, SW2 324_SW324_SWITCH_FOOT_HOLE, U1 USBC_16P_CENTERED

Commit message: updated pogo rig
Parts:
- C4: device clock:C-USC1210 -> clock:CAP0805
Changed lines of the file:
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@@
 <part name="C1" library="clock" deviceset="CAP" device="0805"/>
 <part name="C2" library="clock" deviceset="CAP" device="0805"/>
-<part name="C4" library="clock" deviceset="C-US" device="C1210"/>
 <part name="P+1" library="clock" deviceset="+5V" device=""/>
 <part name="LED1" library="clock" deviceset="LED" device="CHIP-LED0805"/>
@@
 <part name="+3V5" library="supply1" library_urn="urn:adsk.eagle:library:371" deviceset="+3V3" device=""/>
 <part name="SW2" library="3pos_slide_switch" deviceset="324_SW" device="324_SWITCH_FOOT_HOLE" value="324_SW324_SWITCH_FOOT_HOLE"/>
+<part name="C4" library="clock" deviceset="CAP" device="0805"/>
 </parts>
 <sheets>
@@
 <instance part="C1" gate="G$1" x="157.48" y="-129.54"/>
 <instance part="C2" gate="G$1" x="167.64" y="-129.54"/>
-<instance part="C4" gate="G$1" x="106.68" y="-127"/>
 <instance part="P+1" gate="1" x="76.2" y="-121.92"/>
 <instance part="LED1" gate="G$1" x="127" y="-68.58" rot="R90"/>
@@
 <instance part="+3V5" gate="G$1" x="30.48" y="-104.14"/>
 <instance part="SW2" gate="G$1" x="5.08" y="-104.14"/>
+<instance part="C4" gate="G$1" x="106.68" y="-129.54"/>
 </instances>
 <busses>
@@
 <pinref part="IC1" gate="G$1" pin="GND"/>
 <pinref part="GND2" gate="1" pin="GND"/>
-</segment>
-<segment>
-<pinref part="C4" gate="G$1" pin="2"/>
-<pinref part="GND3" gate="1" pin="GND"/>
 </segment>
 <segment>
@@
 <pinref part="GND9" gate="1" pin="GND"/>
 </segment>
+<segment>
+<pinref part="GND3" gate="1" pin="GND"/>
+<pinref part="C4" gate="G$1" pin="2"/>
+</segment>
 </net>
