File: pogo_rig/pcb/exixe_pogo.brd (EAGLE design)
At the start: 90 x 60 mm, 44 parts, among them IC1 REG1117, IC2 STM32F030F4, SW2 324_SW324_SWITCH_FOOT_HOLE, U1 USBC_16P_CENTERED

Commit message: updated pogo rig
Parts:
- C4: device clock:C1210 -> clock:0805
- moved C4 2.40 mm to (38.4, 10.2), turned to 180 degrees
Routing:
- net GND: track 5.02 -> 13.6 mm
- net +5V: track 63.9 -> 61.4 mm
Other:
- board text added: "DFU"
Changed lines of the file:
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@@
 <rectangle x1="35.433" y1="37.338" x2="36.703" y2="59.563" layer="42"/>
 <rectangle x1="35.4584" y1="57.7088" x2="65.9384" y2="59.4868" layer="42"/>
-<rectangle x1="64.262" y1="49.022" x2="66.421" y2="59.69" layer="42"/>
+<rectangle x1="63.881" y1="47.8282" x2="66.8274" y2="59.7662" layer="42"/>
 <rectangle x1="20.32" y1="53.2892" x2="35.7378" y2="54.9402" layer="42"/>
 <rectangle x1="35.433" y1="36.957" x2="40.894" y2="38.735" layer="42"/>
-<rectangle x1="7.62" y1="46.863" x2="11.049" y2="52.197" layer="42"/>
+<rectangle x1="7.6708" y1="47.5742" x2="11.0998" y2="52.9082" layer="42"/>
 <rectangle x1="38.481" y1="30.988" x2="43.815" y2="40.132" layer="42"/>
 <rectangle x1="38.862" y1="35.941" x2="41.021" y2="39.751" layer="41"/>
@@
 <text x="36.576" y="19.431" size="1.27" layer="25" rot="R180">RST</text>
 <text x="56.515" y="19.431" size="1.27" layer="25" rot="R180">PB1</text>
-<text x="73.025" y="22.4536" size="1.4224" layer="26" rot="MR180" align="center">exixe pogo v2
+<text x="55.499" y="14.859" size="1.4224" layer="26" rot="MR180" align="center">exixe pogo v2
 dekuNukem
 JUN2019</text>
@@
 <rectangle x1="9.6012" y1="49.3522" x2="18.2372" y2="51.0032" layer="42"/>
 <rectangle x1="16.0782" y1="51.4604" x2="22.8346" y2="53.1114" layer="42" rot="R45"/>
+<text x="30.4292" y="31.1912" size="1.27" layer="25" rot="R45">DFU</text>
 </plain>
 <attributes>
@@
 <param name="rvMicroViaInner" value="0.25"/>
 <param name="rlMinPadTop" value="7mil"/>
-<param name="rlMaxPadTop" value="8mil"/>
+<param name="rlMaxPadTop" value="7mil"/>
 <param name="rlMinPadInner" value="7mil"/>
 <param name="rlMaxPadInner" value="8mil"/>
@@
 <attribute name="VALUE" x="50.546" y="22.4282" size="0.4064" layer="27"/>
 </element>
-<element name="C4" library="clock" package="C1210" value="" x="37.7962" y="7.8276" smashed="yes" rot="R270">
-<attribute name="NAME" x="37.3082" y="4.192" size="0.8128" layer="25"/>
-</element>
 <element name="LED1" library="clock" package="CHIP-LED0805" value="" x="29.972" y="26.289" smashed="yes" rot="R90">
 <attribute name="VALUE" x="31.242" y="28.829" size="1.27" layer="27" rot="R180"/>
@@
 </element>
 <element name="SW2" library="3pos_slide_switch" package="342_SWICH_FOOT_HOLE" value="324_SW324_SWITCH_FOOT_HOLE" x="32.893" y="30.7594" rot="R225"/>
+<element name="C4" library="clock" package="0805" value="" x="38.354" y="10.16" rot="R180"/>
 </elements>
 <signals>
 <signal name="GND">
 <contactref element="IC1" pad="1"/>
-<contactref element="C4" pad="2"/>
 <contactref element="C3" pad="2"/>
 <polygon width="0.2032" layer="1" isolate="0.3048">
@@
 <wire x1="47.9178" y1="22.675" x2="51.3118" y2="22.675" width="0.2032" layer="1"/>
 <wire x1="51.3118" y1="22.675" x2="52.462" y2="23.8252" width="0.2032" layer="1"/>
-<wire x1="41.772" y1="10.16" x2="41.775" y2="7.6975" width="0" layer="19" extent="1-1"/>
+<contactref element="C4" pad="2"/>
+<wire x1="41.8504" y1="16.8306" x2="42.4276" y2="16.8306" width="0.1524" layer="1"/>
+<wire x1="42.4276" y1="16.8306" x2="43.5102" y2="15.748" width="0.1524" layer="1"/>
+<wire x1="43.5102" y1="15.748" x2="43.5102" y2="11.6586" width="0.1524" layer="1"/>
+<wire x1="42.0116" y1="10.16" x2="41.772" y2="10.16" width="0.1524" layer="1"/>
+<wire x1="43.5102" y1="11.6586" x2="42.0116" y2="10.16" width="0.1524" layer="1"/>
 </signal>
 <signal name="+5V">
 <contactref element="IC1" pad="3"/>
-<contactref element="C4" pad="1"/>
 <contactref element="JP1" pad="5V"/>
 <contactref element="JP2" pad="5V"/>
@@
 <contactref element="U1" pad="A4B9"/>
 <contactref element="U1" pad="B4A9"/>
-<wire x1="42.575" y1="7.6975" x2="42.575" y2="8.6822" width="0.4064" layer="1"/>
-<wire x1="42.575" y1="8.6822" x2="42.291" y2="8.9662" width="0.4064" layer="1"/>
-<wire x1="42.291" y1="8.9662" x2="38.0576" y2="8.9662" width="0.4064" layer="1"/>
-<wire x1="38.0576" y1="8.9662" x2="37.7962" y2="9.2276" width="0.4064" layer="1"/>
-<wire x1="37.7962" y1="9.2276" x2="37.7962" y2="10.3642" width="0.4064" layer="1"/>
-<wire x1="37.7962" y1="10.3642" x2="39.624" y2="12.192" width="0.4064" layer="1"/>
 <wire x1="47.425" y1="7.6975" x2="47.425" y2="6.8358" width="0.3048" layer="1"/>
 <wire x1="47.425" y1="6.8358" x2="46.5074" y2="5.9182" width="0.3048" layer="1"/>
@@
 <wire x1="42.575" y1="6.828" x2="42.575" y2="7.6975" width="0.3048" layer="1"/>
 <wire x1="43.4848" y1="5.9182" x2="42.575" y2="6.828" width="0.3048" layer="1"/>
+<contactref element="C4" pad="1"/>
+<wire x1="42.575" y1="7.6975" x2="42.575" y2="8.8092" width="0.3048" layer="1"/>
+<wire x1="42.575" y1="8.8092" x2="42.3672" y2="9.017" width="0.3048" layer="1"/>
+<wire x1="42.3672" y1="9.017" x2="40.397" y2="9.017" width="0.3048" layer="1"/>
+<wire x1="40.397" y1="9.017" x2="39.254" y2="10.16" width="0.3048" layer="1"/>
+<wire x1="39.254" y1="10.16" x2="39.254" y2="11.822" width="0.3048" layer="1"/>
+<wire x1="39.254" y1="11.822" x2="39.624" y2="12.192" width="0.3048" layer="1"/>
 </signal>
 <signal name="+3V3">
@@
 <via x="40.5638" y="24.2062" extent="1-16" drill="0.5"/>
 <via x="39.37" y="16.9164" extent="1-16" drill="0.5"/>
-<wire x1="37.78" y1="16.891" x2="37.794" y2="16.905" width="0.2032" layer="1"/>
 <wire x1="42.0822" y1="23.975" x2="40.795" y2="23.975" width="0.2032" layer="1"/>
 <wire x1="40.795" y1="23.975" x2="40.5638" y2="24.2062" width="0.2032" layer="1"/>
@@
 <wire x1="48.1076" y1="46.482" x2="39.9075" y2="46.482" width="0.2032" layer="16"/>
 <wire x1="39.9075" y1="46.482" x2="39.9058" y2="46.4837" width="0.2032" layer="16"/>
-<wire x1="69.0825" y1="30.4825" x2="66.7995" y2="30.4825" width="0.2032" layer="16"/>
-<wire x1="52.324" y1="44.958" x2="49.6316" y2="44.958" width="0.2032" layer="16"/>
+<wire x1="69.0825" y1="30.4825" x2="66.4693" y2="30.4825" width="0.2032" layer="16"/>
+<wire x1="51.9938" y1="44.958" x2="49.6316" y2="44.958" width="0.2032" layer="16"/>
 <wire x1="49.6316" y1="44.958" x2="48.1076" y2="46.482" width="0.2032" layer="16"/>
-<wire x1="66.7995" y1="30.4825" x2="52.324" y2="44.958" width="0.2032" layer="16"/>
+<wire x1="66.4693" y1="30.4825" x2="51.9938" y2="44.958" width="0.2032" layer="16"/>
 <wire x1="39.855" y1="46.4837" x2="28.6265" y2="35.2552" width="0.2032" layer="1"/>
 <wire x1="28.6265" y1="35.2552" x2="25.6032" y2="35.2552" width="0.2032" layer="1"/>
@@
 <contactref element="U$2" pad="DIGIT_2"/>
 <wire x1="38.8552" y1="49.2539" x2="32.0327" y2="49.2539" width="0.2032" layer="1"/>
-<wire x1="67.4" y1="33.8" x2="62.2364" y2="38.9636" width="0.2032" layer="16"/>
-<wire x1="62.2364" y1="38.9636" x2="59.3852" y2="38.9636" width="0.2032" layer="16"/>
-<wire x1="59.3852" y1="38.9636" x2="49.0949" y2="49.2539" width="0.2032" layer="16"/>
-<wire x1="49.0949" y1="49.2539" x2="38.8552" y2="49.2539" width="0.2032" layer="16"/>
+<wire x1="67.4" y1="33.8" x2="62.465" y2="38.735" width="0.2032" layer="16"/>
+<wire x1="62.465" y1="38.735" x2="59.2582" y2="38.735" width="0.2032" layer="16"/>
+<wire x1="59.2582" y1="38.735" x2="48.7393" y2="49.2539" width="0.2032" layer="16"/>
+<wire x1="48.7393" y1="49.2539" x2="38.8552" y2="49.2539" width="0.2032" layer="16"/>
 <wire x1="32.0327" y1="49.2539" x2="24.4602" y2="41.6814" width="0.2032" layer="1"/>
 <via x="24.4348" y="41.6814" extent="1-16" drill="0.5"/>
@@
 <wire x1="24.4348" y1="43.3324" x2="21.971" y2="45.7962" width="0.2032" layer="16"/>
 <wire x1="21.971" y1="45.7962" x2="19.0246" y2="45.7962" width="0.2032" layer="16"/>
-<wire x1="19.0246" y1="45.7962" x2="18.288" y2="46.5328" width="0.2032" layer="16"/>
-<wire x1="18.288" y1="46.5328" x2="13.6652" y2="46.5328" width="0.2032" layer="16"/>
-<wire x1="13.6652" y1="46.5328" x2="8.7122" y2="41.5798" width="0.2032" layer="16"/>
+<wire x1="19.0246" y1="45.7962" x2="18.1356" y2="46.6852" width="0.2032" layer="16"/>
+<wire x1="18.1356" y1="46.6852" x2="13.8176" y2="46.6852" width="0.2032" layer="16"/>
+<wire x1="13.8176" y1="46.6852" x2="8.7122" y2="41.5798" width="0.2032" layer="16"/>
 <wire x1="8.7122" y1="41.5798" x2="8.7122" y2="38.7779" width="0.2032" layer="16"/>
 <wire x1="8.7122" y1="38.7779" x2="10.8552" y2="36.6349" width="0.2032" layer="16"/>
@@
 <wire x1="22.9362" y1="43.4848" x2="21.1074" y2="45.3136" width="0.2032" layer="16"/>
 <wire x1="21.1074" y1="45.3136" x2="18.4658" y2="45.3136" width="0.2032" layer="16"/>
-<wire x1="18.4658" y1="45.3136" x2="17.7038" y2="46.0756" width="0.2032" layer="16"/>
-<wire x1="14.1986" y1="46.0756" x2="10.922" y2="42.799" width="0.2032" layer="16"/>
+<wire x1="18.4658" y1="45.3136" x2="17.6784" y2="46.101" width="0.2032" layer="16"/>
+<wire x1="14.224" y1="46.101" x2="10.922" y2="42.799" width="0.2032" layer="16"/>
 <wire x1="10.922" y1="42.799" x2="10.922" y2="39.8663" width="0.2032" layer="16"/>
 <wire x1="10.922" y1="39.8663" x2="11.2123" y2="39.576" width="0.2032" layer="16"/>
 <wire x1="32.9926" y1="52.195" x2="24.2824" y2="43.4848" width="0.2032" layer="1"/>
-<wire x1="17.7038" y1="46.0756" x2="14.1986" y2="46.0756" width="0.2032" layer="16"/>
+<wire x1="17.6784" y1="46.101" x2="14.224" y2="46.101" width="0.2032" layer="16"/>
 </signal>
 <signal name="N$5">
@@
 <wire x1="28.7782" y1="32.893" x2="24.5872" y2="32.893" width="0.2032" layer="1"/>
 <via x="24.5872" y="32.893" extent="1-16" drill="0.5"/>
-<wire x1="24.5872" y1="32.893" x2="20.7264" y2="29.0322" width="0.2032" layer="16"/>
-<wire x1="20.7264" y1="29.0322" x2="15.3924" y2="29.0322" width="0.2032" layer="16"/>
-<wire x1="15.3924" y1="29.0322" x2="14.123" y2="30.3016" width="0.2032" layer="16"/>
+<wire x1="24.5872" y1="32.893" x2="20.9296" y2="29.2354" width="0.2032" layer="16"/>
+<wire x1="20.9296" y1="29.2354" x2="15.1892" y2="29.2354" width="0.2032" layer="16"/>
+<wire x1="15.1892" y1="29.2354" x2="14.123" y2="30.3016" width="0.2032" layer="16"/>
 <wire x1="14.123" y1="30.3016" x2="14.123" y2="31.8997" width="0.2032" layer="16"/>
 </signal>
