File: pcb/exixe12/exixe12.sch (EAGLE design)
At the start: 43 parts, among them IC1 STM32F042K6

Commit message: removed DP resistor, new pogo firmware
Parts:
- removed R12: 10K, joyAnalog:RESISTOR0805-RES
Connections:
- removed net N$22: Q11.C, R12.1
- net NIXIE_DOT_LEFT: now also Q11.C; no longer R12.2
Changed lines of the file:
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@@
 <?xml version="1.0" encoding="utf-8"?>
 <!DOCTYPE eagle SYSTEM "eagle.dtd">
-<eagle version="8.3.2">
+<eagle version="9.1.3">
 <drawing>
 <settings>
-<setting alwaysvectorfont="no"/>
+<setting alwaysvectorfont="yes"/>
 <setting keepoldvectorfont="yes"/>
 <setting verticaltext="up"/>
@@
 <part name="R19" library="joyAnalog" deviceset="RESISTOR" device="0805-RES" value="68K"/>
 <part name="JP3" library="SparkFun-Jumpers" deviceset="JUMPER-SMT_2_NO" device="_NO-SILK"/>
-<part name="R12" library="joyAnalog" deviceset="RESISTOR" device="0805-RES" value="10K"/>
 <part name="R17" library="joyAnalog" deviceset="RESISTOR" device="0805-RES" value="10K"/>
 <part name="GND12" library="joyAnalog" deviceset="GND" device=""/>
@@
 <instance part="R19" gate="G$1" x="401.32" y="-38.1"/>
 <instance part="JP3" gate="G$1" x="414.02" y="-38.1"/>
-<instance part="R12" gate="G$1" x="238.76" y="53.34"/>
 <instance part="R17" gate="G$1" x="439.42" y="33.02" rot="R90"/>
 <instance part="GND12" gate="1" x="439.42" y="25.4"/>
@@
 <label x="238.76" y="-20.32" size="1.778" layer="95"/>
 <pinref part="N1" gate="G$1" pin="LHDP"/>
-<pinref part="R12" gate="G$1" pin="2"/>
-<wire x1="243.84" y1="53.34" x2="248.92" y2="53.34" width="0.1524" layer="91"/>
 <wire x1="248.92" y1="53.34" x2="248.92" y2="-20.32" width="0.1524" layer="91"/>
+<pinref part="Q11" gate="A" pin="C"/>
+<wire x1="228.6" y1="53.34" x2="248.92" y2="53.34" width="0.1524" layer="91"/>
 </segment>
 </net>
@@
 </segment>
 </net>
-<net name="N$22" class="0">
-<segment>
-<pinref part="Q11" gate="A" pin="C"/>
-<pinref part="R12" gate="G$1" pin="1"/>
-<wire x1="228.6" y1="53.34" x2="233.68" y2="53.34" width="0.1524" layer="91"/>
-</segment>
-</net>

Commit message: cleanup
Parts:
- removed R18: 10K, joyAnalog:RESISTOR0805-RES
Connections:
- net +3V3: no longer R18.2
- net SPI_CS: no longer R18.1
Changed lines of the file:
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@@
 <part name="R15" library="joyAnalog" deviceset="RESISTOR" device="0805-RES" value="680"/>
 <part name="R16" library="joyAnalog" deviceset="RESISTOR" device="0805-RES" value="330"/>
-<part name="R18" library="joyAnalog" deviceset="RESISTOR" device="0805-RES" value="10K"/>
-<part name="+3V6" library="joyAnalog" deviceset="+3V3" device=""/>
 <part name="N1" library="exixe12" deviceset="IN-12B" device=""/>
 <part name="R19" library="joyAnalog" deviceset="RESISTOR" device="0805-RES" value="68K"/>
@@
 <instance part="R15" gate="G$1" x="495.3" y="7.62"/>
 <instance part="R16" gate="G$1" x="495.3" y="-7.62"/>
-<instance part="R18" gate="G$1" x="347.98" y="-38.1" rot="R90"/>
-<instance part="+3V6" gate="G$1" x="347.98" y="-30.48" rot="MR0"/>
 <instance part="N1" gate="G$1" x="226.06" y="-33.02"/>
 <instance part="R19" gate="G$1" x="401.32" y="-38.1"/>
@@
 </segment>
 <segment>
-<pinref part="R18" gate="G$1" pin="2"/>
-<pinref part="+3V6" gate="G$1" pin="+3V3"/>
-</segment>
-<segment>
 <pinref part="C2" gate="G$1" pin="1"/>
 <pinref part="C1" gate="G$1" pin="1"/>
@@
 <wire x1="307.34" y1="-43.18" x2="330.2" y2="-43.18" width="0.1524" layer="91"/>
 <label x="307.34" y="-43.18" size="1.778" layer="95"/>
-<pinref part="R18" gate="G$1" pin="1"/>
-<wire x1="330.2" y1="-43.18" x2="347.98" y2="-43.18" width="0.1524" layer="91"/>
-<junction x="330.2" y="-43.18"/>
-</segment>
-<segment>
+</segment>
+<segment>
