File: pcb/exixe12/exixe12.brd (EAGLE design)
At the start: 20 x 40 mm, 43 parts, among them IC1 STM32F042K6

Commit message: removed DP resistor, new pogo firmware
Parts:
- removed R12: 10K, joyAnalog:0805
Connections:
- removed net N$22: Q11.3, R12.1
- net NIXIE_DOT_LEFT: now also Q11.3; no longer R12.2
Routing:
- net N$22: track 2.27 -> 0.00 mm, vias 1 -> 0
- net NIXIE_DOT_LEFT: track 4.10 -> 2.39 mm
Changed lines of the file:
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@@
 <setting verticaltext="up"/>
 </settings>
-<grid distance="5" unitdist="mil" unit="mil" style="lines" multiple="1" display="no" altdistance="1" altunitdist="mil" altunit="mil"/>
+<grid distance="2" unitdist="mil" unit="mil" style="lines" multiple="1" display="no" altdistance="1" altunitdist="mil" altunit="mil"/>
 <layers>
 <layer number="1" name="Top" color="4" fill="1" visible="yes" active="yes"/>
@@
 <layer number="43" name="vRestrict" color="2" fill="10" visible="no" active="yes"/>
 <layer number="44" name="Drills" color="7" fill="1" visible="no" active="yes"/>
-<layer number="45" name="Holes" color="7" fill="1" visible="yes" active="yes"/>
+<layer number="45" name="Holes" color="7" fill="1" visible="no" active="yes"/>
 <layer number="46" name="Milling" color="3" fill="1" visible="no" active="yes"/>
 <layer number="47" name="Measures" color="7" fill="1" visible="no" active="yes"/>
@@
 <vertex x="3.5052" y="39.878"/>
 <vertex x="7.9756" y="39.878"/>
-<vertex x="8.4328" y="39.5732"/>
-<vertex x="8.4328" y="35.9156"/>
+<vertex x="8.7376" y="39.369996875"/>
+<vertex x="8.7376" y="36.2966"/>
 <vertex x="8.0264" y="35.4076"/>
 <vertex x="7.366" y="35.4076"/>
 <vertex x="7.0104" y="36.2204"/>
-<vertex x="1.8288" y="36.2204"/>
-<vertex x="0.6604" y="37.4904"/>
+<vertex x="1.6804625" y="36.2204"/>
+<vertex x="0.6604" y="37.329165625"/>
 <vertex x="0.6604" y="39.0144"/>
 <vertex x="1.524" y="39.878"/>
@@
 </element>
 <element name="JP3" library="SparkFun-Jumpers" package="SMT-JUMPER_2_NO_NO-SILK" value="JUMPER-SMT_2_NO_NO-SILK" x="4.445" y="38.862" smashed="yes" rot="R270"/>
-<element name="R12" library="joyAnalog" package="0805" value="10K" x="8.7884" y="20.6756" smashed="yes" rot="MR0">
-<attribute name="NAME" x="9.7028" y="21.5519" size="0.8128" layer="26" rot="MR0"/>
-</element>
 <element name="R17" library="joyAnalog" package="0805" value="10K" x="8.89" y="14.224" smashed="yes" rot="MR0">
 <attribute name="NAME" x="7.112" y="13.843" size="0.8128" layer="26" rot="MR0"/>
@@
 <signal name="NIXIE_DOT_LEFT">
 <contactref element="N1" pad="LHDP"/>
-<contactref element="R12" pad="2"/>
-<wire x1="7.8884" y1="20.6756" x2="7.8884" y2="19.6766" width="0.1524" layer="16"/>
-<wire x1="7.8884" y1="19.6766" x2="10.0825" y2="17.4825" width="0.1524" layer="16"/>
+<contactref element="Q11" pad="3"/>
+<wire x1="11.049" y1="19.4708" x2="10.0825" y2="18.5043" width="0.1524" layer="1"/>
+<wire x1="10.0825" y1="18.5043" x2="10.0825" y2="17.4825" width="0.1524" layer="1"/>
 </signal>
 <signal name="+3V3">
@@
 <via x="12.446" y="9.768" extent="1-16" drill="0.45"/>
 </signal>
-<signal name="N$22">
-<contactref element="Q11" pad="3"/>
-<contactref element="R12" pad="1"/>
-<via x="10.1854" y="19.4708" extent="1-16" drill="0.4"/>
-<wire x1="11.049" y1="19.4708" x2="10.1854" y2="19.4708" width="0.1524" layer="1"/>
-<wire x1="9.6884" y1="20.6756" x2="10.1854" y2="20.1786" width="0.1524" layer="16"/>
-<wire x1="10.1854" y1="20.1786" x2="10.1854" y2="19.4708" width="0.1524" layer="16"/>
-</signal>
 <signal name="N$14">

Commit message: cleanup
Parts:
- removed R18: 10K, joyAnalog:0805
Connections:
- net +3V3: no longer R18.2
- net SPI_CS: no longer R18.1
Routing:
- net SPI_CS: track 16.9 -> 14.9 mm
- net +3V3: track 28.3 -> 27.2 mm, vias 5 -> 4
Changed lines of the file:
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@@
 <attribute name="NAME" x="19.1262" y="12.3063" size="0.8128" layer="25" font="vector" rot="R180"/>
-</element>
-<element name="R18" library="joyAnalog" package="0805" value="10K" x="14.1478" y="16.129" smashed="yes">
-<attribute name="NAME" x="12.4079" y="16.256" size="0.8128" layer="25" font="vector" rot="R90"/>
 </element>
 <element name="N1" library="exixe12" package="IN-12" value="IN-12B" x="10.4" y="26.3" smashed="yes"/>
@@
 </polygon>
 <contactref element="D1" pad="1"/>
-<contactref element="R18" pad="2"/>
 <contactref element="JP1" pad="7"/>
 <via x="4.3688" y="13.7668" extent="1-16" drill="0.4"/>
@@
 <wire x1="14.2926" y1="5.7878" x2="14.3146" y2="5.7658" width="0.254" layer="1"/>
 <via x="10.668" y="29.3624" extent="1-16" drill="0.45"/>
-<via x="15.0368" y="15.0368" extent="1-16" drill="0.5"/>
-<wire x1="15.0478" y1="16.129" x2="15.0478" y2="15.0478" width="0.1524" layer="1"/>
-<wire x1="15.0478" y1="15.0478" x2="15.0368" y2="15.0368" width="0.1524" layer="1"/>
 <wire x1="4.3688" y1="13.7668" x2="5.4212" y2="13.7668" width="0.3048" layer="1"/>
 <wire x1="5.4212" y1="13.7668" x2="5.5118" y2="13.8574" width="0.3048" layer="1"/>
@@
 <signal name="SPI_CS">
 <contactref element="JP2" pad="5"/>
-<contactref element="R18" pad="1"/>
 <contactref element="IC1" pad="25"/>
 <via x="14.5288" y="14.0208" extent="1-16" drill="0.5"/>
-<wire x1="14.257" y1="14.2926" x2="12.8" y2="14.2926" width="0.1524" layer="1"/>
 <wire x1="14.257" y1="14.2926" x2="14.5288" y2="14.0208" width="0.1524" layer="1"/>
 <wire x1="14.5288" y1="5.1816" x2="12.5476" y2="3.2004" width="0.1524" layer="16"/>
@@
 <wire x1="12.5476" y1="1.8076" x2="12.54" y2="1.8" width="0.1524" layer="16"/>
 <wire x1="14.5288" y1="14.0208" x2="14.5288" y2="5.1816" width="0.1524" layer="16"/>
-<wire x1="12.8" y1="14.2926" x2="12.8" y2="15.6812" width="0.1524" layer="1"/>
-<wire x1="12.8" y1="15.6812" x2="13.2478" y2="16.129" width="0.1524" layer="1"/>
+<wire x1="12.8" y1="14.2926" x2="14.257" y2="14.2926" width="0.1524" layer="1"/>
 </signal>
 <signal name="SWD_DIO">

Commit message: prepare for a new production run
Other:
- board text added: "PD4 SEPT19"
- board text removed: "NOV18"
Changed lines of the file:
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@@
 <grid distance="2" unitdist="mil" unit="mil" style="lines" multiple="1" display="no" altdistance="1" altunitdist="mil" altunit="mil"/>
 <layers>
-<layer number="1" name="Top" color="4" fill="1" visible="yes" active="yes"/>
-<layer number="2" name="Route2" color="1" fill="3" visible="yes" active="yes"/>
-<layer number="3" name="Route3" color="4" fill="3" visible="yes" active="yes"/>
-<layer number="4" name="Route4" color="1" fill="4" visible="yes" active="yes"/>
-<layer number="5" name="Route5" color="4" fill="4" visible="yes" active="yes"/>
-<layer number="6" name="Route6" color="1" fill="8" visible="yes" active="yes"/>
-<layer number="7" name="Route7" color="4" fill="8" visible="yes" active="yes"/>
-<layer number="8" name="Route8" color="1" fill="2" visible="yes" active="yes"/>
-<layer number="9" name="Route9" color="4" fill="2" visible="yes" active="yes"/>
-<layer number="10" name="Route10" color="1" fill="7" visible="yes" active="yes"/>
-<layer number="11" name="Route11" color="4" fill="7" visible="yes" active="yes"/>
-<layer number="12" name="Route12" color="1" fill="5" visible="yes" active="yes"/>
-<layer number="13" name="Route13" color="4" fill="5" visible="yes" active="yes"/>
-<layer number="14" name="Route14" color="1" fill="6" visible="yes" active="yes"/>
-<layer number="15" name="Route15" color="4" fill="6" visible="yes" active="yes"/>
+<layer number="1" name="Top" color="4" fill="1" visible="no" active="yes"/>
+<layer number="2" name="Route2" color="1" fill="3" visible="no" active="yes"/>
+<layer number="3" name="Route3" color="4" fill="3" visible="no" active="yes"/>
+<layer number="4" name="Route4" color="1" fill="4" visible="no" active="yes"/>
+<layer number="5" name="Route5" color="4" fill="4" visible="no" active="yes"/>
+<layer number="6" name="Route6" color="1" fill="8" visible="no" active="yes"/>
+<layer number="7" name="Route7" color="4" fill="8" visible="no" active="yes"/>
+<layer number="8" name="Route8" color="1" fill="2" visible="no" active="yes"/>
+<layer number="9" name="Route9" color="4" fill="2" visible="no" active="yes"/>
+<layer number="10" name="Route10" color="1" fill="7" visible="no" active="yes"/>
+<layer number="11" name="Route11" color="4" fill="7" visible="no" active="yes"/>
+<layer number="12" name="Route12" color="1" fill="5" visible="no" active="yes"/>
+<layer number="13" name="Route13" color="4" fill="5" visible="no" active="yes"/>
+<layer number="14" name="Route14" color="1" fill="6" visible="no" active="yes"/>
+<layer number="15" name="Route15" color="4" fill="6" visible="no" active="yes"/>
 <layer number="16" name="Bottom" color="1" fill="1" visible="yes" active="yes"/>
 <layer number="17" name="Pads" color="2" fill="1" visible="yes" active="yes"/>
@@
 <layer number="19" name="Unrouted" color="6" fill="1" visible="yes" active="yes"/>
 <layer number="20" name="Dimension" color="15" fill="1" visible="yes" active="yes"/>
-<layer number="21" name="tPlace" color="7" fill="1" visible="yes" active="yes"/>
+<layer number="21" name="tPlace" color="7" fill="1" visible="no" active="yes"/>
 <layer number="22" name="bPlace" color="7" fill="1" visible="yes" active="yes"/>
-<layer number="23" name="tOrigins" color="15" fill="1" visible="yes" active="yes"/>
+<layer number="23" name="tOrigins" color="15" fill="1" visible="no" active="yes"/>
 <layer number="24" name="bOrigins" color="15" fill="1" visible="yes" active="yes"/>
-<layer number="25" name="tNames" color="7" fill="1" visible="yes" active="yes"/>
+<layer number="25" name="tNames" color="7" fill="1" visible="no" active="yes"/>
 <layer number="26" name="bNames" color="7" fill="1" visible="yes" active="yes"/>
 <layer number="27" name="tValues" color="7" fill="1" visible="no" active="yes"/>
@@
 <layer number="37" name="tTest" color="7" fill="1" visible="no" active="yes"/>
 <layer number="38" name="bTest" color="7" fill="1" visible="no" active="yes"/>
-<layer number="39" name="tKeepout" color="4" fill="11" visible="yes" active="yes"/>
+<layer number="39" name="tKeepout" color="4" fill="11" visible="no" active="yes"/>
 <layer number="40" name="bKeepout" color="1" fill="11" visible="yes" active="yes"/>
-<layer number="41" name="tRestrict" color="4" fill="10" visible="yes" active="yes"/>
+<layer number="41" name="tRestrict" color="4" fill="10" visible="no" active="yes"/>
 <layer number="42" name="bRestrict" color="1" fill="10" visible="yes" active="yes"/>
 <layer number="43" name="vRestrict" color="2" fill="10" visible="no" active="yes"/>
@@
 <layer number="49" name="Reference" color="7" fill="1" visible="no" active="yes"/>
 <layer number="50" name="dxf" color="7" fill="1" visible="no" active="yes"/>
-<layer number="51" name="tDocu" color="7" fill="1" visible="yes" active="yes"/>
+<layer number="51" name="tDocu" color="7" fill="1" visible="no" active="yes"/>
 <layer number="52" name="bDocu" color="7" fill="1" visible="yes" active="yes"/>
 <layer number="53" name="tGND_GNDA" color="7" fill="1" visible="no" active="yes"/>
@@
 <circle x="14.097" y="18.4912" radius="1.5748" width="0.254" layer="25"/>
 <polygon width="0.3048" layer="42">
-<vertex x="1.27" y="40.132"/>
+<vertex x="0.254" y="40.132"/>
 <vertex x="3.302" y="40.132"/>
 <vertex x="3.81" y="39.624"/>
 <vertex x="3.81" y="36.83"/>
 <vertex x="3.302" y="36.322"/>
-<vertex x="2.032" y="36.322"/>
-<vertex x="1.27" y="37.084"/>
+<vertex x="0.4572" y="36.322"/>
+<vertex x="0.254" y="36.5252"/>
 </polygon>
 <text x="12.446" y="19.9644" size="1.016" layer="25" font="vector">A</text>
-<text x="1.778" y="35.56" size="1.016" layer="26" font="vector" rot="MR270">NOV18</text>
+<text x="1.778" y="35.56" size="1.016" layer="26" font="vector" rot="MR270">PD4 SEPT19</text>
 </plain>
 <attributes>
