File: pcb/exixe14/exixe14.sch (EAGLE design)
At the start: 50 parts, among them IC1 STM32F042K6

Commit message: removed DP resistor, new pogo firmware
Parts:
- removed R20, R21: 10K, joyAnalog:RESISTOR0805-RES
Connections:
- removed net N$17: Q12.C, R21.1
- removed net N$18: Q11.C, R20.1
- net NIXIE_DOT_LEFT: now also Q11.C; no longer R20.2
- net NIXIE_DOT_RIGHT: now also Q12.C; no longer R21.2
Changed lines of the file:
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@@
 <?xml version="1.0" encoding="utf-8"?>
 <!DOCTYPE eagle SYSTEM "eagle.dtd">
-<eagle version="8.3.2">
+<eagle version="9.1.3">
 <drawing>
 <settings>
-<setting alwaysvectorfont="no"/>
+<setting alwaysvectorfont="yes"/>
 <setting keepoldvectorfont="yes"/>
 <setting verticaltext="up"/>
@@
 <part name="GND18" library="joyAnalog" deviceset="GND" device=""/>
 <part name="R19" library="joyAnalog" deviceset="RESISTOR" device="0805-RES" value="1M"/>
-<part name="R20" library="joyAnalog" deviceset="RESISTOR" device="0805-RES" value="10K"/>
-<part name="R21" library="joyAnalog" deviceset="RESISTOR" device="0805-RES" value="10K"/>
 <part name="R25" library="joyAnalog" deviceset="RESISTOR" device="0805-RES" value="10K"/>
 <part name="GND16" library="joyAnalog" deviceset="GND" device=""/>
@@
 <instance part="GND18" gate="1" x="378.46" y="-76.2"/>
 <instance part="R19" gate="G$1" x="378.46" y="-58.42" rot="R270"/>
-<instance part="R20" gate="G$1" x="238.76" y="53.34"/>
-<instance part="R21" gate="G$1" x="238.76" y="27.94"/>
 <instance part="R25" gate="G$1" x="429.26" y="33.02" rot="R90"/>
 <instance part="GND16" gate="1" x="429.26" y="25.4"/>
@@
 </segment>
 <segment>
-<pinref part="R20" gate="G$1" pin="2"/>
-<wire x1="261.62" y1="53.34" x2="243.84" y2="53.34" width="0.1524" layer="91"/>
+<wire x1="261.62" y1="53.34" x2="228.6" y2="53.34" width="0.1524" layer="91"/>
 <label x="248.92" y="53.34" size="1.778" layer="95"/>
+<pinref part="Q11" gate="A" pin="C"/>
 </segment>
 </net>
@@
 </segment>
 <segment>
-<pinref part="R21" gate="G$1" pin="2"/>
-<wire x1="261.62" y1="27.94" x2="243.84" y2="27.94" width="0.1524" layer="91"/>
+<wire x1="261.62" y1="27.94" x2="228.6" y2="27.94" width="0.1524" layer="91"/>
 <label x="248.92" y="27.94" size="1.778" layer="95"/>
+<pinref part="Q12" gate="A" pin="C"/>
 </segment>
 </net>
@@
 </segment>
 </net>
-<net name="N$17" class="0">
-<segment>
-<pinref part="Q12" gate="A" pin="C"/>
-<pinref part="R21" gate="G$1" pin="1"/>
-<wire x1="228.6" y1="27.94" x2="233.68" y2="27.94" width="0.1524" layer="91"/>
-</segment>
-</net>
-<net name="N$18" class="0">
-<segment>
-<pinref part="Q11" gate="A" pin="C"/>
-<pinref part="R20" gate="G$1" pin="1"/>
-<wire x1="228.6" y1="53.34" x2="233.68" y2="53.34" width="0.1524" layer="91"/>
-</segment>
-</net>

Commit message: cleanup
Parts:
- removed R18: 10K, joyAnalog:RESISTOR0805-RES
Connections:
- net +3V3: no longer R18.2
- net SPI_CS: no longer R18.1
Changed lines of the file:
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@@
 <part name="R15" library="joyAnalog" deviceset="RESISTOR" device="0805-RES" value="680"/>
 <part name="R16" library="joyAnalog" deviceset="RESISTOR" device="0805-RES" value="330"/>
-<part name="R18" library="joyAnalog" deviceset="RESISTOR" device="0805-RES" value="10K"/>
-<part name="+3V6" library="joyAnalog" deviceset="+3V3" device=""/>
 <part name="R22" library="joyAnalog" deviceset="RESISTOR" device="0805-RES" value="1M"/>
 <part name="R23" library="joyAnalog" deviceset="RESISTOR" device="0805-RES" value="68K"/>
@@
 <instance part="R15" gate="G$1" x="495.3" y="7.62"/>
 <instance part="R16" gate="G$1" x="495.3" y="-7.62"/>
-<instance part="R18" gate="G$1" x="347.98" y="-38.1" rot="R90"/>
-<instance part="+3V6" gate="G$1" x="347.98" y="-30.48" rot="MR0"/>
 <instance part="R22" gate="G$1" x="391.16" y="-63.5" rot="R180"/>
 <instance part="R23" gate="G$1" x="406.4" y="-73.66" rot="R90"/>
@@
 </segment>
 <segment>
-<pinref part="R18" gate="G$1" pin="2"/>
-<pinref part="+3V6" gate="G$1" pin="+3V3"/>
-</segment>
-<segment>
 <pinref part="C3" gate="G$1" pin="1"/>
 <pinref part="C2" gate="G$1" pin="1"/>
@@
 <wire x1="307.34" y1="-43.18" x2="330.2" y2="-43.18" width="0.1524" layer="91"/>
 <label x="307.34" y="-43.18" size="1.778" layer="95"/>
-<pinref part="R18" gate="G$1" pin="1"/>
-<wire x1="330.2" y1="-43.18" x2="347.98" y2="-43.18" width="0.1524" layer="91"/>
-<junction x="330.2" y="-43.18"/>
-</segment>
-<segment>
+</segment>
+<segment>
