File: pogo_rig/pcb/v0/exixe_pogo.brd (EAGLE design)
At the start: 90 x 60 mm, 44 parts, among them IC1 REG1117, IC2 STM32F030F4, SW2 324_SW324_SWITCH_FOOT_HOLE, U1 USBC_16P_CENTERED

Commit message: updated pogo board
Parts:
- removed R6, R7: 5.1K, joyAnalog:0805
- removed SW2: 324_SW324_SWITCH_FOOT_HOLE, 3pos_slide_switch:342_SWICH_FOOT_HOLE
- removed U1: USBC_16P_CENTERED, my_usbc_16p_centered:USBC_16P_FOOT
- added JP6, JP7: (no value), pinhead:1X06
- added LED2: (no value), clock:CHIP-LED0805
- added TP1, TP10, TP11, TP3, TP4, TP5, TP6, TP7, TP8, TP9: TEST-POINT3X5, clock:PAD.03X.05
- added X1: USB-MICROB, clock:USB-MICROB
- R2: value 22K -> (none); device joyAnalog:0805 -> clock:0805
- moved R2 25.9 mm to (60.4, 28.2), turned to 270 degrees
- moved C3 3.33 mm to (49.0, 8.00)
- moved C4 3.21 mm to (41.0, 8.00), turned to 180 degrees
- moved LED1 2.79 mm to (32.0, 28.2), turned to 0 degrees
- moved TP2 1.64 mm to (40.5, 24.4)
- moved JP3 1.27 mm to (30.0, 9.81)
- moved R4 1.27 mm to (9.14, 52.8)
- moved JP5 1.15 mm to (10.5, 56.0)
- moved JP4 1.02 mm to (60.0, 9.81)
- moved R1 0.51 mm to (29.5, 28.2), turned to 270 degrees
- moved C2 0.20 mm to (51.6, 23.6)
Connections:
- new net N$20: IC2.2, TP1.P$1
- new net N$23: TP5.P$1, U$1.PB6
- new net N$24: TP6.P$1, U$1.PA9
- new net N$26: TP8.P$1, U$2.PF0
- new net N$28: TP10.P$1, U$2.PB3
- new net N$29: TP11.P$1, U$2.PB6
- new net N$30: TP3.P$1, U$1.PF0
- net +3V3: now also JP6.1, JP7.1; no longer SW2.P$1, SW2.P$4
- net +5V: now also X1.VBUS; no longer U1.A4B9, U1.B4A9
- net GND: now also IC2.1, JP6.6, JP7.6, X1.GND, X1.P1, X1.P2, X1.P3, X1.P4, X1.P5, X1.P6; no longer R6.2, R7.2, U1.A1B12, U1.B11A12, U1.P$13, U1.P$14, U1.P$15, U1.P$16
- net HV_EN: now also IC2.18; no longer IC2.2
- net N$18: now also LED2.C, R2.1; no longer IC2.18, U1.A6, U1.B6
- net N$19: now also LED2.A; no longer U1.A7, U1.B7
- net N$22: now also TP4.P$1, U$1.PF1; no longer IC2.1, R2.1, SW2.P$2, SW2.P$3
- net N$25: now also TP7.P$1, U$1.PA1; no longer R6.1, U1.B5
- net N$27: now also TP9.P$1, U$2.PF1; no longer R7.1, U1.A5
Routing:
- net N$18: track 30.2 -> 2.59 mm, vias 2 -> 0
- net CS: track 65.3 -> 84.2 mm, vias 3 -> 1
- net N$19: track 26.9 -> 11.2 mm
- net N$3: track 79.1 -> 68.2 mm, vias 1 -> 0
- net +3V3: track 28.6 -> 20.1 mm, vias 7 -> 5
- net N$22: track 14.1 -> 5.72 mm
- net N$1: track 76.9 -> 69.0 mm, vias 1 -> 0
- net +5V: track 63.9 -> 58.0 mm
- net N$23: track 0.00 -> 5.34 mm
- net N$24: track 0.00 -> 5.22 mm
- net N$30: track 0.00 -> 5.10 mm
- net N$4: track 73.5 -> 69.1 mm, vias 1 -> 0
- net N$2: track 11.4 -> 15.6 mm
- net N$26: track 0.00 -> 3.42 mm
- net N$28: track 0.00 -> 3.21 mm
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Other:
- board text added: "A"
- board text added: "B"
- board text added: "C"
- board text added: "D"
- board text added: "E"
- board text added: "F"
- board text added: "G"
- board text added: "H"
- board text added: "HV_ON"
- board text added: "PA9"
- board text added: "PF0"
- board text added: "exixe pogo rig dekuNukem 2017"
- board text removed: "exixe pogo v2 dekuNukem JUN2019"
