File: pogo_rig/pcb/v0/exixe_pogo.sch (EAGLE design)
At the start: 44 parts, among them IC1 REG1117, IC2 STM32F030F4, SW2 324_SW324_SWITCH_FOOT_HOLE, U1 USBC_16P_CENTERED

Commit message: updated pogo board
Parts:
- removed R6, R7: 5.1K, joyAnalog:RESISTOR0805-RES
- removed SW2: 324_SW324_SWITCH_FOOT_HOLE, 3pos_slide_switch:324_SW324_SWITCH_FOOT_HOLE
- removed U1: USBC_16P_CENTERED, my_usbc_16p_centered:USBC_16P_CENTERED
- added JP6, JP7: (no value), pinhead:PINHD-1X6
- added LED2: (no value), clock:LEDCHIP-LED0805
- added TP1, TP10, TP11, TP3, TP4, TP5, TP6, TP7, TP8, TP9: TEST-POINT3X5, clock:TEST-POINT3X5
- added X1: USB-MICROB, clock:USB-MICROB
- R2: value 22K -> (none); device joyAnalog:RESISTOR0805-RES -> clock:RESISTOR0805-RES
Connections:
- new net N$20: IC2.PF0/OSC_IN, TP1.1
- new net N$23: TP5.1, U$1.PB6
- new net N$24: TP6.1, U$1.PA9
- new net N$26: TP8.1, U$2.PF0
- new net N$28: TP10.1, U$2.PB3
- new net N$29: TP11.1, U$2.TX
- new net N$30: TP3.1, U$1.PF0
- net +3V3: now also JP6.1, JP7.1; no longer SW2.1, SW2.4
- net +5V: now also X1.VBUS; no longer U1.VBUS
- net GND: now also IC2.BOOT0, JP6.6, JP7.6, X1.GND; no longer R6.2, R7.2, U1.GND
- net HV_EN: now also IC2.PA10; no longer IC2.PF0/OSC_IN
- net N$18: now also LED2.C, R2.1; no longer IC2.PA10, U1.DP1, U1.DP2
- net N$19: now also LED2.A; no longer U1.DN1, U1.DN2
- net N$22: now also TP4.1, U$1.PF1; no longer IC2.BOOT0, R2.1, SW2.2, SW2.3
- net N$25: now also TP7.1, U$1.PA1; no longer R6.1, U1.CC2
- net N$27: now also TP9.1, U$2.PF1; no longer R7.1, U1.CC1
Other:
- moved on the sheet: R2
